File: EEZ_DIB_BP3C_R3B3/EEZ_DIB_BP3C_r3B3.kicad_pcb (KiCad board)
At the start: 4 copper layers, 110 x 90 mm, 63 parts, among them IC1 TCA9534PWR, K1 RT424005, K2 RT424005, K3 RT424005, K4 RT424005, Q1 2N7002, Q2 2N7002, Q3 2N7002, Q4 2N7002, X1 ZL202-20G, X2 ZL202-20G, X3 ZL202-20G, X4 DS1022-2*20RF11, X5 DS1023-2*14S21, X6 DS1023-2*14S21, X7 DS1023-2*14S21

Commit message: Boards are now combined, but not synced with schematics
Parts:
- moved C2 364.0 mm to (556.2, 105.5)
- moved D1 364.0 mm to (526.9, 145.9)
- moved Q1 364.0 mm to (528.7, 150.9)
- moved Q4 364.0 mm to (541.6, 150.9)
- moved R10 364.0 mm to (558.9, 81.3)
- moved R11 364.0 mm to (558.9, 84.1)
- moved R3 364.0 mm to (559.3, 146.3)
- moved R5 364.0 mm to (559.3, 148.5)
- moved U$4 364.0 mm to (525.8, 76.5)
- moved X2 364.0 mm to (515.3, 119.6)
- moved X3 364.0 mm to (550.8, 119.6)
- moved X6 364.0 mm to (515.3, 72.6)
- moved X7 364.0 mm to (550.8, 72.6)
- moved D3 364.0 mm to (522.7, 150.9)
- moved D4 364.0 mm to (500.4, 150.9)
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