File: EEZ_BB3_CM4_R1B0/EEZ_DIB_BP3C_r3B3.kicad_pcb (KiCad board)
At the start: 4 copper layers, 110 x 90 mm, 63 parts, among them IC1 TCA9534PWR, K1 RT424005, K2 RT424005, K3 RT424005, K4 RT424005, Q1 2N7002, Q2 2N7002, Q3 2N7002, Q4 2N7002, X1 ZL202-20G, X2 ZL202-20G, X3 ZL202-20G, X4 DS1022-2*20RF11, X5 DS1023-2*14S21, X6 DS1023-2*14S21, X7 DS1023-2*14S21

Commit message: Importing BP3
Parts:
- Q201: renamed from Q1; value 2N7002 -> (none)
- Q202: renamed from Q2; value 2N7002 -> (none)
- Q203: renamed from Q3; value 2N7002 -> (none)
- Q204: renamed from Q4; value 2N7002 -> (none)
- renumbered C1 to C201, C2 to C301, D3 to D201, D4 to D202, D1 to D203, D2 to D204, D5 to D205, D6 to D206, D9 to D301, D7 to D302, D8 to D303, FM1 to FM201, FM2 to FM202, FM3 to FM203, IC1 to IC201, JP1 to JP201, JP2 to JP301, JP8 to JP302, JP3 to JP303, JP4 to JP304, JP9 to JP305, JP5 to JP306, JP6 to JP307, JP10 to JP308, JP7 to JP309, K1 to K201, K3 to K202, K4 to K203, K2 to K204, LABEL1 to LABEL201, LED1 to LED201, LED2 to LED202, LED3 to LED203, LED4 to LED204, LED5 to LED301, LED6 to LED302, R2 to R201, R4 to R202, R6 to R203, R8 to R204, R1 to R205, R3 to R206, R5 to R207, R7 to R208, R10 to R301, R11 to R302, R9 to R303, X1 to X201, X2 to X202, X3 to X203, X5 to X301, X4 to X302, X6 to X303, X7 to X304, ZD1 to ZD201
Connections:
- net +VAUX renamed /EEZ_DIB_BP3C_r3B3_3/+VAUX
- net CH1_IN+ renamed /EEZ_DIB_BP3C_r3B3_2/CH1_IN+
- net CH1_OUT+ renamed /EEZ_DIB_BP3C_r3B3_2/CH1_OUT+
- net CH1_OUT- renamed /EEZ_DIB_BP3C_r3B3_2/CH1_OUT-
- net CH2_IN+ renamed /EEZ_DIB_BP3C_r3B3_2/CH2_IN+
- net CH2_IN- renamed /EEZ_DIB_BP3C_r3B3_2/CH2_IN-
- net CH2_OUT+ renamed /EEZ_DIB_BP3C_r3B3_2/CH2_OUT+
- net CH2_OUT- renamed /EEZ_DIB_BP3C_r3B3_2/CH2_OUT-
- net CH3+ renamed /EEZ_DIB_BP3C_r3B3_2/CH3+
- net CH3- renamed /EEZ_DIB_BP3C_r3B3_2/CH3-
- net OE_SYNC renamed /EEZ_DIB_BP3C_r3B3_3/OE_SYNC
- net OUT_CGND renamed /EEZ_DIB_BP3C_r3B3_2/OUT_CGND
- net OUT_PAR renamed /EEZ_DIB_BP3C_r3B3_2/OUT_PAR
- net OUT_SER renamed /EEZ_DIB_BP3C_r3B3_2/OUT_SER
- net OUT_SRA renamed /EEZ_DIB_BP3C_r3B3_2/OUT_SRA
- net SER_PAR renamed Net-(K202-Pad11A)
- net SPI2_CLK renamed /EEZ_DIB_BP3C_r3B3_3/SPI2_CLK
- net SPI2_CSA renamed /EEZ_DIB_BP3C_r3B3_3/SPI2_CSA
- net SPI2_CSB renamed /EEZ_DIB_BP3C_r3B3_3/SPI2_CSB
- net SPI2_IRQ renamed /EEZ_DIB_BP3C_r3B3_3/SPI2_IRQ
- net SPI2_MISO renamed /EEZ_DIB_BP3C_r3B3_3/SPI2_MISO
- net SPI2_MOSI renamed /EEZ_DIB_BP3C_r3B3_3/SPI2_MOSI
- net SPI4_CLK renamed /EEZ_DIB_BP3C_r3B3_3/SPI4_CLK
- net SPI4_CSA renamed /EEZ_DIB_BP3C_r3B3_3/SPI4_CSA
- net SPI4_CSB renamed /EEZ_DIB_BP3C_r3B3_3/SPI4_CSB
- net SPI4_CSC renamed /EEZ_DIB_BP3C_r3B3_3/SPI4_CSC
- net SPI4_IRQ renamed /EEZ_DIB_BP3C_r3B3_3/SPI4_IRQ
- net SPI4_MISO renamed /EEZ_DIB_BP3C_r3B3_3/SPI4_MISO
- net SPI4_MOSI renamed /EEZ_DIB_BP3C_r3B3_3/SPI4_MOSI
- net SPI5_CLK renamed /EEZ_DIB_BP3C_r3B3_3/SPI5_CLK
- net SPI5_CSA renamed /EEZ_DIB_BP3C_r3B3_3/SPI5_CSA
- net SPI5_CSB renamed /EEZ_DIB_BP3C_r3B3_3/SPI5_CSB
- net SPI5_CSC renamed /EEZ_DIB_BP3C_r3B3_3/SPI5_CSC
- net SPI5_IRQ renamed /EEZ_DIB_BP3C_r3B3_3/SPI5_IRQ
- net SPI5_MISO renamed /EEZ_DIB_BP3C_r3B3_3/SPI5_MISO
- net SPI5_MOSI renamed /EEZ_DIB_BP3C_r3B3_3/SPI5_MOSI
- net UART_RX renamed /EEZ_DIB_BP3C_r3B3_3/UART_RX
- net UART_TX renamed /EEZ_DIB_BP3C_r3B3_3/UART_TX
- net ~{FAULT} renamed /EEZ_DIB_BP3C_r3B3_3/~{FAULT}
- net ~{MRESET} renamed /EEZ_DIB_BP3C_r3B3_3/~{MRESET}
- net ~{RESET} renamed /EEZ_DIB_BP3C_r3B3_3/~{RESET}
- IC201 pad 13: (no net) -> unconnected-(IC201-Pad13)
- K201 pad 12A: (no net) -> unconnected-(K201-Pad12A)
- K201 pad 12B: (no net) -> unconnected-(K201-Pad12B)
- K204 pad 12A: (no net) -> unconnected-(K204-Pad12A)
- X301 pad 20: (no net) -> unconnected-(X301-Pad20)
- X303 pad 20: (no net) -> unconnected-(X303-Pad20)
- X304 pad 20: (no net) -> unconnected-(X304-Pad20)
Routing:
- net HOLE_MCU4: vias 1 -> 0
- net HOLE_MCU3: vias 1 -> 0
- net HOLE_MCU2: vias 1 -> 0
- net HOLE_MCU1: vias 1 -> 0
- net (no net): vias 0 -> 4
