File: EEZ_BB3_CM4_R1B0/EEZ_DIB_BP3C_r3B3_2.kicad_sch (KiCad schematic)
At the start: 37 parts, among them IC1 TCA9534PWR, K1 RT424005, K2 RT424005, K3 RT424005, K4 RT424005, X1 ZL202-20G, X2 ZL202-20G, X3 ZL202-20G

Commit message: Importing BP3
Parts:
- renumbered C1 to C201, D3 to D201, D4 to D202, D1 to D203, D2 to D204, D5 to D205, D6 to D206, FM1 to FM201, FM2 to FM202, FM3 to FM203, IC1 to IC201, JP1 to JP201, K1 to K201, K3 to K202, K4 to K203, K2 to K204, LABEL1 to LABEL201, LED1 to LED201, LED2 to LED202, LED3 to LED203, LED4 to LED204, Q1 to Q201, Q2 to Q202, Q3 to Q203, Q4 to Q204, R2 to R201, R4 to R202, R6 to R203, R8 to R204, R1 to R205, R3 to R206, R5 to R207, R7 to R208, X1 to X201, X2 to X202, X3 to X203, ZD1 to ZD201

Commit message: Removing Backups, addin new version
Parts:
- removed LABEL201: HR000002, EEZ_DIB_BP3C_r3B3:CERT-SMALL-SILK, symbol EEZ_DIB_BP3C_r3B3-eagle-import:OSHWA-CERT-SMALL
Changed lines of the file:
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@@
     (pin "20")
-  )
-  (symbol (lib_id "EEZ_DIB_BP3C_r3B3-eagle-import:OSHWA-CERT-SMALL") (at 26.035 189.23 0) (unit 1)
-    (in_bom yes) (on_board yes)
-    (property "Reference" "LABEL201" (id 0) (at 26.035 189.23 0)
-      (effects (font (size 1.27 1.27)) hide)
-    )
-    (property "Value" "HR000002" (id 1) (at 20.066 191.77 0)
-      (effects (font (size 1.778 1.778)) (justify left bottom))
-    )
-    (property "Footprint" "EEZ_DIB_BP3C_r3B3:CERT-SMALL-SILK" (id 2) (at 26.035 189.23 0)
-      (effects (font (size 1.27 1.27)) hide)
-    )
-    (property "Datasheet" "" (id 3) (at 26.035 189.23 0)
-      (effects (font (size 1.27 1.27)) hide)
-    )
   )
   (symbol (lib_id "EEZ_DIB_BP3C_r3B3-eagle-import:R-EU_R0805") (at 124.46 93.98 180) (unit 1)
