File: EEZ_BB3_CM4_R1B0/IO_connectors_Encoder_user_SW.kicad_sch (KiCad schematic)
At the start: 39 parts, among them IC1 TPD4E001DRLR, IC2 74AUP1G74DC.125, IC3 CD74HC4050PWR, SW1 TL1100CF160Q, SW2 PEC16-2215F-S0024, X1 DS1024-2*20R0, X2 DS1013-16SSIB1, X3 691322110005

Commit message: Removing Backups, addin new version
Parts:
- removed LABEL1: HR000002, EEZ_DIB_MCU_r3B4:CERT-SMALL-SILK, symbol EEZ_DIB_MCU_r3B4-eagle-import:OSHWA-CERT-SMALL
Changed lines of the file:
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@@
     (pin "2")
-  )
-  (symbol (lib_id "EEZ_DIB_MCU_r3B4-eagle-import:OSHWA-CERT-SMALL") (at 26.67 186.69 0) (unit 1)
-    (in_bom yes) (on_board yes)
-    (property "Reference" "LABEL1" (id 0) (at 26.67 186.69 0)
-      (effects (font (size 1.27 1.27)) hide)
-    )
-    (property "Value" "HR000002" (id 1) (at 20.701 189.23 0)
-      (effects (font (size 1.778 1.778)) (justify left bottom))
-    )
-    (property "Footprint" "EEZ_DIB_MCU_r3B4:CERT-SMALL-SILK" (id 2) (at 26.67 186.69 0)
-      (effects (font (size 1.27 1.27)) hide)
-    )
-    (property "Datasheet" "" (id 3) (at 26.67 186.69 0)
-      (effects (font (size 1.27 1.27)) hide)
-    )
   )
   (symbol (lib_id "EEZ_DIB_MCU_r3B4-eagle-import:SN74LVC1G74DCTR-VSSOP") (at 241.3 149.86 0) (unit 2)
