File: EEZ_DIB_MCU_r3B4/SDRAM.kicad_sch (KiCad schematic)
At the start: 8 parts, among them IC7 IS42S16400J

Commit message: Switching MCU to KiCad 7 - moving MCU and SDRAM from board
Other:
- note removed: "SDRAM, JTAG, I2C EEPROM, SD Card"
Changed lines of the file:
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@@
     (effects (font (size 1.27 1.0795)) (justify left bottom))
   )
-  (text "SDRAM, JTAG, I2C EEPROM, SD Card" (at 182.88 170.18 0)
+  (text "SDRAM" (at 182.88 170.18 0)
     (effects (font (size 2.54 2.54)) (justify left bottom))
   )
