File: EEZ_DIB_MCU_r3B4/STM32F7_MCU.kicad_sch (KiCad schematic)
At the start: 50 parts, among them IC4 STM32F769IIT6, IC5 LD1117ADT33TR, Y1 25MHz, Y2 XTAL016178-85SMX

Commit message: Switching MCU to KiCad 7 - moving MCU and SDRAM from board
Parts:
- removed C14: EEEFK1V220R, EEZ_DIB_MCU_r3B4:PANASONIC_C, symbol EEZ_DIB_MCU_r3B4-eagle-import:ECAPPANASONIC_C
- removed C15: 100n, EEZ_DIB_MCU_r3B4:C0603, symbol EEZ_DIB_MCU_r3B4-eagle-import:C-EUC0603
- removed D1: SMBJ5.0A-TR, EEZ_DIB_MCU_r3B4:DO214AA, symbol EEZ_DIB_MCU_r3B4-eagle-import:DIODEDO214AA
- removed IC5: LD1117ADT33TR, EEZ_DIB_MCU_r3B4:DPACK, symbol EEZ_DIB_MCU_r3B4-eagle-import:LD117A?DT
- added C39: N.C., EEZ_DIB_MCU_r3B4:C0603, symbol EEZ_DIB_MCU_r3B4-eagle-import:C-EUC0603
- added IC6: N.C., EEZ_DIB_MCU_r3B4:DRL6, symbol EEZ_DIB_MCU_r3B4-eagle-import:TPD4E001-DRL
- added JP5: JP2-CUT, EEZ_DIB_MCU_r3B4:JP2-CUT, symbol EEZ_DIB_MCU_r3B4-eagle-import:JP2-CUT
- added R19, R20, R21, R22: N.C., EEZ_DIB_MCU_r3B4:R0805, symbol EEZ_DIB_MCU_r3B4-eagle-import:R-EU_R0805
- added X4: N.C., EEZ_DIB_MCU_r3B4:SSW-106-02-S-S, symbol EEZ_DIB_MCU_r3B4-eagle-import:SSW-106-02-S-S
Connections:
- net +3V3: now also C39.1, IC6.6 (VCC), JP5.1
- net GND: now also C39.2, IC6.3 (GND), R19.1, X4.3 (1)
- net SYS_JTCK-SWCLK: now also R21.1
- net SYS_JTDO-SWO: now also IC6.5 (IO4), X4.6 (1)
- net SYS_JTMS-SWDIO: now also R20.1
- net ~{RESET}: now also R22.1
- new net: IC6.4 (IO3), R22.2, X4.5 (1)
- new net: JP5.2, R19.2, X4.1
- new net TCK: IC6.1 (IO1), R21.2, X4.2 (1)
- new net TMS: IC6.2 (IO2), R20.2, X4.4 (1)
Other:
- note added: "Gnd 3"
- note added: "JTAG/SWD (optional)"
- note added: "NRST 5"
- note added: "STM-32 board SWD header"
- note added: "SWCLK 2"
- note added: "SWDIO 4"
- note added: "SWO 6"
- note added: "Vdd target 1"
