File: EEZ_DIB_MCU_r3B4/EEZ_DIB_MCU_r3B4.kicad_pcb (KiCad board)
At the start: 4 copper layers, 139.5 x 70 mm, 200 parts, among them IC1 TPD4E001DRLR, IC11 TPS2051BDBVR, IC12 TPS61169DCKR, IC13 TPD4E001DRLR, IC14 TSC2007IPW, IC15 N.C., IC16 DP83848CVV/NOPB, IC2 74AUP1G74DC.125, IC3 CD74HC4050PWR, IC4 STM32F769IIT6, IC5 LD1117ADT33TR, IC6 N.C., IC7 IS42S16400J, IC8 AT24C256C-SSHL-B, IC9 N.C., J1 5033981892, J2 67803-8020, Q1 N.C., Q2 2N7002, SW1 TL1100CF160Q, SW2 PEC16-2215F-S0024, X1 DS1024-2*20R0, X2 DS1013-16SSIB1, X3 691322110005, X4 N.C., X5 LMJTAB881243M-L, Y1 25MHz, Y2 XTAL016178-85SMX

Commit message: Adding connectors, grouping parts, removing most of the routing
Parts:
- removed SH1: , EEZ_DIB_MCU_r3B4:SHORT_NOHOLE
- added J10: DF40C-100DP-0.4V(51), connectors:HRS_DF40C-100DP-0.4V(51), B.Cu at (196.3, -58.6)
- added J11: DF40C-100DP-0.4V(51), connectors:HRS_DF40C-100DP-0.4V(51), B.Cu at (196.3, -92.6)
- added Module1: ComputeModule4-CM4, CM4IO:Raspberry-Pi-4-Compute-Module, F.Cu at (113.3, 107.7)
- moved C57 163.5 mm to (-51.6, 181.8)
- moved C58 163.5 mm to (-53.5, 181.8)
- moved IC14 163.5 mm to (-56.4, 181.1)
- moved C15 148.2 mm to (-11.5, 254.3)
- moved D1 148.2 mm to (-15.9, 215.3)
- moved C14 148.2 mm to (-16.8, 253.7)
- moved IC5 148.2 mm to (-9.87, 262.1)
- moved C50 137.1 mm to (-55.0, 54.4)
- moved C53 137.1 mm to (-45.6, 60.1)
- moved JP8 137.1 mm to (-44.4, 73.8)
- moved R26 137.1 mm to (-52.8, 54.9)
- moved R29 137.1 mm to (-47.9, 55.1)
- moved ZD1 137.1 mm to (-53.1, 66.7)
- moved C51 137.1 mm to (-47.9, 60.1)
- moved D2 137.1 mm to (-50.0, 59.8)
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Routing:
- net I2C1_SDA: track 125.2 -> 0.91 mm, vias 7 -> 0
- net I2C1_SCL: track 126.7 -> 2.86 mm, vias 6 -> 0
- net UART_TX/DOUT1: track 115.2 -> 0.00 mm, vias 6 -> 0
- net SPI2_MISO: track 111.5 -> 0.71 mm, vias 4 -> 0
- net RTC_REF: track 99.2 -> 0.68 mm, vias 2 -> 0
- net PWR_SSTART: track 94.4 -> 0.00 mm, vias 2 -> 0
- net OE_SYNC: track 78.5 -> 0.59 mm, vias 2 -> 0
- net SPI2_IRQ: track 74.8 -> 0.88 mm, vias 4 -> 0
- net SPI5_CSA: track 70.8 -> 0.00 mm, vias 1 -> 0
- net SPI5_CLK: track 68.6 -> 0.00 mm, vias 1 -> 0
- net SPI5_MISO: track 65.1 -> 0.00 mm, vias 1 -> 0
- net SPI5_MOSI: track 64.4 -> 0.00 mm, vias 1 -> 0
- net SPI2_MOSI: track 62.9 -> 0.00 mm, vias 2 -> 0
- net /STM32F7 MCU/VBAT: track 69.6 -> 8.70 mm, vias 5 -> 0
- net USER_SW: track 88.5 -> 28.3 mm, vias 2 -> 0
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
Commit message: Splitting SoM and MCU board
Parts:
- removed C10, C12: 18p, EEZ_DIB_MCU_r3B4:C0603
- removed C11, C13: 4p7, EEZ_DIB_MCU_r3B4:C0603
- removed C16, C17, C18, C19, C20, C21, C22, C23, C25, C26, C27, C28, C29, C30, C33, C36, C42, C43, C44, C45, C46, C47, C48, C60, C61, C62, C63, C64, C65, C67, C68, C69, C70, C71: 100n, EEZ_DIB_MCU_r3B4:C0603
- removed C24, C34, C35: 1u, EEZ_DIB_MCU_r3B4:C0805
- removed C31, C32, C37, C38: 2u2, EEZ_DIB_MCU_r3B4:C0805
- removed C39, C59: N.C., EEZ_DIB_MCU_r3B4:C0603
- removed C66: 10u, EEZ_DIB_MCU_r3B4:EC1206
- removed IC15, IC6: N.C., EEZ_DIB_MCU_r3B4:DRL6
- removed IC16: DP83848CVV/NOPB, EEZ_DIB_MCU_r3B4:PT48
- removed IC4: STM32F769IIT6, EEZ_DIB_MCU_r3B4:LQFP-176_24X24MM
- removed IC7: IS42S16400J, EEZ_DIB_MCU_r3B4:TSOPII-54
- removed J10, J11: DF40C-100DP-0.4V(51), connectors:HRS_DF40C-100DP-0.4V(51)
- removed JP10, JP11, JP12, JP5: JP2-CUT, EEZ_DIB_MCU_r3B4:JP2-CUT
- removed JP13, JP14: JP2-NOCUT, EEZ_DIB_MCU_r3B4:JP2-NOCUT
- removed JP3, JP4: ~, EEZ_DIB_MCU_r3B4:R_0805
- removed L1, L3: BLM18AG102SH1D, EEZ_DIB_MCU_r3B4:BEAD0603
- removed LED2: N.C., EEZ_DIB_MCU_r3B4:LED_0805
- removed R12, R15: 4K7, EEZ_DIB_MCU_r3B4:R0805
- removed R13: 10K, EEZ_DIB_MCU_r3B4:R0805
- removed R14, R19, R20, R21, R22, R41, R44, R45, R46: N.C., EEZ_DIB_MCU_r3B4:R0805
- removed R16, R17, R38: 1K5, EEZ_DIB_MCU_r3B4:R0805
- removed R18: 47R, EEZ_DIB_MCU_r3B4:R0805
- removed R39, R40, R43, R48: 49R9, EEZ_DIB_MCU_r3B4:R0805
- removed R42, R47, R49, R52, R53, R55: 2K2, EEZ_DIB_MCU_r3B4:R0805
- removed R50, R51: 220R, EEZ_DIB_MCU_r3B4:R0805
- removed R54: 4K87, EEZ_DIB_MCU_r3B4:R0805
- removed RN1, RN2, RN3, RN4, RN5, RN6, RN7: DR1206-33R-4/8, EEZ_DIB_MCU_r3B4:CAY16
- removed TP1: ~, EEZ_DIB_MCU_r3B4:PCB_SHIELD_TAB
- removed X4: N.C., EEZ_DIB_MCU_r3B4:SSW-106-02-S-S
- removed Y1: 25MHz, EEZ_DIB_MCU_r3B4:HC-49_4H
- removed Y2: XTAL016178-85SMX, EEZ_DIB_MCU_r3B4:85SMX
- moved C57 156.1 mm to (103.5, 163.9)
- moved C58 156.1 mm to (101.6, 163.9)
- moved IC14 156.1 mm to (98.7, 163.3)
- moved C53 129.3 mm to (27.8, 166.6)
- moved IC12 129.3 mm to (22.9, 161.7)
- moved JP8 129.3 mm to (29.0, 180.3)
- moved L2 129.3 mm to (19.8, 166.5)
- moved R26 129.3 mm to (20.5, 161.3)
- moved R29 129.3 mm to (25.5, 161.6)
- moved C51 129.3 mm to (25.4, 166.6)
- moved D2 129.3 mm to (23.4, 166.3)
- moved JP9 129.3 mm to (49.9, 178.7)
- moved R37 129.3 mm to (46.6, 179.5)
- moved C50 129.3 mm to (18.4, 160.9)
- moved ZD1 129.3 mm to (20.3, 173.2)
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Connections:
- Module1 pad 1: unconnected-(Module1A-GND-Pad1) -> GND
- Module1 pad 100: unconnected-(Module1A-nEXTRST-Pad100) -> RESET
- Module1 pad 13: unconnected-(Module1A-GND-Pad13) -> GND
- Module1 pad 14: unconnected-(Module1A-GND-Pad14) -> GND
- Module1 pad 2: unconnected-(Module1A-GND-Pad2) -> GND
- Module1 pad 21: unconnected-(Module1A-PI_nLED_Activity-Pad21) -> ACT_LED
- Module1 pad 22: unconnected-(Module1A-GND-Pad22) -> GND
- Module1 pad 23: unconnected-(Module1A-GND-Pad23) -> GND
- Module1 pad 24: unconnected-(Module1A-GPIO26-Pad24) -> SPI5_CSB
- Module1 pad 25: unconnected-(Module1A-GPIO21-Pad25) -> SPI4_CLK
- Module1 pad 26: unconnected-(Module1A-GPIO19-Pad26) -> SPI4_MISO
- Module1 pad 27: unconnected-(Module1A-GPIO20-Pad27) -> SPI4_MOSI
- Module1 pad 28: unconnected-(Module1A-GPIO13-Pad28) -> SPI5_MISO
- Module1 pad 29: unconnected-(Module1A-GPIO16-Pad29) -> DOUT2
- Module1 pad 30: unconnected-(Module1A-GPIO6-Pad30) -> SPI2_IRQ
- Module1 pad 31: unconnected-(Module1A-GPIO12-Pad31) -> SPI5_CSA
- Module1 pad 32: unconnected-(Module1A-GND-Pad32) -> GND
- Module1 pad 33: unconnected-(Module1A-GND-Pad33) -> GND
- Module1 pad 34: unconnected-(Module1A-GPIO5-Pad34) -> DAC_OUT1
- Module1 pad 35: unconnected-(Module1A-ID_SC-Pad35) -> UART_RX/DIN1
- Module1 pad 36: unconnected-(Module1A-ID_SD-Pad36) -> UART_TX/DOUT1
- Module1 pad 37: unconnected-(Module1A-GPIO7-Pad37) -> SPI2_CSB
- Module1 pad 38: unconnected-(Module1A-GPIO11-Pad38) -> SPI2_CLK
- Module1 pad 39: unconnected-(Module1A-GPIO8-Pad39) -> SPI2_CSA
- Module1 pad 40: unconnected-(Module1A-GPIO9-Pad40) -> SPI2_MISO
- Module1 pad 41: unconnected-(Module1A-GPIO25-Pad41) -> DIN2
- Module1 pad 42: unconnected-(Module1A-GND-Pad42) -> GND
- Module1 pad 43: unconnected-(Module1A-GND-Pad43) -> GND
- Module1 pad 44: unconnected-(Module1A-GPIO10-Pad44) -> SPI2_MOSI
- Module1 pad 45: unconnected-(Module1A-GPIO24-Pad45) -> ENC_SW
- Module1 pad 46: unconnected-(Module1A-GPIO22-Pad46) -> SPI5_IRQ
- Module1 pad 47: unconnected-(Module1A-GPIO23-Pad47) -> USER_SW
- Module1 pad 48: unconnected-(Module1A-GPIO27-Pad48) -> SPI4_IRQ
- Module1 pad 49: unconnected-(Module1A-GPIO18-Pad49) -> SPI4_CSA
- Module1 pad 50: unconnected-(Module1A-GPIO17-Pad50) -> SPI4_CSB
- Module1 pad 51: unconnected-(Module1A-GPIO15-Pad51) -> SPI5_CLK
- Module1 pad 52: unconnected-(Module1A-GND-Pad52) -> GND
- Module1 pad 53: unconnected-(Module1A-GND-Pad53) -> GND
- Module1 pad 54: unconnected-(Module1A-GPIO4-Pad54) -> IRQ_TOUCH
- Module1 pad 55: unconnected-(Module1A-GPIO14-Pad55) -> SPI5_MOSI
- Module1 pad 56: unconnected-(Module1A-GPIO3-Pad56) -> ENC_B
- Module1 pad 57: unconnected-(Module1A-SD_CLK-Pad57) -> SDMMC1_CK
- Module1 pad 58: unconnected-(Module1A-GPIO2-Pad58) -> ENC_A
- Module1 pad 59: unconnected-(Module1A-GND-Pad59) -> GND
- Module1 pad 60: unconnected-(Module1A-GND-Pad60) -> GND
- Module1 pad 61: unconnected-(Module1A-SD_DAT3-Pad61) -> SDMMC1_D0
- Module1 pad 62: unconnected-(Module1A-SD_CMD-Pad62) -> SDMMC1_CMD
- Module1 pad 63: unconnected-(Module1A-SD_DAT0-Pad63) -> SDMMC1_D0
- Module1 pad 65: unconnected-(Module1A-GND-Pad65) -> GND
- Module1 pad 66: unconnected-(Module1A-GND-Pad66) -> GND
- Module1 pad 7: unconnected-(Module1A-GND-Pad7) -> GND
- Module1 pad 71: unconnected-(Module1A-GND-Pad71) -> GND
- Module1 pad 74: unconnected-(Module1A-GND-Pad74) -> GND
- Module1 pad 75: unconnected-(Module1A-SD_PWR_ON-Pad75) -> SD_DETECT
- Module1 pad 77: unconnected-(Module1A-+5v_(Input)-Pad77) -> +5V
- Module1 pad 79: unconnected-(Module1A-+5v_(Input)-Pad79) -> +5V
- Module1 pad 8: unconnected-(Module1A-GND-Pad8) -> GND
- Module1 pad 80: unconnected-(Module1A-SCL0-Pad80) -> I2C1_SCL
- Module1 pad 81: unconnected-(Module1A-+5v_(Input)-Pad81) -> +5V
- Module1 pad 82: unconnected-(Module1A-SDA0-Pad82) -> I2C1_SDA
- Module1 pad 83: unconnected-(Module1A-+5v_(Input)-Pad83) -> +5V
- Module1 pad 84: unconnected-(Module1A-+3.3v_(Output)-Pad84) -> CM4_3.3V
- Module1 pad 85: unconnected-(Module1A-+5v_(Input)-Pad85) -> +5V
- Module1 pad 86: unconnected-(Module1A-+3.3v_(Output)-Pad86) -> CM4_3.3V
- Module1 pad 87: unconnected-(Module1A-+5v_(Input)-Pad87) -> +5V
- Module1 pad 93: unconnected-(Module1A-nRPIBOOT-Pad93) -> BOOT0
- Module1 pad 94: unconnected-(Module1A-AnalogIP1-Pad94) -> ADC2_IN6
- Module1 pad 95: unconnected-(Module1A-nPI_LED_PWR-Pad95) -> CM4_3.3V
- Module1 pad 96: unconnected-(Module1A-AnalogIP0-Pad96) -> ADC1_IN5
- Module1 pad 97: unconnected-(Module1A-Camera_GPIO-Pad97) -> CAM_GPIO
- Module1 pad 98: unconnected-(Module1A-GND-Pad98) -> GND
- Module1 pad 99: unconnected-(Module1A-Global_EN-Pad99) -> EN_GPIO
Routing:
- net GND: track 140.1 -> 36.0 mm, vias 248 -> 219
- net +3V3: track 83.9 -> 30.5 mm, vias 44 -> 32
- net UART_RX/DIN1: track 66.4 -> 39.3 mm, vias 2 -> 0
- net FMC_A12: track 22.0 -> 0.00 mm, vias 3 -> 0
- net FMC_BA1: track 21.5 -> 0.00 mm, vias 1 -> 0
- net FMC_SDCKE0: track 21.4 -> 0.00 mm, vias 1 -> 0
- net FMC_D2: track 20.9 -> 0.00 mm, vias 1 -> 0
- net FMC_D0: track 20.9 -> 0.00 mm, vias 1 -> 0
- net FMC_D8: track 20.9 -> 0.00 mm, vias 1 -> 0
- net FMC_D4: track 20.8 -> 0.00 mm, vias 1 -> 0
- net FMC_D6: track 20.8 -> 0.00 mm, vias 1 -> 0
- net FMC_NBL0: track 20.8 -> 0.00 mm, vias 1 -> 0
- net FMC_D5: track 20.8 -> 0.00 mm, vias 1 -> 0
- net FMC_D11: track 20.8 -> 0.00 mm, vias 1 -> 0
- net FMC_D7: track 20.7 -> 0.00 mm, vias 1 -> 0
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
Commit message: Adding ICN6211
Parts:
- removed JP1, JP2: JP2-NOCUT, EEZ_DIB_MCU_r3B4:JP2-NOCUT
- added C10: 22nF, Capacitor_SMD:C_0603_1608Metric, F.Cu at (121.4, 77.0)
- added C11: 22nF, Capacitor_SMD:C_0603_1608Metric, F.Cu at (124.4, 77.0)
- added C12: 22nF, Capacitor_SMD:C_0603_1608Metric, F.Cu at (127.5, 77.0)
- added C13: 22nF, Capacitor_SMD:C_0603_1608Metric, F.Cu at (130.6, 77.0)
- added C16: 22nF, Capacitor_SMD:C_0603_1608Metric, F.Cu at (122.9, 77.0)
- added C17: 22nF, Capacitor_SMD:C_0603_1608Metric, F.Cu at (126.0, 77.0)
- added C18: 22nF, Capacitor_SMD:C_0603_1608Metric, F.Cu at (129.0, 77.0)
- added C19: 22nF, Capacitor_SMD:C_0603_1608Metric, F.Cu at (132.1, 77.0)
- added C20: 10nF, Capacitor_SMD:C_0603_1608Metric, F.Cu at (46.4, 88.7)
- added C21: 1uF, Capacitor_SMD:C_0603_1608Metric, F.Cu at (46.4, 91.2)
- added C22: 10nF, Capacitor_SMD:C_0603_1608Metric, F.Cu at (46.4, 93.7)
- added C23: 1uF, Capacitor_SMD:C_0603_1608Metric, F.Cu at (46.4, 96.2)
- added C24: 10nF, Capacitor_SMD:C_0603_1608Metric, F.Cu at (46.4, 99.7)
- added C25: 1uF, Capacitor_SMD:C_0603_1608Metric, F.Cu at (46.4, 101.2)
- added D3: 3.6V, Diode_SMD:D_SOD-323_HandSoldering, F.Cu at (137.0, 79.5)
- added GPDI1: GPDI-D, conn-fci:CONN-10029449-111RLF, F.Cu at (127.8, 70.1)
- added R12: 0, Resistor_SMD:R_0603_1608Metric, F.Cu at (85.1, 69.3)
- added R13: 0, Resistor_SMD:R_0603_1608Metric, F.Cu at (86.6, 69.3)
- added R14: 0, Resistor_SMD:R_0603_1608Metric, F.Cu at (88.1, 69.3)
- added R15: 0, Resistor_SMD:R_0603_1608Metric, F.Cu at (89.7, 69.3)
- added R16: 0, Resistor_SMD:R_0603_1608Metric, F.Cu at (91.2, 69.3)
- added R17: 0, Resistor_SMD:R_0603_1608Metric, F.Cu at (92.7, 69.3)
- added R18: 549, Resistor_SMD:R_0603_1608Metric, F.Cu at (133.6, 77.0)
- added R19: 4.7K, Resistor_SMD:R_0603_1608Metric, F.Cu at (46.4, 103.8)
- added R20: 549, Resistor_SMD:R_0603_1608Metric, F.Cu at (135.1, 77.0)
- added R21: 4.7K, Resistor_SMD:R_0603_1608Metric, F.Cu at (46.4, 106.3)
- added U1: ICN6211, Package_DFN_QFN:QFN-48-1EP_6x6mm_P0.4mm_EP4.2x4.2mm, F.Cu at (73.7, 92.2)
- moved U$5 141.7 mm to (193.2, 150.5)
- moved U$6 141.7 mm to (184.9, 153.9)
- moved U$1 141.7 mm to (194.9, 153.9)
- moved Q2 117.1 mm to (134.9, 105.0)
- moved SP1 113.6 mm to (127.1, 106.1), turned to 90 degrees
- moved C56 112.4 mm to (121.0, 108.2), turned to -90 degrees
- moved R25 111.7 mm to (150.5, 108.6)
- moved IC9 108.2 mm to (141.4, 108.1)
- moved JP6 108.0 mm to (141.3, 104.8)
- moved B1 63.8 mm to (196.3, 102.7)
- moved R10 55.3 mm to (19.8, 163.8), turned to 180 degrees
- moved R6 53.8 mm to (19.8, 161.8), turned to 180 degrees
- moved IC8 53.4 mm to (57.0, 105.5)
- moved C40 53.3 mm to (55.0, 109.1)
- moved C4 50.3 mm to (21.1, 144.8), turned to 180 degrees
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Connections:
- LCD1 pad 13: Net-(LCD1-B0) -> LTDC_G0
- LCD1 pad 14: Net-(LCD1-B0) -> LTDC_G1
- LCD1 pad 21: Net-(LCD1-B0) -> LTDC_B0
- LCD1 pad 22: Net-(LCD1-B0) -> LTDC_B1
- LCD1 pad 23: Net-(LCD1-B0) -> LTDC_B2
- LCD1 pad 5: Net-(LCD1-B0) -> LTDC_R0
- LCD1 pad 6: Net-(LCD1-B0) -> LTDC_R1
- LCD1 pad 7: Net-(LCD1-B0) -> LTDC_R2
- Module1 pad 101: unconnected-(Module1B-USB_OTG_ID-Pad101) -> USB_OTG_FS_ID
- Module1 pad 102: unconnected-(Module1B-PCIe_CLK_nREQ-Pad102) -> PCIe_CLK_nREQ
- Module1 pad 103: unconnected-(Module1B-USB2_N-Pad103) -> USB_OTG_FS_D_N
- Module1 pad 105: unconnected-(Module1B-USB2_P-Pad105) -> USB_OTG_FS_D_P
- Module1 pad 107: unconnected-(Module1B-GND-Pad107) -> GND
- Module1 pad 108: unconnected-(Module1B-GND-Pad108) -> GND
- Module1 pad 109: unconnected-(Module1B-PCIe_nRST-Pad109) -> PCIe_nRST
- Module1 pad 110: unconnected-(Module1B-PCIe_CLK_P-Pad110) -> PCIe_CLK_P
- Module1 pad 111: unconnected-(Module1B-VDAC_COMP-Pad111) -> VDAC_COMP
- Module1 pad 112: unconnected-(Module1B-PCIe_CLK_N-Pad112) -> PCIe_CLK_N
- Module1 pad 113: unconnected-(Module1B-GND-Pad113) -> GND
- Module1 pad 114: unconnected-(Module1B-GND-Pad114) -> GND
- Module1 pad 116: unconnected-(Module1B-PCIe_RX_P-Pad116) -> PCIe_RX_P
- Module1 pad 118: unconnected-(Module1B-PCIe_RX_N-Pad118) -> PCIe_RX_N
- Module1 pad 119: unconnected-(Module1B-GND-Pad119) -> GND
- Module1 pad 120: unconnected-(Module1B-GND-Pad120) -> GND
- Module1 pad 122: unconnected-(Module1B-PCIe_TX_P-Pad122) -> PCIe_TX_P
- Module1 pad 124: unconnected-(Module1B-PCIe_TX_N-Pad124) -> PCIe_TX_N
- Module1 pad 125: unconnected-(Module1B-GND-Pad125) -> GND
- Module1 pad 126: unconnected-(Module1B-GND-Pad126) -> GND
- Module1 pad 128: unconnected-(Module1B-CAM0_D0_N-Pad128) -> CAM0_D0_N
- Module1 pad 130: unconnected-(Module1B-CAM0_D0_P-Pad130) -> CAM0_D0_P
- Module1 pad 131: unconnected-(Module1B-GND-Pad131) -> GND
- Module1 pad 132: unconnected-(Module1B-GND-Pad132) -> GND
- Module1 pad 134: unconnected-(Module1B-CAM0_D1_N-Pad134) -> CAM0_D1_N
- Module1 pad 136: unconnected-(Module1B-CAM0_D1_P-Pad136) -> CAM0_D1_P
- Module1 pad 137: unconnected-(Module1B-GND-Pad137) -> GND
- Module1 pad 138: unconnected-(Module1B-GND-Pad138) -> GND
- Module1 pad 140: unconnected-(Module1B-CAM0_C_N-Pad140) -> CAM0_C_N
- Module1 pad 142: unconnected-(Module1B-CAM0_C_P-Pad142) -> CAM0_C_P
- Module1 pad 144: unconnected-(Module1B-GND-Pad144) -> GND
- Module1 pad 150: unconnected-(Module1B-GND-Pad150) -> GND
- Module1 pad 151: unconnected-(Module1B-HDMI0_CEC-Pad151) -> GPDI0_CEC
- Module1 pad 153: unconnected-(Module1B-HDMI0_HOTPLUG-Pad153) -> GPDI0_HOTPLUG
- Module1 pad 155: unconnected-(Module1B-GND-Pad155) -> GND
- Module1 pad 156: unconnected-(Module1B-GND-Pad156) -> GND
- Module1 pad 157: unconnected-(Module1B-DSI0_D0_N-Pad157) -> DSIHOST_D0N
- Module1 pad 159: unconnected-(Module1B-DSI0_D0_P-Pad159) -> DSIHOST_D0P
- Module1 pad 161: unconnected-(Module1B-GND-Pad161) -> GND
- Module1 pad 162: unconnected-(Module1B-GND-Pad162) -> GND
- Module1 pad 163: unconnected-(Module1B-DSI0_D1_N-Pad163) -> DSIHOST_D1N
- Module1 pad 165: unconnected-(Module1B-DSI0_D1_P-Pad165) -> DSIHOST_D1P
- Module1 pad 167: unconnected-(Module1B-GND-Pad167) -> GND
- Module1 pad 168: unconnected-(Module1B-GND-Pad168) -> GND
- Module1 pad 169: unconnected-(Module1B-DSI0_C_N-Pad169) -> DSIHOST_CKN
- Module1 pad 170: unconnected-(Module1B-HDMI0_TX2_P-Pad170) -> GPDI0_TX2_P
- Module1 pad 171: unconnected-(Module1B-DSI0_C_P-Pad171) -> DSIHOST_CKP
- Module1 pad 172: unconnected-(Module1B-HDMI0_TX2_N-Pad172) -> GPDI0_TX2_N
- Module1 pad 173: unconnected-(Module1B-GND-Pad173) -> GND
- Module1 pad 174: unconnected-(Module1B-GND-Pad174) -> GND
- Module1 pad 176: unconnected-(Module1B-HDMI0_TX1_P-Pad176) -> GPDI0_TX1_P
- Module1 pad 178: unconnected-(Module1B-HDMI0_TX1_N-Pad178) -> GPDI0_TX1_N
- Module1 pad 179: unconnected-(Module1B-GND-Pad179) -> GND
- Module1 pad 180: unconnected-(Module1B-GND-Pad180) -> GND
- Module1 pad 182: unconnected-(Module1B-HDMI0_TX0_P-Pad182) -> GPDI0_TX0_P
- Module1 pad 184: unconnected-(Module1B-HDMI0_TX0_N-Pad184) -> GPDI0_TX0_N
- Module1 pad 185: unconnected-(Module1B-GND-Pad185) -> GND
- Module1 pad 186: unconnected-(Module1B-GND-Pad186) -> GND
- Module1 pad 188: unconnected-(Module1B-HDMI0_CLK_P-Pad188) -> GPDI0_CLK_P
- Module1 pad 190: unconnected-(Module1B-HDMI0_CLK_N-Pad190) -> GPDI0_CLK_N
- Module1 pad 191: unconnected-(Module1B-GND-Pad191) -> GND
- Module1 pad 192: unconnected-(Module1B-GND-Pad192) -> GND
- Module1 pad 197: unconnected-(Module1B-GND-Pad197) -> GND
- Module1 pad 198: unconnected-(Module1B-GND-Pad198) -> GND
- Module1 pad 199: unconnected-(Module1B-HDMI0_SDA-Pad199) -> GPDI0_SDA
- Module1 pad 200: unconnected-(Module1B-HDMI0_SCL-Pad200) -> GPDI0_SCL
- X2 pad 13: Net-(X2M-1) -> I2C1_SCL
- X2 pad 14: Net-(X2N-1) -> I2C1_SDA
Routing:
- net +VAUX: track 112.6 -> 0.00 mm, vias 1 -> 0
- net +5V: track 186.1 -> 289.9 mm, vias 7 -> 13
- net SPI5_CSB: track 0.00 -> 99.9 mm
- net Net-(X2M-1): track 98.8 -> 0.00 mm
- net SPI2_CSB: track 0.00 -> 95.3 mm, vias 0 -> 1
- net SPI4_CLK: track 0.00 -> 94.8 mm, vias 0 -> 1
- net Net-(X2N-1): track 94.0 -> 0.00 mm
- net SPI4_MOSI: track 0.00 -> 93.9 mm, vias 0 -> 1
- net SPI5_IRQ: track 0.00 -> 92.7 mm, vias 0 -> 1
- net SPI5_MISO: track 0.00 -> 92.6 mm
- net SPI2_CSA: track 0.00 -> 92.1 mm, vias 0 -> 1
- net SPI2_MOSI: track 0.00 -> 88.0 mm, vias 0 -> 1
- net SPI2_MISO: track 0.00 -> 86.9 mm, vias 0 -> 1
- net SPI2_CLK: track 0.00 -> 85.3 mm, vias 0 -> 1
- net USER_SW: track 27.4 -> 112.6 mm, vias 0 -> 2
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
Commit message: Moving footprints - change 0804 to 0603
Parts:
- C15, C4, C40, C55, C6, C9: footprint EEZ_DIB_MCU_r3B4:C0603 -> Capacitor_SMD:C_0603_1608Metric
- C2, C3, C5, C51, C53, C7, C8: footprint EEZ_DIB_MCU_r3B4:C0805 -> Capacitor_SMD:C_0603_1608Metric
- C41: moved to B.Cu
- C57: footprint EEZ_DIB_MCU_r3B4:C0603 -> Capacitor_SMD:C_0603_1608Metric; moved to B.Cu
- C58: footprint EEZ_DIB_MCU_r3B4:C0805 -> Capacitor_SMD:C_0603_1608Metric; moved to B.Cu
- R1, R10, R11, R2, R25, R26, R27, R28, R29, R3, R30, R31, R32, R33, R34, R35, R36, R4, R5, R6, R7, R8, R9: footprint EEZ_DIB_MCU_r3B4:R0805 -> Resistor_SMD:R_0603_1608Metric
- R23, R24, R37: footprint EEZ_DIB_MCU_r3B4:R0805 -> Resistor_SMD:R_0603_1608Metric; moved to B.Cu
- moved R32 72.5 mm to (81.4, 80.4)
- moved R33 72.5 mm to (83.3, 80.4)
- moved IC14 71.2 mm to (120.8, 95.6), turned to 0 degrees
- moved C58 67.1 mm to (120.7, 99.6), turned to 180 degrees
- moved C57 64.5 mm to (120.6, 101.7), turned to 180 degrees
- moved R6 63.9 mm to (58.8, 111.2), turned to 90 degrees
- moved R10 62.2 mm to (58.8, 115.3), turned to -90 degrees
- moved JP8 59.8 mm to (42.7, 112.1), turned to -90 degrees
- moved ZD1 59.6 mm to (70.8, 113.9)
- moved R37 54.4 mm to (98.5, 127.5), turned to 0 degrees
- moved JP9 53.6 mm to (98.5, 125.3), turned to 180 degrees
- moved IC3 49.9 mm to (49.2, 113.2)
- moved C6 49.8 mm to (45.4, 108.3), turned to 180 degrees
- moved R9 49.3 mm to (49.8, 108.9), turned to 180 degrees
- moved C4 47.0 mm to (55.3, 112.5), turned to 0 degrees
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Routing:
- net SDMMC1_CMD: track 38.3 -> 35.0 mm, vias 2 -> 1
- net /TFT LCD Audio USB/LCD_DISP: track 11.7 -> 8.37 mm
- net GND: track 56.1 -> 53.3 mm, vias 243 -> 242
- net +3V3: track 39.7 -> 37.8 mm, vias 34 -> 32
- net SDMMC1_CK: track 27.2 -> 25.8 mm

Commit message: Removing non used components in schematic
Parts:
- removed B1: DS1092-10-W6L, EEZ_DIB_MCU_r3B4:DS1092-10-W6L
- removed EEZ_SIGNATURE0: SIGNATURESMALL, EEZ_DIB_MCU_r3B4:SIGNATURE_5MM
- removed JP8: JP3-CUT-0805-ROTATED, EEZ_DIB_MCU_r3B4:JP3-0805-CUT2
- removed U$1: , EEZ_DIB_MCU_r3B4:RECYCLE_BIN1_8
- removed U$3: , EEZ_DIB_MCU_r3B4:CE_5MM
- removed U$5: , EEZ_DIB_MCU_r3B4:PB_SMALL
- removed U$6: , EEZ_DIB_MCU_r3B4:ESD_SYMBOL
- removed X5: LMJTAB881243M-L, EEZ_DIB_MCU_r3B4:RJ45-TRAFO-LED
Routing:
- net Net-(R4-Pad1): track 5.20 -> 0.00 mm
- net Net-(X3B-1): track 4.83 -> 0.00 mm
