File: EEZ_DIB_MCU_r3B4/EEZ_DIB_MCU_r3B4.kicad_pcb (KiCad board)
At the start: 4 copper layers, 139.5 x 70 mm, 113 parts, among them IC1 TPD4E001DRLR, IC11 TPS2051BDBVR, IC12 TPS61169DCKR, IC13 TPD4E001DRLR, IC14 TSC2007IPW, IC2 74AUP1G74DC.125, IC3 CD74HC4050PWR, IC5 LD1117ADT33TR, IC8 AT24C256C-SSHL-B, IC9 N.C., J1 5033981892, J2 67803-8020, Q1 N.C., Q2 2N7002, SW1 TL1100CF160Q, SW2 PEC16-2215F-S0024, U1 ICN6211, X1 DS1024-2*20R0, X2 DS1013-16SSIB1, X3 691322110005

Commit message: Updating 3D models
Parts:
- added J3: HR911130A, HR911130A:HANRUN_HR911130A, F.Cu at (50.3, 73.4)
- R32, R33: moved to B.Cu
- moved R16 41.2 mm to (59.1, 95.1), turned to 180 degrees
- moved R15 39.0 mm to (59.1, 93.6), turned to 180 degrees
- moved R17 38.5 mm to (58.2, 86.5), turned to -90 degrees
- moved R14 36.8 mm to (59.1, 92.0), turned to 180 degrees
- moved C23 34.2 mm to (80.5, 96.2), turned to 90 degrees
- moved R12 33.5 mm to (59.1, 90.5), turned to 180 degrees
- moved C22 32.8 mm to (79.0, 96.2), turned to 90 degrees
- moved R13 31.8 mm to (59.8, 86.5), turned to -90 degrees
- moved C20 26.4 mm to (72.6, 86.5), turned to -90 degrees
- moved C21 25.2 mm to (71.1, 86.5), turned to -90 degrees
- moved IC14 23.6 mm to (109.5, 116.2)
- moved C58 23.1 mm to (104.0, 115.5), turned to -90 degrees
- moved C57 15.6 mm to (109.3, 112.5)
- moved R10 15.1 mm to (46.3, 106.8), turned to 90 degrees
- moved C25 13.9 mm to (60.2, 101.5), turned to 90 degrees
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Connections:
- C1 pad 1: +3V3 -> CM4_3.3V
- C40 pad 2: +3V3 -> CM4_3.3V
- C41 pad 1: +3V3 -> CM4_3.3V
- C53 pad 1: +3V3 -> CM4_3.3V
- C56 pad 2: +3V3 -> CM4_3.3V
- C57 pad 2: +3V3 -> CM4_3.3V
- C58 pad 2: +3V3 -> CM4_3.3V
- C6 pad 1: +3V3 -> CM4_3.3V
- C9 pad 1: +3V3 -> CM4_3.3V
- IC14 pad 1: +3V3 -> CM4_3.3V
- IC2 pad 2: +3V3 -> CM4_3.3V
- IC2 pad 6: +3V3 -> CM4_3.3V
- IC2 pad 7: +3V3 -> CM4_3.3V
- IC2 pad 8: +3V3 -> CM4_3.3V
- IC3 pad 1: +3V3 -> CM4_3.3V
- IC5 pad 4: +3V3 -> CM4_3.3V
- IC8 pad 8: +3V3 -> CM4_3.3V
- IC9 pad 5: +3V3 -> CM4_3.3V
- J1 pad 4: +3V3 -> CM4_3.3V
- JP6 pad NC: +3V3 -> CM4_3.3V
- LCD1 pad 4: +3V3 -> CM4_3.3V
- LED1 pad A: +3V3 -> CM4_3.3V
- R1 pad 1: +3V3 -> CM4_3.3V
- R23 pad 1: +3V3 -> CM4_3.3V
- R24 pad 1: +3V3 -> CM4_3.3V
- R3 pad 1: +3V3 -> CM4_3.3V
- R37 pad 2: +3V3 -> CM4_3.3V
- R7 pad 1: +3V3 -> CM4_3.3V
- SP1 pad +: +3V3 -> CM4_3.3V
- SP1 pad +B: +3V3 -> CM4_3.3V
- X1 pad 7: +3V3 -> CM4_3.3V
- X2 pad 16: +3V3 -> CM4_3.3V
Routing:
- net ~{FAULT}: track 0.00 -> 158.7 mm, vias 0 -> 1
- net OE_SYNC: track 0.00 -> 126.2 mm, vias 0 -> 1
- net GPDI0_HOTPLUG: track 2.04 -> 55.8 mm
- net GPDI0_CEC: track 0.00 -> 53.5 mm
- net CM4_3.3V: track 2.00 -> 54.7 mm, vias 3 -> 50
- net GND: track 53.3 -> 104.1 mm, vias 242 -> 306
- net USB_OTG_FS_ID: track 19.7 -> 67.5 mm, vias 1 -> 2
- net /TFT LCD Audio USB/USB_D_P: track 18.6 -> 58.4 mm
- net CAM0_C_N: track 0.00 -> 39.6 mm
- net /TFT LCD Audio USB/USB_D_N: track 19.6 -> 59.1 mm
- net CAM0_C_P: track 0.00 -> 39.4 mm
- net CAM0_D1_P: track 0.00 -> 37.9 mm
- net +3V3: track 37.8 -> 0.00 mm, vias 32 -> 0
- net CAM0_D1_N: track 0.00 -> 36.8 mm
- net CAM0_D0_N: track 0.00 -> 35.0 mm
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- added copper zone on B.Cu, net CM4_3.3V
- added copper zone on F.Cu, net CM4_3.3V
- added copper zone on In2.Cu, net CM4_3.3V
- removed copper zone on B.Cu, net +3V3
- removed copper zone on F.Cu, net +3V3
- removed copper zone on In2.Cu, net +3V3

Commit message: Adding connections to Ethernet connector
Connections:
- J3 pad 1: unconnected-(J3-P1-Pad1) -> Net-(J3-P1)
- J3 pad 10: unconnected-(J3-P10-Pad10) -> Net-(J3-P10)
- J3 pad 11: unconnected-(J3-Pad11) -> Net-(J3-Pad11)
- J3 pad 12: unconnected-(J3-Pad12) -> GND
- J3 pad 13: unconnected-(J3-Pad13) -> GND
- J3 pad 14: unconnected-(J3-Pad14) -> Net-(J3-Pad14)
- J3 pad 2: unconnected-(J3-P2-Pad2) -> /CM4_IO_slow/eth_0p
- J3 pad 3: unconnected-(J3-P3-Pad3) -> /CM4_IO_slow/eth_0n
- J3 pad 4: unconnected-(J3-P4-Pad4) -> /CM4_IO_slow/eth_1p
- J3 pad 5: unconnected-(J3-P5-Pad5) -> /CM4_IO_slow/eth_2p
- J3 pad 6: unconnected-(J3-P6-Pad6) -> /CM4_IO_slow/eth_2n
- J3 pad 7: unconnected-(J3-P7-Pad7) -> /CM4_IO_slow/eth_1n
- J3 pad 8: unconnected-(J3-P8-Pad8) -> /CM4_IO_slow/eth_3p
- J3 pad 9: unconnected-(J3-P9-Pad9) -> /CM4_IO_slow/eth_3n
- J3 pad S1: Net-(J3-SHIELD-PadS1) -> GND
- J3 pad S2: Net-(J3-SHIELD-PadS1) -> GND
- Module1 pad 10: unconnected-(Module1A-Ethernet_Pair0_N-Pad10) -> /CM4_IO_slow/eth_0n
- Module1 pad 11: unconnected-(Module1A-Ethernet_Pair2_P-Pad11) -> /CM4_IO_slow/eth_2n
- Module1 pad 12: unconnected-(Module1A-Ethernet_Pair0_P-Pad12) -> /CM4_IO_slow/eth_0p
- Module1 pad 15: unconnected-(Module1A-Ethernet_nLED3(3.3v)-Pad15) -> /CM4_IO_slow/eth_led3
- Module1 pad 17: unconnected-(Module1A-Ethernet_nLED2(3.3v)-Pad17) -> /CM4_IO_slow/eth_led2
- Module1 pad 19: unconnected-(Module1A-Ethernet_nLED1(3.3v)-Pad19) -> /CM4_IO_slow/eth_led1
- Module1 pad 3: unconnected-(Module1A-Ethernet_Pair3_P-Pad3) -> /CM4_IO_slow/eth_3p
- Module1 pad 4: unconnected-(Module1A-Ethernet_Pair1_P-Pad4) -> /CM4_IO_slow/eth_1p
- Module1 pad 5: unconnected-(Module1A-Ethernet_Pair3_N-Pad5) -> /CM4_IO_slow/eth_3n
- Module1 pad 6: unconnected-(Module1A-Ethernet_Pair1_N-Pad6) -> /CM4_IO_slow/eth_1n
- Module1 pad 9: unconnected-(Module1A-Ethernet_Pair2_N-Pad9) -> /CM4_IO_slow/eth_2p

Commit message: Adding DSI connector
Parts:
- added C26: C_Small, Capacitor_SMD:C_0603_1608Metric, F.Cu at (53.0, 56.8)
- added J4: Conn_01x22_Socket, Connector_FFC-FPC:Hirose_FH12-22S-0.5SH_1x22-1MP_P0.50mm_Horizontal, F.Cu at (44.1, 135.8)
- added R22: R_Small, Resistor_SMD:R_0603_1608Metric, F.Cu at (50.5, 56.8)
- added R38: R_Small, Resistor_SMD:R_0603_1608Metric, F.Cu at (48.0, 56.8)
- added R39: R_Small, Resistor_SMD:R_0603_1608Metric, F.Cu at (45.5, 56.8)
- moved R10 15.4 mm to (61.7, 105.3), turned to 0 degrees
- moved R9 14.9 mm to (54.5, 102.5), turned to 0 degrees
- moved IC8 14.4 mm to (43.4, 87.5)
- moved IC3 8.91 mm to (57.3, 109.5), turned to -90 degrees
- moved C40 5.02 mm to (52.5, 104.0)
- moved C6 3.77 mm to (52.3, 106.9)

Commit message: More routing
Parts:
- R38, R39: moved to B.Cu
- moved R22 21.2 mm to (45.2, 77.3), turned to 90 degrees
- moved C26 20.5 mm to (54.9, 77.2)
- moved IC3 18.1 mm to (44.5, 96.7)
- moved R9 18.0 mm to (58.4, 120.1), turned to 90 degrees
- moved R38 17.4 mm to (53.0, 73.4)
- moved IC5 16.8 mm to (34.6, 111.0), turned to 90 degrees
- moved R39 16.8 mm to (47.9, 73.4)
- moved C40 15.9 mm to (44.0, 90.6), turned to -90 degrees
- moved R10 14.4 mm to (50.5, 96.2)
- moved C6 11.6 mm to (59.2, 116.3), turned to 90 degrees
- moved J4 11.5 mm to (44.2, 124.3)
- moved R6 10.8 mm to (50.5, 97.7)
- moved C15 9.95 mm to (43.2, 106.7)
- moved C14 8.21 mm to (44.4, 111.3), turned to -90 degrees
- moved C25 5.95 mm to (60.1, 107.4), turned to 0 degrees
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Routing:
- net CM4_3.3V: track 54.7 -> 159.7 mm, vias 50 -> 57
- net I2C1_SCL: track 100.3 -> 151.3 mm, vias 3 -> 4
- net DSIHOST_D1P: track 31.2 -> 79.5 mm, vias 2 -> 3
- net DSIHOST_D1N: track 31.2 -> 79.5 mm, vias 2 -> 3
- net DSIHOST_CKN: track 33.0 -> 80.8 mm, vias 2 -> 3
- net DSIHOST_D0P: track 30.2 -> 78.0 mm, vias 2 -> 3
- net DSIHOST_D0N: track 30.2 -> 78.0 mm, vias 2 -> 3
- net DSIHOST_CKP: track 33.0 -> 80.5 mm, vias 2 -> 3
- net I2C1_SDA: track 94.3 -> 140.4 mm
- net Net-(IC3G-I): track 0.00 -> 32.7 mm, vias 0 -> 2
- net PWR_SSTART: track 0.00 -> 30.5 mm
- net Net-(IC1-IO4): track 23.5 -> 53.5 mm, vias 0 -> 2
- net Net-(IC1-IO3): track 18.7 -> 48.1 mm, vias 0 -> 2
- net PWR_DIRECT: track 0.00 -> 27.5 mm
- net Net-(IC3E-I): track 0.00 -> 24.9 mm
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
Commit message: Routing
Connections:
- net /CM4_IO_slow/eth_0n renamed /CM4_IO_slow/ETH_0N
- net /CM4_IO_slow/eth_0p renamed /CM4_IO_slow/ETH_0P
- net /CM4_IO_slow/eth_1n renamed /CM4_IO_slow/ETH_1N
- net /CM4_IO_slow/eth_1p renamed /CM4_IO_slow/ETH_1P
- net /CM4_IO_slow/eth_2n renamed /CM4_IO_slow/ETH_2N
- net /CM4_IO_slow/eth_2p renamed /CM4_IO_slow/ETH_2P
- net /CM4_IO_slow/eth_3n renamed /CM4_IO_slow/ETH_3N
- net /CM4_IO_slow/eth_3p renamed /CM4_IO_slow/ETH_3P
Routing:
- net /CM4_IO_slow/ETH_2P: track 0.00 -> 64.5 mm, vias 0 -> 3
- net /CM4_IO_slow/ETH_1N: track 0.00 -> 61.0 mm, vias 0 -> 3
- net /CM4_IO_slow/ETH_3P: track 0.00 -> 58.5 mm, vias 0 -> 3
- net /CM4_IO_slow/ETH_3N: track 0.00 -> 57.2 mm, vias 0 -> 3
- net /CM4_IO_slow/ETH_2N: track 0.00 -> 57.1 mm, vias 0 -> 3
- net /CM4_IO_slow/ETH_1P: track 0.00 -> 50.4 mm, vias 0 -> 3
- net /CM4_IO_slow/ETH_0P: track 0.00 -> 50.1 mm, vias 0 -> 3
- net /CM4_IO_slow/ETH_0N: track 0.00 -> 47.9 mm, vias 0 -> 3
- net DSIHOST_CKP: track 80.5 -> 127.7 mm
- net DSIHOST_CKN: track 80.8 -> 126.6 mm
- net DSIHOST_D1P: track 79.5 -> 121.6 mm, vias 3 -> 4
- net DSIHOST_D1N: track 79.5 -> 120.5 mm, vias 3 -> 4
- net DSIHOST_D0P: track 78.0 -> 116.6 mm
- net DSIHOST_D0N: track 78.0 -> 115.5 mm
- net LTDC_DE: track 68.4 -> 70.7 mm, vias 2 -> 4
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
Commit message: Routing almost finished
Parts:
- moved C24 1.08 mm to (59.1, 105.6)
- moved C25 1.08 mm to (59.1, 107.2)
Routing:
- net UART_TX/DOUT1: track 6.55 -> 147.0 mm, vias 1 -> 7
- net I2C1_SCL: track 151.3 -> 257.7 mm, vias 4 -> 10
- net I2C1_SDA: track 140.4 -> 237.0 mm, vias 3 -> 9
- net +5V: track 313.5 -> 405.4 mm, vias 18 -> 21
- net /CM4_IO_slow/eth_led1: track 0.00 -> 76.5 mm, vias 0 -> 5
- net /CM4_IO_slow/eth_led2: track 0.00 -> 74.1 mm, vias 0 -> 5
- net DOUT2: track 6.63 -> 70.8 mm, vias 1 -> 6
- net UART_RX/DIN1: track 94.0 -> 154.5 mm, vias 0 -> 4
- net TFT_BRIGHTNESS: track 0.00 -> 54.9 mm, vias 0 -> 2
- net DIN2: track 0.81 -> 49.0 mm, vias 1 -> 4
- net IRQ_TOUCH: track 0.00 -> 40.1 mm, vias 0 -> 3
- net RTC_REF: track 0.00 -> 40.0 mm, vias 0 -> 2
- net ENC_B: track 28.4 -> 53.5 mm, vias 1 -> 4
- net ENC_A: track 18.6 -> 43.5 mm, vias 1 -> 4
- net BOOT0: track 28.1 -> 52.7 mm, vias 1 -> 3
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
Commit message: Routing
Connections:
- Module1 pad 61: SDMMC1_D0 -> unconnected-(Module1A-SD_DAT3-Pad61)
Routing:
- net SDMMC1_D0: track 37.4 -> 38.2 mm
Changed lines of the file:
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@@
   (net 254 "unconnected-(J4-Pin_11-Pad11)")
   (net 255 "unconnected-(J4-Pin_12-Pad12)")
+  (net 256 "unconnected-(Module1A-SD_DAT3-Pad61)")
   (footprint "Resistor_SMD:R_0603_1608Metric" (layer "F.Cu")
     (at 127.4552 114.707 -90)
@@
     (pad "4" smd roundrect (at 0 -2.38 90) (size 5.8 6.2) (layers "F.Cu" "F.Paste" "F.Mask") (roundrect_rratio 0.00875862069)
       (net 117 "CM4_3.3V") (pinfunction "OUT") (pintype "passive") (solder_mask_margin 0.0635))
+    (model ":KICAD7_3DMODEL_DIR:Package_TO_SOT_SMD.3dshapes/TO-252-2.wrl"
+      (offset (xyz 0 0 0))
+      (scale (xyz 1 1 1))
+      (rotate (xyz 0 0 -90))
+    )
   )
   (footprint "EEZ_DIB_MCU_r3B4:DO214AA" (layer "F.Cu")
@@
       (net 1 "GND") (pinfunction "GND") (pintype "power_in"))
     (pad "61" smd rect (at -2 -19.3) (size 0.2 0.7) (layers "F.Cu" "F.Paste" "F.Mask")
-      (net 22 "SDMMC1_D0") (pinfunction "SD_DAT3") (pintype "passive"))
+      (net 256 "unconnected-(Module1A-SD_DAT3-Pad61)") (pinfunction "SD_DAT3") (pintype "passive+no_connect"))
     (pad "62" smd rect (at 1.08 -19.3) (size 0.2 0.7) (layers "F.Cu" "F.Paste" "F.Mask")
       (net 27 "SDMMC1_CMD") (pinfunction "SD_CMD") (pintype "passive"))
@@
     (pad "2" smd roundrect (at 1.9812 0 270) (size 2.8702 0.762) (layers "F.Cu" "F.Paste" "F.Mask") (roundrect_rratio 0.06666666667)
       (net 1 "GND") (pinfunction "-") (pintype "passive") (solder_mask_margin 0.0635))
+    (model ":KICAD7_3DMODEL_DIR:Capacitor_SMD.3dshapes/CP_Elec_5x4.4.step"
+      (offset (xyz 0 0 0))
+      (scale (xyz 1 1 1))
+      (rotate (xyz 0 0 0))
+    )
   )
   (footprint "EEZ_DIB_MCU_r3B4:EC1206" (layer "F.Cu")
@@
       (chamfer_ratio 0.2928932188) (chamfer top_left top_right bottom_left bottom_right)
       (net 51 "Net-(IC1-IO4)") (pinfunction "1") (pintype "passive") (solder_mask_margin 0.0635))
+    (model "${KIPRJMOD}/footprints/3D/138370836-659-691322110005/691322110005.stp"
+      (offset (xyz 0 -3.5 3.5))
+      (scale (xyz 1 1 1))
+      (rotate (xyz -90 0 0))
+    )
   )
   (footprint "EEZ_DIB_MCU_r3B4:DBV5" (layer "F.Cu")
@@
     (pad "2" smd roundrect (at 1.9812 0 180) (size 2.8702 0.762) (layers "F.Cu" "F.Paste" "F.Mask") (roundrect_rratio 0.06666666667)
       (net 1 "GND") (pinfunction "-") (pintype "passive") (solder_mask_margin 0.0635))
+    (model ":KICAD7_3DMODEL_DIR:Capacitor_SMD.3dshapes/CP_Elec_5x4.4.step"
+      (offset (xyz 0 0 0))
+      (scale (xyz 1 1 1))
+      (rotate (xyz 0 0 0))
+    )
   )
   (footprint "EEZ_DIB_MCU_r3B4:SOT23-BEC" (layer "F.Cu")
@@
     (pad "MP" smd rect (at -7.15 1.4) (size 1.8 2.2) (layers "F.Cu" "F.Paste" "F.Mask"))
     (pad "MP" smd rect (at 7.15 1.4) (size 1.8 2.2) (layers "F.Cu" "F.Paste" "F.Mask"))
-    (model "${KICAD6_3DMODEL_DIR}/Connector_FFC-FPC.3dshapes/Hirose_FH12-22S-0.5SH_1x22-1MP_P0.50mm_Horizontal.wrl"
+    (model "${KICAD7_3DMODEL_DIR}/Connector_FFC-FPC.3dshapes/Hirose_FH12-22S-0.5SH_1x22-1MP_P0.50mm_Horizontal.wrl"
       (offset (xyz 0 0 0))
       (scale (xyz 1 1 1))
       (rotate (xyz 0 0 0))
     )
+    (model ":KICAD7_3DMODEL_DIR:Connector_FFC-FPC.3dshapes/TE_2-84953-2_1x22-1MP_P1.0mm_Horizontal.wrl"
+      (offset (xyz 0 -0.5 0))
+      (scale (xyz 0.5 0.9 0.5))
+      (rotate (xyz 0 0 0))
+    )
   )
   (footprint "EEZ_DIB_MCU_r3B4:FPC_40" (layer "F.Cu")
@@
   (segment (start 105.1 104.34) (end 112.583333 111.823333) (width 0.127) (layer "B.Cu") (net 21))
   (segment (start 96.96 104.35) (end 98.54 104.35) (width 0.127) (layer "B.Cu") (net 21))
-  (segment (start 94.4 110.4) (end 94.42 110.42) (width 0.127) (layer "F.Cu") (net 22))
+  (segment (start 94.42 110.42) (end 94.4 110.4) (width 0.127) (layer "F.Cu") (net 22))
+  (segment (start 94.4 110.4) (end 94.4 109.66) (width 0.127) (layer "F.Cu") (net 22))
   (segment (start 89.77 126.11) (end 92.18 128.52) (width 0.127) (layer "F.Cu") (net 22))
   (segment (start 80.04 126.11) (end 89.77 126.11) (width 0.127) (layer "F.Cu") (net 22))
