File: EEZ_DIB_MCU_r3B4/EEZ_DIB_MCU_r3B4.kicad_pcb (KiCad board)
At the start: 4 copper layers, 139.5 x 70 mm, 119 parts, among them IC1 TPD4E001DRLR, IC11 TPS2051BDBVR, IC12 TPS61169DCKR, IC13 TPD4E001DRLR, IC14 TSC2007IPW, IC2 74AUP1G74DC.125, IC3 CD74HC4050PWR, IC5 LD1117ADT33TR, IC8 AT24C256C-SSHL-B, IC9 N.C., J1 5033981892, J2 67803-8020, J3 HR911130A, J4 Conn_01x22_Socket, Q1 N.C., Q2 2N7002, SW1 TL1100CF160Q, SW2 PEC16-2215F-S0024, U1 ICN6211, X1 DS1024-2*20R0, X2 DS1013-16SSIB1, X3 691322110005

Commit message: Update pictures and 3D models
Parts:
- removed LABEL1: HR000002, EEZ_DIB_MCU_r3B4:CERT-SMALL-SILK
- added REF**: OSHW-Logo_5.7x6mm_SilkScreen, Symbol:OSHW-Logo_5.7x6mm_SilkScreen, F.Cu at (99.3, 67.4)
- added REF**: KiCad-Logo2_5mm_SilkScreen, Symbol:KiCad-Logo2_5mm_SilkScreen, F.Cu at (145.5, 76.3)
Other:
- board text added: "Buzzer"
- board text added: "CM4 compatible"
- board text added: "DSI"
- board text added: "DSI to RGB"
- board text added: "EEZ BB3 CM4 (6/2023 r0A1) Project source code: https://github.com/intergalaktik/bb3-cm4"
- board text removed: "1 Vdd target 2 SWCLK 3 Gnd 4 SWDIO 5 ~RESET~ 6 SWO"
- board text removed: "EEZ DIB MCU (10/2021 r3B4)"
- board text removed: "EEZ DIB MCU (10/2021 r3B4) Project source code: github.com/eez-open/modular-psu"

Commit message: Adding temperary PCIe connector - adding logos
Parts:
- added C27: 4u7, EEZ_DIB_MCU_r3B4:EC1206, F.Cu at (43.5, 116.3)
- added F1: 500mA, Fuse:Fuse_0805_2012Metric, F.Cu at (51.6, 119.2)
- added G***: LOGO, intergalaktik:intergalaktik, F.Cu at (125.5, 95.0)
- added G***: LOGO, nlnet:nlnet, F.Cu at (121.7, 98.6)
- added IC4: TPS2051BDBVR, EEZ_DIB_MCU_r3B4:DBV5, F.Cu at (49.1, 115.3)
- added J5: USB1086-GF-B_REVA, USB1086-GF-B_REVA:GCT_USB1086-GF-B_REVA, F.Cu at (144.2, 80.7)
- added J6: 1586041-6, 1586041-6:TE_1586041-6, F.Cu at (140.5, 70.0)
- added R40: 0R, Resistor_SMD:R_0603_1608Metric, F.Cu at (49.1, 112.3)
- added R41: 10K, Resistor_SMD:R_0603_1608Metric, F.Cu at (47.6, 118.5)
- added R42: 0, Resistor_SMD:R_0603_1608Metric, F.Cu at (136.7, 75.2)
- added radiona: radiona, radiona:radiona, F.Cu at (125.7, 90.2)
- C1: footprint EEZ_DIB_MCU_r3B4:PANASONIC_C -> Fuse:Fuse_0805_2012Metric
- C26, R22: moved to B.Cu
- moved FM4 33.1 mm to (111.3, 65.5)
- moved FM8 33.1 mm to (111.3, 65.5)
- moved REF** 22.1 mm to (125.0, 84.6)
- moved R17 8.12 mm to (59.1, 94.6), turned to 180 degrees
- moved REF** 6.66 mm to (105.9, 67.6)
- moved D3 3.59 mm to (135.1, 76.5), turned to 90 degrees
- moved R12 3.53 mm to (59.1, 87.0)
- moved R13 2.09 mm to (59.1, 88.5), turned to 180 degrees
- moved R16 2.06 mm to (59.1, 93.1)
- moved R15 2.05 mm to (59.1, 91.5)
- moved R14 2.02 mm to (59.1, 90.0)
- moved C10 1.81 mm to (119.5, 77.0)
- moved C16 1.78 mm to (121.1, 77.0)
- moved C17 1.78 mm to (124.2, 77.0)
- moved C12 1.77 mm to (125.7, 77.0)
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Connections:
- IC3 pad 10: Net-(IC1-IO4) -> Net-(IC3B-O)
- IC3 pad 6: Net-(IC1-IO4) -> Net-(IC3B-O)
Routing:
- net PCIe_CLK_P: track 0.00 -> 74.1 mm, vias 0 -> 2
- net PCIe_CLK_N: track 0.00 -> 73.0 mm, vias 0 -> 1
- net PCIe_TX_P: track 0.00 -> 71.9 mm, vias 0 -> 2
- net PCIe_TX_N: track 0.00 -> 71.5 mm, vias 0 -> 1
- net PCIe_RX_P: track 0.00 -> 67.6 mm, vias 0 -> 1
- net PCIe_RX_N: track 0.00 -> 67.2 mm, vias 0 -> 1
- net PCIe_CLK_nREQ: track 0.00 -> 44.4 mm, vias 0 -> 1
- net ~{FAULT}: track 181.4 -> 159.2 mm, vias 3 -> 1
- net Net-(J5-SHIELD-PadS1): track 0.00 -> 22.0 mm
- net GND: track 131.6 -> 153.2 mm, vias 323 -> 326
- net Net-(IC3B-O): track 0.00 -> 21.0 mm
- net PCIe_nRST: track 0.00 -> 21.0 mm, vias 0 -> 1
- net +5V: track 405.4 -> 426.2 mm
- net Net-(IC1-IO4): track 53.5 -> 35.3 mm, vias 2 -> 3
- net DOUT2: track 70.8 -> 88.8 mm, vias 6 -> 10
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Other:
- board text added: "BB3 CM4 v001"
- board text added: "PCIe"

Commit message: Adding missing 3D models, refreshing pictures
Parts:
- added G***: LOGO, EEZ:eez, F.Cu at (137.9, 90.9)
Routing:
- net PCIe_nRST: track 21.0 -> 70.0 mm, vias 1 -> 2
- net PCIe_TX_N: track 71.5 -> 70.6 mm
- net PCIe_TX_P: track 71.9 -> 71.0 mm
