File: EEZ_DIB_MCU_r3B4/EEZ_DIB_MCU_r3B4.kicad_sch (KiCad schematic)
At the start: 0 parts

Commit message: Switching MCU to KiCad 7 - moving MCU and SDRAM from board
Other:
- sheet SDRAM JTAG SD card EEPROM renamed SDRAM
- removed sheet BP3C
- added sheet EEPROM (eeprom.kicad_sch)
- added sheet PSU (PSU.kicad_sch)
- added sheet SD (SD.kicad_sch)
- added sheet WatchDog (WatchDog.kicad_sch)
- sheet SDRAM: file SDRAM_JTAG_SD_card_EEPROM.kicad_sch -> SDRAM.kicad_sch

Commit message: Adding connectors, grouping parts, removing most of the routing
Other:
- added sheet CM4_IO_fast (cm4_io_fast.kicad_sch)
- added sheet CM4_IO_slow (cm4_io_slow.kicad_sch)
- added sheet CM4_SOM_Connectors (cm4_SoM_connectors.kicad_sch)
Changed lines of the file:
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@@
+    )
+  )
+  (sheet (at 67.31 78.74) (size 45.72 19.05) (fields_autoplaced)
+    (stroke (width 0.1524) (type solid))
+    (fill (color 0 0 0 0.0000))
+    (property "Sheetname" "CM4_IO_slow" (at 67.31 78.0284 0)
+      (effects (font (size 1.27 1.27)) (justify left bottom))
+    )
+    (property "Sheetfile" "cm4_io_slow.kicad_sch" (at 67.31 98.3746 0)
+      (effects (font (size 1.27 1.27)) (justify left top))
+    )
+    (instances
+      (project "EEZ_DIB_MCU_r3B4"
+        (path "/58be380a-4a3a-4b30-b3f5-a03bc3bf2660" (page "12"))
+      )
     )
   )
@@
       (project "EEZ_DIB_MCU_r3B4"
         (path "/58be380a-4a3a-4b30-b3f5-a03bc3bf2660" (page "5"))
+      )
+    )
+  )
+  (sheet (at 153.67 81.28) (size 39.37 16.51) (fields_autoplaced)
+    (stroke (width 0.1524) (type solid))
+    (fill (color 0 0 0 0.0000))
+    (property "Sheetname" "CM4_SOM_Connectors" (at 153.67 80.5684 0)
+      (effects (font (size 1.27 1.27)) (justify left bottom))
+    )
+    (property "Sheetfile" "cm4_SoM_connectors.kicad_sch" (at 153.67 98.3746 0)
+      (effects (font (size 1.27 1.27)) (justify left top))
+    )
+    (instances
+      (project "EEZ_DIB_MCU_r3B4"
+        (path "/58be380a-4a3a-4b30-b3f5-a03bc3bf2660" (page "11"))
       )
     )
@@
       )
     )
+  )
+  (sheet (at 66.04 45.72) (size 46.99 20.32) (fields_autoplaced)
+    (stroke (width 0.1524) (type solid))
+    (fill (color 0 0 0 0.0000))
+    (property "Sheetname" "CM4_IO_fast" (at 66.04 45.0084 0)
+      (effects (font (size 1.27 1.27)) (justify left bottom))
+    )
+    (property "Sheetfile" "cm4_io_fast.kicad_sch" (at 66.04 66.6246 0)
+      (effects (font (size 1.27 1.27)) (justify left top))
+    )
+    (instances
+      (project "EEZ_DIB_MCU_r3B4"
+        (path "/58be380a-4a3a-4b30-b3f5-a03bc3bf2660" (page "13"))
+      )
+    )

Commit message: Splitting SoM and MCU board
Other:
- removed sheet CM4_SOM_Connectors
- removed sheet Ethernet PHY
- removed sheet SDRAM
- removed sheet STM32F7 MCU
Changed lines of the file:
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@@
-    )
-  )
-  (sheet (at 80.01 144.78) (size 12.7 3.81) (fields_autoplaced)
-    (stroke (width 0) (type solid))
-    (fill (color 0 0 0 0.0000))
-    (property "Sheetname" "STM32F7 MCU" (at 80.01 144.0684 0)
-      (effects (font (size 1.27 1.27)) (justify left bottom))
-    )
-    (property "Sheetfile" "STM32F7_MCU.kicad_sch" (at 80.01 149.1746 0)
-      (effects (font (size 1.27 1.27)) (justify left top))
-    )
-    (instances
-      (project "EEZ_DIB_MCU_r3B4"
-        (path "/58be380a-4a3a-4b30-b3f5-a03bc3bf2660" (page "3"))
-      )
     )
   )
@@
       (project "EEZ_DIB_MCU_r3B4"
         (path "/58be380a-4a3a-4b30-b3f5-a03bc3bf2660" (page "5"))
-      )
-    )
-  )
-  (sheet (at 153.67 81.28) (size 39.37 16.51) (fields_autoplaced)
-    (stroke (width 0.1524) (type solid))
-    (fill (color 0 0 0 0.0000))
-    (property "Sheetname" "CM4_SOM_Connectors" (at 153.67 80.5684 0)
-      (effects (font (size 1.27 1.27)) (justify left bottom))
-    )
-    (property "Sheetfile" "cm4_SoM_connectors.kicad_sch" (at 153.67 98.3746 0)
-      (effects (font (size 1.27 1.27)) (justify left top))
-    )
-    (instances
-      (project "EEZ_DIB_MCU_r3B4"
-        (path "/58be380a-4a3a-4b30-b3f5-a03bc3bf2660" (page "11"))
       )
     )
@@
       )
     )
-  )
-  (sheet (at 130.81 144.78) (size 12.7 3.81) (fields_autoplaced)
-    (stroke (width 0) (type solid))
-    (fill (color 0 0 0 0.0000))
-    (property "Sheetname" "SDRAM" (at 130.81 144.0684 0)
-      (effects (font (size 1.27 1.27)) (justify left bottom))
-    )
-    (property "Sheetfile" "SDRAM.kicad_sch" (at 130.81 149.1746 0)
-      (effects (font (size 1.27 1.27)) (justify left top))
-    )
-    (instances
-      (project "EEZ_DIB_MCU_r3B4"
-        (path "/58be380a-4a3a-4b30-b3f5-a03bc3bf2660" (page "4"))
-      )
-    )
-  )
-  (sheet (at 232.41 144.78) (size 12.7 3.81) (fields_autoplaced)
-    (stroke (width 0) (type solid))
-    (fill (color 0 0 0 0.0000))
-    (property "Sheetname" "Ethernet PHY" (at 232.41 144.0684 0)
-      (effects (font (size 1.27 1.27)) (justify left bottom))
-    )
-    (property "Sheetfile" "Ethernet_PHY.kicad_sch" (at 232.41 149.1746 0)
-      (effects (font (size 1.27 1.27)) (justify left top))
-    )
-    (instances
-      (project "EEZ_DIB_MCU_r3B4"
-        (path "/58be380a-4a3a-4b30-b3f5-a03bc3bf2660" (page "6"))
-      )
-    )

Commit message: Updating 3D models
Changed lines of the file:
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@@
 (kicad_sch (version 20230121) (generator eeschema)
   (paper "A4")
+  (wire (pts (xy 143.51 71.12) (xy 143.51 76.2))
+    (stroke (width 0) (type default))
+  )
+  (global_label "CM4_3.3V" (shape input) (at 143.51 76.2 270) (fields_autoplaced)
+    (effects (font (size 1.27 1.27)) (justify right))
+    (property "Intersheetrefs" "${INTERSHEET_REFS}" (at 143.51 88.1167 90)
+      (effects (font (size 1.27 1.27)) (justify right) hide)
+    )
+  )
+  (symbol (lib_id "EEZ_DIB_MCU_r3B4-eagle-import:+3V3") (at 143.51 68.58 0) (mirror y) (unit 1)
+    (in_bom yes) (on_board yes) (dnp no)
+    (property "Reference" "#+3V01" (at 143.51 68.58 0)
+      (effects (font (size 1.27 1.27)) hide)
+    )
+    (property "Value" "+3V3" (at 140.97 69.215 90)
+      (effects (font (size 1.778 1.5113)) (justify left bottom))
+    )
+    (property "Footprint" "EEZ_DIB_MCU_r3B4:" (at 143.51 68.58 0)
+      (effects (font (size 1.27 1.27)) hide)
+    )
+    (property "Datasheet" "" (at 143.51 68.58 0)
+      (effects (font (size 1.27 1.27)) hide)
+    )
+    (pin "1")
+    (instances
+      (project "EEZ_DIB_MCU_r3B4"
+        (path "/58be380a-4a3a-4b30-b3f5-a03bc3bf2660/b81c6957-169a-4ded-90bd-8546b86f332e"
+          (reference "#+3V01") (unit 1)
+        )
+        (path "/58be380a-4a3a-4b30-b3f5-a03bc3bf2660"
+          (reference "#+3V01") (unit 1)
+        )
+      )
+    )
+  )
   (sheet (at 106.68 163.83) (size 20.32 6.35) (fields_autoplaced)
     (stroke (width 0.1524) (type solid))
@@
     )
   )
-  (sheet (at 181.61 144.78) (size 12.7 3.81) (fields_autoplaced)
+  (sheet (at 80.01 146.05) (size 12.7 3.81) (fields_autoplaced)
     (stroke (width 0) (type solid))
     (fill (color 0 0 0 0.0000))
-    (property "Sheetname" "TFT LCD Audio USB" (at 181.61 144.0684 0)
+    (property "Sheetname" "TFT LCD Audio USB" (at 80.01 145.3384 0)
       (effects (font (size 1.27 1.27)) (justify left bottom))
     )
-    (property "Sheetfile" "TFT_LCD_Audio_USB.kicad_sch" (at 181.61 149.1746 0)
+    (property "Sheetfile" "TFT_LCD_Audio_USB.kicad_sch" (at 80.01 150.4446 0)
       (effects (font (size 1.27 1.27)) (justify left top))
     )

Commit message: Updating License informations
Other:
- company: (none) -> Intergalaktik d.o.o.
- title: (none) -> BB3 CM3
Changed lines of the file:
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@@
 (kicad_sch (version 20230121) (generator eeschema)
   (paper "A4")
+  (title_block
+    (title "BB3 CM3")
+    (date "2023-06-28")
+    (rev "v001")
+    (company "Intergalaktik d.o.o.")
+    (comment 1 "This hardware is licensed under CERN-OHL-S v2 or later.")
+  )
   (wire (pts (xy 143.51 71.12) (xy 143.51 76.2))
     (stroke (width 0) (type default))
