File: EEZ_DIB_MCU_r3B4/PSU.kicad_sch (KiCad schematic)
At the start: 4 parts, among them IC5 LD1117ADT33TR

Commit message: Moving footprints - change 0804 to 0603
Parts:
- C15: footprint EEZ_DIB_MCU_r3B4:C0603 -> Capacitor_SMD:C_0603_1608Metric
Changed lines of the file:
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@@
       (effects (font (size 1.778 1.5113)) (justify right top))
     )
-    (property "Footprint" "EEZ_DIB_MCU_r3B4:C0603" (at 115.57 66.04 0)
+    (property "Footprint" "Capacitor_SMD:C_0603_1608Metric" (at 115.57 66.04 0)
       (effects (font (size 1.27 1.27)) hide)
     )

Commit message: Updating License informations
Other:
- company: (none) -> Intergalaktik d.o.o.
- title: (none) -> BB3 CM3
Changed lines of the file:
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@@
 (kicad_sch (version 20230121) (generator eeschema)
   (paper "A4")
+  (title_block
+    (title "BB3 CM3")
+    (date "2023-06-28")
+    (rev "v001")
+    (company "Intergalaktik d.o.o.")
+    (comment 1 "This hardware is licensed under CERN-OHL-S v2 or later.")
+  )
   (junction (at 115.57 60.96) (diameter 0) (color 0 0 0 0)
   )
