File: EEZ_DIB_MCU_r3B4/WatchDog.kicad_sch (KiCad schematic)
At the start: 3 parts, among them IC9 N.C.

Commit message: Moving footprints - change 0804 to 0603
Parts:
- R25: footprint EEZ_DIB_MCU_r3B4:R0805 -> Resistor_SMD:R_0603_1608Metric
Changed lines of the file:
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@@
       (effects (font (size 1.778 1.5113)) (justify left bottom))
     )
-    (property "Footprint" "EEZ_DIB_MCU_r3B4:R0805" (at 132.08 93.98 0)
+    (property "Footprint" "Resistor_SMD:R_0603_1608Metric" (at 132.08 93.98 0)
       (effects (font (size 1.27 1.27)) hide)
     )

Commit message: Updating License informations
Other:
- company: (none) -> Intergalaktik d.o.o.
- title: (none) -> BB3 CM3
Changed lines of the file:
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@@
 (kicad_sch (version 20230121) (generator eeschema)
   (paper "A4")
+  (title_block
+    (title "BB3 CM3")
+    (date "2023-06-28")
+    (rev "v001")
+    (company "Intergalaktik d.o.o.")
+    (comment 1 "This hardware is licensed under CERN-OHL-S v2 or later.")
+  )
   (wire (pts (xy 127 101.6) (xy 127 104.14))
     (stroke (width 0) (type default))
