File: EEZ_DIB_MCU_r3B4/cm4_io_slow.kicad_sch (KiCad schematic)
At the start: 1 part

Commit message: Splitting SoM and MCU board
Connections:
- net GND: now reaches Module1.1 (GND)
- net GND: now also Module1.13 (GND), Module1.14 (GND), Module1.2 (GND), Module1.22 (GND), Module1.23 (GND), Module1.32 (GND), Module1.33 (GND), Module1.42 (GND), Module1.43 (GND), Module1.52 (GND), Module1.53 (GND), Module1.59 (GND), Module1.60 (GND), Module1.65 (GND), Module1.66 (GND), Module1.7 (GND), Module1.71 (GND), Module1.74 (GND), Module1.8 (GND), Module1.98 (GND)
- net RESET: now reaches Module1.100 (nEXTRST)
- net ACT_LED: now reaches Module1.21 (PI_nLED_Activity)
- net SPI5_CSB: now reaches Module1.24 (GPIO26)
- net SPI4_CLK: now reaches Module1.25 (GPIO21)
- net SPI4_MISO: now reaches Module1.26 (GPIO19)
- net SPI4_MOSI: now reaches Module1.27 (GPIO20)
- net SPI5_MISO: now reaches Module1.28 (GPIO13)
- net DOUT2: now reaches Module1.29 (GPIO16)
- net SPI2_IRQ: now reaches Module1.30 (GPIO6)
- net SPI5_CSA: now reaches Module1.31 (GPIO12)
- net DAC_OUT1: now reaches Module1.34 (GPIO5)
- net UART_RX/DIN1: now reaches Module1.35 (ID_SC)
- net UART_TX/DOUT1: now reaches Module1.36 (ID_SD)
- net SPI2_CSB: now reaches Module1.37 (GPIO7)
- net SPI2_CLK: now reaches Module1.38 (GPIO11)
- net SPI2_CSA: now reaches Module1.39 (GPIO8)
- net SPI2_MISO: now reaches Module1.40 (GPIO9)
- net DIN2: now reaches Module1.41 (GPIO25)
- net SPI2_MOSI: now reaches Module1.44 (GPIO10)
- net ENC_SW: now reaches Module1.45 (GPIO24)
- net SPI5_IRQ: now reaches Module1.46 (GPIO22)
- net USER_SW: now reaches Module1.47 (GPIO23)
- net SPI4_IRQ: now reaches Module1.48 (GPIO27)
- net SPI4_CSA: now reaches Module1.49 (GPIO18)
- net SPI4_CSB: now reaches Module1.50 (GPIO17)
- net SPI5_CLK: now reaches Module1.51 (GPIO15)
- net IRQ_TOUCH: now reaches Module1.54 (GPIO4)
- net SPI5_MOSI: now reaches Module1.55 (GPIO14)
- net ENC_B: now reaches Module1.56 (GPIO3)
- net SDMMC1_CK: now reaches Module1.57 (SD_CLK)
- net ENC_A: now reaches Module1.58 (GPIO2)
- net SDMMC1_D0: now reaches Module1.61 (SD_DAT3)
- net SDMMC1_D0: now also Module1.63 (SD_DAT0)
- net SDMMC1_CMD: now reaches Module1.62 (SD_CMD)
- net SD_DETECT: now reaches Module1.75 (SD_PWR_ON)
- net +5V: now reaches Module1.77 (+5v_(Input))
- net +5V: now also Module1.79 (+5v_(Input)), Module1.81 (+5v_(Input)), Module1.83 (+5v_(Input)), Module1.85 (+5v_(Input)), Module1.87 (+5v_(Input))
- net I2C1_SCL: now reaches Module1.80 (SCL0)
- net I2C1_SDA: now reaches Module1.82 (SDA0)
- net CM4_3.3V: now reaches Module1.84 (+3.3v_(Output))
- net CM4_3.3V: now also Module1.86 (+3.3v_(Output)), Module1.95 (nPI_LED_PWR)
- net BOOT0: now reaches Module1.93 (nRPIBOOT)
- net ADC2_IN6: now reaches Module1.94 (AnalogIP1)
- net ADC1_IN5: now reaches Module1.96 (AnalogIP0)
- net CAM_GPIO: now reaches Module1.97 (Camera_GPIO)
- net EN_GPIO: now reaches Module1.99 (Global_EN)

Commit message: Adding ICN6211
Connections:
- no-connect marks 0 -> 17
Other:
- moved on the sheet: Module1A

Commit message: Updating 3D models
Parts:
- added J3: HR911130A, HR911130A:HANRUN_HR911130A, symbol HR911130A:HR911130A
Connections:
- new net: J3.S1 (SHIELD), J3.S2 (SHIELD)
Changed lines of the file:
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@@
+    )
+  )
+  (symbol (lib_id "HR911130A:HR911130A") (at 229.87 105.41 0) (unit 1)
+    (in_bom yes) (on_board yes) (dnp no) (fields_autoplaced)
+    (property "Reference" "J3" (at 238.76 106.045 0)
+      (effects (font (size 1.27 1.27)) (justify left))
+    )
+    (property "Value" "HR911130A" (at 238.76 108.585 0)
+      (effects (font (size 1.27 1.27)) (justify left))
+    )
+    (property "Footprint" "HR911130A:HANRUN_HR911130A" (at 229.87 105.41 0)
+      (effects (font (size 1.27 1.27)) (justify bottom) hide)
+    )
+    (property "Datasheet" "" (at 229.87 105.41 0)
+      (effects (font (size 1.27 1.27)) hide)
+    )
+    (property "PARTREV" "A" (at 229.87 105.41 0)
+      (effects (font (size 1.27 1.27)) (justify bottom) hide)
+    )
+    (property "MANUFACTURER" "HanRun" (at 229.87 105.41 0)
+      (effects (font (size 1.27 1.27)) (justify bottom) hide)
+    )
+    (property "MAXIMUM_PACKAGE_HEIGHT" "13.75 mm" (at 229.87 105.41 0)
+      (effects (font (size 1.27 1.27)) (justify bottom) hide)
+    )
+    (property "STANDARD" "Manufacturer Recommendations" (at 229.87 105.41 0)
+      (effects (font (size 1.27 1.27)) (justify bottom) hide)
+    )
+    (pin "1")
+    (pin "10")
+    (pin "11")
+    (pin "12")
+    (pin "13")
+    (pin "14")
+    (pin "2")
+    (pin "3")
+    (pin "4")
+    (pin "5")
+    (pin "6")
+    (pin "7")
+    (pin "8")
+    (pin "9")
+    (pin "S1")
+    (pin "S2")
+    (instances
+      (project "EEZ_DIB_MCU_r3B4"
+        (path "/58be380a-4a3a-4b30-b3f5-a03bc3bf2660/4fa14b62-9505-4857-82d9-8b729da152fe"
+          (reference "J3") (unit 1)
+        )
+      )
     )
   )

Commit message: Adding connections to Ethernet connector
Parts:
- added C26: C_Small, symbol Device:C_Small
- added R22, R38, R39: R_Small, symbol Device:R_Small
Connections:
- net GND: now also J3.12, J3.13, J3.S1 (SHIELD), J3.S2 (SHIELD), C26.1, R22.2
- net at J3.1 (P1): now also C26.2
- net at J3.10 (P10): now also R22.1
- net at J3.11: now also R38.1
- net at J3.14: now also R39.1
- net eth_0p: now reaches J3.2 (P2)
- net eth_0p: now also Module1.12 (Ethernet_Pair0_P)
- net eth_0n: now reaches J3.3 (P3)
- net eth_0n: now also Module1.10 (Ethernet_Pair0_N)
- net eth_1p: now reaches J3.4 (P4)
- net eth_1p: now also Module1.4 (Ethernet_Pair1_P)
- net eth_2p: now reaches J3.5 (P5)
- net eth_2p: now also Module1.9 (Ethernet_Pair2_N)
- net eth_2n: now reaches J3.6 (P6)
- net eth_2n: now also Module1.11 (Ethernet_Pair2_P)
- net eth_1n: now reaches J3.7 (P7)
- net eth_1n: now also Module1.6 (Ethernet_Pair1_N)
- net eth_3p: now reaches J3.8 (P8)
- net eth_3p: now also Module1.3 (Ethernet_Pair3_P)
- net eth_3n: now reaches J3.9 (P9)
- net eth_3n: now also Module1.5 (Ethernet_Pair3_N)
- net eth_led3: now reaches Module1.15 (Ethernet_nLED3(3.3v))
- net eth_led2: now reaches Module1.17 (Ethernet_nLED2(3.3v))
- net eth_led2: now also R38.2
- net eth_led1: now reaches Module1.19 (Ethernet_nLED1(3.3v))
- net eth_led1: now also R39.2

Commit message: Adding DSI connector
Parts:
- C26: footprint (none) -> Capacitor_SMD:C_0603_1608Metric
- R22, R38, R39: footprint (none) -> Resistor_SMD:R_0603_1608Metric
Changed lines of the file:
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@@
       (effects (font (size 1.27 1.27)))
     )
-    (property "Value" "R_Small" (at 212.09 105.41 90)
-      (effects (font (size 1.27 1.27)))
-    )
-    (property "Footprint" "" (at 212.09 107.95 0)
+    (property "Value" "R_Small" (at 205.74 109.22 90)
+      (effects (font (size 1.27 1.27)))
+    )
+    (property "Footprint" "Resistor_SMD:R_0603_1608Metric" (at 212.09 107.95 0)
       (effects (font (size 1.27 1.27)) hide)
     )
@@
       (effects (font (size 1.27 1.27)))
     )
-    (property "Footprint" "" (at 208.28 80.01 0)
+    (property "Footprint" "Capacitor_SMD:C_0603_1608Metric" (at 208.28 80.01 0)
       (effects (font (size 1.27 1.27)) hide)
     )
@@
       (effects (font (size 1.27 1.27)))
     )
-    (property "Value" "R_Small" (at 212.09 118.11 90)
-      (effects (font (size 1.27 1.27)))
-    )
-    (property "Footprint" "" (at 212.09 120.65 0)
+    (property "Value" "R_Small" (at 205.74 121.92 90)
+      (effects (font (size 1.27 1.27)))
+    )
+    (property "Footprint" "Resistor_SMD:R_0603_1608Metric" (at 212.09 120.65 0)
       (effects (font (size 1.27 1.27)) hide)
     )
@@
       (effects (font (size 1.27 1.27)))
     )
-    (property "Value" "R_Small" (at 212.09 100.33 90)
-      (effects (font (size 1.27 1.27)))
-    )
-    (property "Footprint" "" (at 212.09 102.87 0)
-      (effects (font (size 1.27 1.27)) hide)
-    )
+    (property "Value" "R_Small" (at 205.74 104.14 90)
+      (effects (font (size 1.27 1.27)))
+    )
+    (property "Footprint" "Resistor_SMD:R_0603_1608Metric" (at 212.09 102.87 0)
+      (effects (font (size 1.27 1.27)) hide)
+    )

Commit message: Routing
Connections:
- net eth_0n renamed ETH_0N
- net eth_0p renamed ETH_0P
- net eth_1n renamed ETH_1N
- net eth_1p renamed ETH_1P
- net eth_2n renamed ETH_2N
- net eth_2p renamed ETH_2P
- net eth_3n renamed ETH_3N
- net eth_3p renamed ETH_3P
Changed lines of the file:
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@@
     )
   )
-  (label "eth_1p" (at 205.74 87.63 180) (fields_autoplaced)
+  (label "ETH_1P" (at 205.74 87.63 180) (fields_autoplaced)
     (effects (font (size 1.27 1.27)) (justify right bottom))
   )
-  (label "eth_2n" (at 205.74 92.71 180) (fields_autoplaced)
+  (label "ETH_2N" (at 205.74 92.71 180) (fields_autoplaced)
     (effects (font (size 1.27 1.27)) (justify right bottom))
   )
@@
     (effects (font (size 1.27 1.27)) (justify right bottom))
   )
-  (label "eth_3n" (at 90.17 85.09 180) (fields_autoplaced)
+  (label "ETH_3N" (at 90.17 85.09 180) (fields_autoplaced)
     (effects (font (size 1.27 1.27)) (justify right bottom))
   )
-  (label "eth_3n" (at 205.74 100.33 180) (fields_autoplaced)
+  (label "ETH_3N" (at 205.74 100.33 180) (fields_autoplaced)
     (effects (font (size 1.27 1.27)) (justify right bottom))
   )
-  (label "eth_3p" (at 90.17 82.55 180) (fields_autoplaced)
+  (label "ETH_3P" (at 90.17 82.55 180) (fields_autoplaced)
     (effects (font (size 1.27 1.27)) (justify right bottom))
   )
-  (label "eth_2p" (at 205.74 90.17 180) (fields_autoplaced)
+  (label "ETH_2P" (at 205.74 90.17 180) (fields_autoplaced)
     (effects (font (size 1.27 1.27)) (justify right bottom))
   )
-  (label "eth_3p" (at 205.74 97.79 180) (fields_autoplaced)
+  (label "ETH_3P" (at 205.74 97.79 180) (fields_autoplaced)
     (effects (font (size 1.27 1.27)) (justify right bottom))
   )
-  (label "eth_1p" (at 172.72 82.55 0) (fields_autoplaced)
+  (label "ETH_1P" (at 172.72 82.55 0) (fields_autoplaced)
     (effects (font (size 1.27 1.27)) (justify left bottom))
   )
-  (label "eth_1n" (at 205.74 95.25 180) (fields_autoplaced)
+  (label "ETH_1N" (at 205.74 95.25 180) (fields_autoplaced)
     (effects (font (size 1.27 1.27)) (justify right bottom))
   )
-  (label "eth_0n" (at 205.74 85.09 180) (fields_autoplaced)
+  (label "ETH_0N" (at 205.74 85.09 180) (fields_autoplaced)
     (effects (font (size 1.27 1.27)) (justify right bottom))
   )
-  (label "eth_2p" (at 90.17 90.17 180) (fields_autoplaced)
+  (label "ETH_2P" (at 90.17 90.17 180) (fields_autoplaced)
     (effects (font (size 1.27 1.27)) (justify right bottom))
   )
@@
     (effects (font (size 1.27 1.27)) (justify right bottom))
   )
-  (label "eth_0p" (at 172.72 92.71 0) (fields_autoplaced)
+  (label "ETH_0P" (at 172.72 92.71 0) (fields_autoplaced)
     (effects (font (size 1.27 1.27)) (justify left bottom))
   )
-  (label "eth_2n" (at 90.17 92.71 180) (fields_autoplaced)
+  (label "ETH_2N" (at 90.17 92.71 180) (fields_autoplaced)
     (effects (font (size 1.27 1.27)) (justify right bottom))
   )
-  (label "eth_1n" (at 172.72 85.09 0) (fields_autoplaced)
+  (label "ETH_1N" (at 172.72 85.09 0) (fields_autoplaced)
     (effects (font (size 1.27 1.27)) (justify left bottom))
   )
-  (label "eth_0p" (at 205.74 82.55 180) (fields_autoplaced)
+  (label "ETH_0P" (at 205.74 82.55 180) (fields_autoplaced)
     (effects (font (size 1.27 1.27)) (justify right bottom))
   )
-  (label "eth_0n" (at 172.72 90.17 0) (fields_autoplaced)
+  (label "ETH_0N" (at 172.72 90.17 0) (fields_autoplaced)
     (effects (font (size 1.27 1.27)) (justify left bottom))
   )

Commit message: Update pictures and 3D models
Connections:
- net SDMMC1_D0: no longer Module1.61 (SD_DAT3)
- no-connect marks 17 -> 18
Changed lines of the file:
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@@
   (no_connect (at 162.56 194.31))
   (no_connect (at 101.6 166.37))
+  (no_connect (at 101.6 156.21))
   (no_connect (at 162.56 100.33))
   (no_connect (at 162.56 189.23))
@@
     (stroke (width 0) (type default))
   )
-  (wire (pts (xy 101.6 156.21) (xy 97.79 156.21))
-    (stroke (width 0) (type default))
-  )
   (wire (pts (xy 101.6 146.05) (xy 97.79 146.05))
     (stroke (width 0) (type default))
@@
       (effects (font (size 1.27 1.27)) (justify right) hide)
     )
-  )
-  (global_label "SDMMC1_D0" (shape input) (at 97.79 156.21 180) (fields_autoplaced)
-    (effects (font (size 1.27 1.27)) (justify right))
-    (property "Intersheetrefs" "${INTERSHEET_REFS}" (at 83.5753 156.21 0)
-      (effects (font (size 1.27 1.27)) (justify right) hide)
-    )

Commit message: Updating License informations
Other:
- company: (none) -> Intergalaktik d.o.o.
- title: (none) -> BB3 CM3
Changed lines of the file:
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@@
 (kicad_sch (version 20230121) (generator eeschema)
   (paper "A4")
+  (title_block
+    (title "BB3 CM3")
+    (date "2023-06-28")
+    (rev "v001")
+    (company "Intergalaktik d.o.o.")
+    (comment 1 "This hardware is licensed under CERN-OHL-S v2 or later.")
+  )
   (junction (at 194.31 102.87) (diameter 0) (color 0 0 0 0)
   )
