File: EEZ_DIB_MCU_r3B4/IO_connectors_Encoder_user_SW.kicad_sch (KiCad schematic)
At the start: 39 parts, among them IC1 TPD4E001DRLR, IC2 74AUP1G74DC.125, IC3 CD74HC4050PWR, SW1 TL1100CF160Q, SW2 PEC16-2215F-S0024, X1 DS1024-2*20R0, X2 DS1013-16SSIB1, X3 691322110005

Commit message: Adding ICN6211
Parts:
- removed JP1, JP2: JP2-NOCUT, EEZ_DIB_MCU_r3B4:JP2-NOCUT, symbol EEZ_DIB_MCU_r3B4-eagle-import:JP2-NOCUT
Connections:
- net I2C1_SCL: now also X2.13 (1)
- net I2C1_SDA: now also X2.14 (1)
Changed lines of the file:
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@@
     (stroke (width 0) (type default))
   )
-  (wire (pts (xy 78.74 58.42) (xy 83.82 58.42))
+  (wire (pts (xy 78.74 58.42) (xy 96.52 58.42))
     (stroke (width 0) (type default))
   )
@@
     (stroke (width 0) (type default))
   )
-  (wire (pts (xy 43.18 58.42) (xy 48.26 58.42))
-    (stroke (width 0) (type default))
-  )
   (wire (pts (xy 187.96 134.62) (xy 187.96 139.7))
     (stroke (width 0) (type default))
@@
     (stroke (width 0) (type default))
   )
-  (wire (pts (xy 86.36 58.42) (xy 96.52 58.42))
-    (stroke (width 0) (type default))
-  )
   (wire (pts (xy 34.29 45.72) (xy 33.02 45.72))
     (stroke (width 0) (type default))
@@
     (stroke (width 0) (type default))
   )
-  (wire (pts (xy 40.64 58.42) (xy 30.48 58.42))
+  (wire (pts (xy 30.48 58.42) (xy 48.26 58.42))
     (stroke (width 0) (type default))
   )
@@
     )
   )
-  (symbol (lib_id "EEZ_DIB_MCU_r3B4-eagle-import:JP2-NOCUT") (at 40.64 58.42 0) (unit 1)
-    (in_bom yes) (on_board yes) (dnp no)
-    (property "Reference" "JP1" (at 40.64 57.785 0)
-      (effects (font (size 1.778 1.5113)) (justify left bottom))
-    )
-    (property "Value" "JP2-NOCUT" (at 40.64 58.42 0)
-      (effects (font (size 1.27 1.27)) hide)
-    )
-    (property "Footprint" "EEZ_DIB_MCU_r3B4:JP2-NOCUT" (at 40.64 58.42 0)
-      (effects (font (size 1.27 1.27)) hide)
-    )
-    (property "Datasheet" "" (at 40.64 58.42 0)
-      (effects (font (size 1.27 1.27)) hide)
-    )
-    (pin "1")
-    (pin "2")
-    (instances
-      (project "EEZ_DIB_MCU_r3B4"
-        (path "/58be380a-4a3a-4b30-b3f5-a03bc3bf2660/bdd2bf4d-fded-4f6c-9725-0b2ab500c01f"
-          (reference "JP1") (unit 1)
-        )
-      )
-    )
-  )
   (symbol (lib_id "EEZ_DIB_MCU_r3B4-eagle-import:R-EU_R0805") (at 238.76 121.92 180) (unit 1)
     (in_bom yes) (on_board yes) (dnp no)
@@
         )
       )
-    )
-  )
-  (symbol (lib_id "EEZ_DIB_MCU_r3B4-eagle-import:JP2-NOCUT") (at 83.82 58.42 0) (unit 1)
-    (in_bom yes) (on_board yes) (dnp no)
-    (property "Reference" "JP2" (at 83.185 57.785 0)
-      (effects (font (size 1.778 1.5113)) (justify left bottom))
-    )
-    (property "Value" "JP2-NOCUT" (at 83.82 58.42 0)
-      (effects (font (size 1.27 1.27)) hide)
-    )
-    (property "Footprint" "EEZ_DIB_MCU_r3B4:JP2-NOCUT" (at 83.82 58.42 0)
-      (effects (font (size 1.27 1.27)) hide)
-    )
-    (property "Datasheet" "" (at 83.82 58.42 0)
-      (effects (font (size 1.27 1.27)) hide)
-    )
-    (pin "1")
-    (pin "2")
-    (instances
-      (project "EEZ_DIB_MCU_r3B4"
-        (path "/58be380a-4a3a-4b30-b3f5-a03bc3bf2660/bdd2bf4d-fded-4f6c-9725-0b2ab500c01f"
-          (reference "JP2") (unit 1)
-        )
-      )

Commit message: Moving footprints - change 0804 to 0603
Parts:
- C2, C3, C5, C7, C8: footprint EEZ_DIB_MCU_r3B4:C0805 -> Capacitor_SMD:C_0603_1608Metric
- C4, C6, C9: footprint EEZ_DIB_MCU_r3B4:C0603 -> Capacitor_SMD:C_0603_1608Metric
- R1, R10, R11, R2, R3, R4, R5, R6, R7, R8, R9: footprint EEZ_DIB_MCU_r3B4:R0805 -> Resistor_SMD:R_0603_1608Metric
Changed lines of the file:
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@@
       (effects (font (size 1.778 1.5113)) (justify right top))
     )
-    (property "Footprint" "EEZ_DIB_MCU_r3B4:C0805" (at 208.28 127 0)
+    (property "Footprint" "Capacitor_SMD:C_0603_1608Metric" (at 208.28 127 0)
       (effects (font (size 1.27 1.27)) hide)
     )
@@
       (effects (font (size 1.778 1.5113)) (justify left top))
     )
-    (property "Footprint" "EEZ_DIB_MCU_r3B4:R0805" (at 119.38 134.62 0)
+    (property "Footprint" "Resistor_SMD:R_0603_1608Metric" (at 119.38 134.62 0)
       (effects (font (size 1.27 1.27)) hide)
     )
@@
       (effects (font (size 1.778 1.5113)) (justify left top))
     )
-    (property "Footprint" "EEZ_DIB_MCU_r3B4:R0805" (at 76.2 134.62 0)
+    (property "Footprint" "Resistor_SMD:R_0603_1608Metric" (at 76.2 134.62 0)
       (effects (font (size 1.27 1.27)) hide)
     )
@@
       (effects (font (size 1.778 1.5113)) (justify right top))
     )
-    (property "Footprint" "EEZ_DIB_MCU_r3B4:R0805" (at 195.58 116.84 0)
+    (property "Footprint" "Resistor_SMD:R_0603_1608Metric" (at 195.58 116.84 0)
       (effects (font (size 1.27 1.27)) hide)
     )
@@
       (effects (font (size 1.778 1.5113)) (justify right bottom))
     )
-    (property "Footprint" "EEZ_DIB_MCU_r3B4:R0805" (at 198.12 139.7 0)
+    (property "Footprint" "Resistor_SMD:R_0603_1608Metric" (at 198.12 139.7 0)
       (effects (font (size 1.27 1.27)) hide)
     )
@@
       (effects (font (size 1.778 1.5113)) (justify right bottom))
     )
-    (property "Footprint" "EEZ_DIB_MCU_r3B4:R0805" (at 203.2 121.92 0)
+    (property "Footprint" "Resistor_SMD:R_0603_1608Metric" (at 203.2 121.92 0)
       (effects (font (size 1.27 1.27)) hide)
     )
@@
       (effects (font (size 1.778 1.5113)) (justify right top))
     )
-    (property "Footprint" "EEZ_DIB_MCU_r3B4:R0805" (at 238.76 121.92 0)
+    (property "Footprint" "Resistor_SMD:R_0603_1608Metric" (at 238.76 121.92 0)
       (effects (font (size 1.27 1.27)) hide)
     )
@@
       (effects (font (size 1.778 1.5113)) (justify right top))
     )
-    (property "Footprint" "EEZ_DIB_MCU_r3B4:R0805" (at 190.5 129.54 0)
+    (property "Footprint" "Resistor_SMD:R_0603_1608Metric" (at 190.5 129.54 0)
       (effects (font (size 1.27 1.27)) hide)
     )
@@
       (effects (font (size 1.778 1.5113)) (justify left top))
     )
-    (property "Footprint" "EEZ_DIB_MCU_r3B4:R0805" (at 76.2 124.46 0)
+    (property "Footprint" "Resistor_SMD:R_0603_1608Metric" (at 76.2 124.46 0)
       (effects (font (size 1.27 1.27)) hide)
     )
@@
       (effects (font (size 1.778 1.5113)) (justify right top))
     )
-    (property "Footprint" "EEZ_DIB_MCU_r3B4:C0805" (at 180.34 111.76 0)
+    (property "Footprint" "Capacitor_SMD:C_0603_1608Metric" (at 180.34 111.76 0)
       (effects (font (size 1.27 1.27)) hide)
     )
@@
       (effects (font (size 1.778 1.5113)) (justify left top))
     )
-    (property "Footprint" "EEZ_DIB_MCU_r3B4:R0805" (at 60.96 134.62 0)
+    (property "Footprint" "Resistor_SMD:R_0603_1608Metric" (at 60.96 134.62 0)
       (effects (font (size 1.27 1.27)) hide)
     )
@@
       (effects (font (size 1.778 1.5113)) (justify left bottom))
     )
-    (property "Footprint" "EEZ_DIB_MCU_r3B4:C0805" (at 254 96.52 0)
+    (property "Footprint" "Capacitor_SMD:C_0603_1608Metric" (at 254 96.52 0)
       (effects (font (size 1.27 1.27)) hide)
     )
@@
       (effects (font (size 1.778 1.5113)) (justify left bottom))
     )
-    (property "Footprint" "EEZ_DIB_MCU_r3B4:C0805" (at 208.28 142.24 0)
+    (property "Footprint" "Capacitor_SMD:C_0603_1608Metric" (at 208.28 142.24 0)
       (effects (font (size 1.27 1.27)) hide)
     )
@@
       (effects (font (size 1.778 1.5113)) (justify left top))
     )
-    (property "Footprint" "EEZ_DIB_MCU_r3B4:R0805" (at 60.96 124.46 0)
+    (property "Footprint" "Resistor_SMD:R_0603_1608Metric" (at 60.96 124.46 0)
       (effects (font (size 1.27 1.27)) hide)
     )
@@
       (effects (font (size 1.778 1.5113)) (justify left bottom))
     )
-    (property "Footprint" "EEZ_DIB_MCU_r3B4:C0805" (at 172.72 78.74 0)
+    (property "Footprint" "Capacitor_SMD:C_0603_1608Metric" (at 172.72 78.74 0)
       (effects (font (size 1.27 1.27)) hide)
     )
@@
       (effects (font (size 1.778 1.5113)) (justify left top))
     )
-    (property "Footprint" "EEZ_DIB_MCU_r3B4:R0805" (at 119.38 124.46 0)
+    (property "Footprint" "Resistor_SMD:R_0603_1608Metric" (at 119.38 124.46 0)
       (effects (font (size 1.27 1.27)) hide)
     )
@@
       (effects (font (size 1.778 1.5113)) (justify left bottom))
     )
-    (property "Footprint" "EEZ_DIB_MCU_r3B4:C0603" (at 152.4 121.92 0)
+    (property "Footprint" "Capacitor_SMD:C_0603_1608Metric" (at 152.4 121.92 0)
       (effects (font (size 1.27 1.27)) hide)
     )
@@
       (effects (font (size 1.778 1.5113)) (justify left bottom))
     )
-    (property "Footprint" "EEZ_DIB_MCU_r3B4:C0603" (at 116.84 104.14 0)
+    (property "Footprint" "Capacitor_SMD:C_0603_1608Metric" (at 116.84 104.14 0)
       (effects (font (size 1.27 1.27)) hide)
     )
@@
       (effects (font (size 1.778 1.5113)) (justify left bottom))
     )
-    (property "Footprint" "EEZ_DIB_MCU_r3B4:C0603" (at 236.22 149.86 0)
+    (property "Footprint" "Capacitor_SMD:C_0603_1608Metric" (at 236.22 149.86 0)
       (effects (font (size 1.27 1.27)) hide)
     )

Commit message: Update pictures and 3D models
Parts:
- removed LABEL1: HR000002, EEZ_DIB_MCU_r3B4:CERT-SMALL-SILK, symbol EEZ_DIB_MCU_r3B4-eagle-import:OSHWA-CERT-SMALL
Changed lines of the file:
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@@
-    )
-  )
-  (symbol (lib_id "EEZ_DIB_MCU_r3B4-eagle-import:OSHWA-CERT-SMALL") (at 26.67 186.69 0) (unit 1)
-    (in_bom yes) (on_board yes) (dnp no)
-    (property "Reference" "LABEL1" (at 26.67 186.69 0)
-      (effects (font (size 1.27 1.27)) hide)
-    )
-    (property "Value" "HR000002" (at 20.701 189.23 0)
-      (effects (font (size 1.778 1.778)) (justify left bottom))
-    )
-    (property "Footprint" "EEZ_DIB_MCU_r3B4:CERT-SMALL-SILK" (at 26.67 186.69 0)
-      (effects (font (size 1.27 1.27)) hide)
-    )
-    (property "Datasheet" "" (at 26.67 186.69 0)
-      (effects (font (size 1.27 1.27)) hide)
-    )
-    (instances
-      (project "EEZ_DIB_MCU_r3B4"
-        (path "/58be380a-4a3a-4b30-b3f5-a03bc3bf2660/bdd2bf4d-fded-4f6c-9725-0b2ab500c01f"
-          (reference "LABEL1") (unit 1)
-        )
-      )
     )
   )

Commit message: Updating License informations
Other:
- note removed: "Licensed under the TAPR Open Hardware License (www.tapr.org/OHL)"
- note removed: "More info at http://www.envox.hr/eez"
- note removed: "Repository: https://github.com/eez-open"
- company: (none) -> Intergalaktik d.o.o.
- title: (none) -> BB3 CM3
Changed lines of the file:
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@@
 (kicad_sch (version 20230121) (generator eeschema)
   (paper "User" 303.403 218.491)
+  (title_block
+    (title "BB3 CM3")
+    (date "2023-06-28")
+    (rev "v001")
+    (company "Intergalaktik d.o.o.")
+    (comment 1 "This hardware is licensed under CERN-OHL-S v2 or later.")
+  )
   (junction (at 241.3 157.48) (diameter 0) (color 0 0 0 0)
   )
@@
     (effects (font (size 1.4224 1.209)) (justify left bottom))
   )
-  (text "More info at http://www.envox.hr/eez" (at 20.32 193.675 0)
-    (effects (font (size 1.27 1.0795)) (justify left bottom))
-  )
   (text "User / Boot0 switch" (at 228.6 93.98 0)
     (effects (font (size 1.778 1.5113)) (justify left bottom))
@@
     (effects (font (size 1.4224 1.209)) (justify left bottom))
   )
-  (text "Licensed under the TAPR Open Hardware License (www.tapr.org/OHL)"
-    (at 20.32 191.77 0)
-    (effects (font (size 1.27 1.0795)) (justify left bottom))
-  )
   (text "DIN2 2" (at 41.91 102.235 0)
     (effects (font (size 1.4224 1.209)) (justify right bottom))
   )
-  (text "Repository: https://github.com/eez-open" (at 20.32 195.58 0)
-    (effects (font (size 1.27 1.0795)) (justify left bottom))
-  )
   (text "40-pin DIB v1.0 backplane socket" (at 233.68 31.115 0)
     (effects (font (size 2.1844 1.8567)) (justify left bottom))
@@
         )
       )
-    )
-  )
-  (symbol (lib_id "EEZ_DIB_MCU_r3B4-eagle-import:DINA4_L") (at 180.34 198.12 0) (unit 2)
-    (in_bom yes) (on_board yes) (dnp no)
-    (property "Reference" "#FRAME1" (at 180.34 198.12 0)
-      (effects (font (size 1.27 1.27)) hide)
-    )
-    (property "Value" "DINA4_L" (at 180.34 198.12 0)
-      (effects (font (size 1.27 1.27)) hide)
-    )
-    (property "Footprint" "EEZ_DIB_MCU_r3B4:" (at 180.34 198.12 0)
-      (effects (font (size 1.27 1.27)) hide)
-    )
-    (property "Datasheet" "" (at 180.34 198.12 0)
-      (effects (font (size 1.27 1.27)) hide)
-    )
-    (instances
-      (project "EEZ_DIB_MCU_r3B4"
-        (path "/58be380a-4a3a-4b30-b3f5-a03bc3bf2660/bdd2bf4d-fded-4f6c-9725-0b2ab500c01f"
-          (reference "#FRAME1") (unit 2)
-        )
-      )

Commit message: Adding temperary PCIe connector - adding logos
Parts:
- added C?: 4u7, EEZ_DIB_MCU_r3B4:EC1206, symbol EEZ_DIB_MCU_r3B4-eagle-import:ECAP1206
- added F1: 500mA, Fuse:Fuse_0805_2012Metric, symbol Device:Fuse_Small
- added IC?: TPS2051BDBVR, EEZ_DIB_MCU_r3B4:DBV5, symbol EEZ_DIB_MCU_r3B4-eagle-import:TPS2051B
- added R40: 0R, Resistor_SMD:R_0603_1608Metric, symbol EEZ_DIB_MCU_r3B4-eagle-import:R-EU_R0805
- added R?: 10K, Resistor_SMD:R_0603_1608Metric, symbol EEZ_DIB_MCU_r3B4-eagle-import:R-EU_R0805
- C1: footprint EEZ_DIB_MCU_r3B4:PANASONIC_C -> Fuse:Fuse_0805_2012Metric
Connections:
- net +5V: now also IC?.5 (IN)
- net DOUT2: now also IC?.4 (EN), R?.2
- net GND: now also C?.-, IC?.2 (GND), R?.1
- net at IC1.5 (IO4), X3.5 (1): now also F1.1, R40.1; no longer IC3.10 (O), IC3.6 (O)
- new net: IC3.10 (O), IC3.6 (O), R40.2
- new net: C?.+, IC?.1 (OUT)
- new net 5V_SWITCH_OUT: F1.2, IC?.3 (~{OC})
Other:
- note added: "5V out switch"
- note added: "Default - power off"
- note added: "Tant."
- moved on the sheet: IC3B, IC3C
