File: EEZ_DIB_MCU_r3B4/TFT_LCD_Audio_USB.kicad_sch (KiCad schematic)
At the start: 36 parts, among them IC11 TPS2051BDBVR, IC12 TPS61169DCKR, IC13 TPD4E001DRLR, IC14 TSC2007IPW, J2 67803-8020, Q1 N.C., Q2 2N7002

Commit message: Adding ICN6211
Parts:
- removed JP8: JP3-CUT-0805-ROTATED, EEZ_DIB_MCU_r3B4:JP3-0805-CUT2, symbol EEZ_DIB_MCU_r3B4-eagle-import:JP3-CUT-0805-ROTATED
Connections:
- new net LTDC_B0: LCD1.21 (B0)
- new net LTDC_B1: LCD1.22 (B1)
- new net LTDC_B2: LCD1.23 (B2)
- new net LTDC_G0: LCD1.13 (G0)
- new net LTDC_G1: LCD1.14 (G1)
- new net LTDC_R0: LCD1.5 (R0)
- new net LTDC_R1: LCD1.6 (R1)
- new net LTDC_R2: LCD1.7 (R2)

Commit message: Moving footprints - change 0804 to 0603
Parts:
- C51, C53, C58: footprint EEZ_DIB_MCU_r3B4:C0805 -> Capacitor_SMD:C_0603_1608Metric
- C55, C57: footprint EEZ_DIB_MCU_r3B4:C0603 -> Capacitor_SMD:C_0603_1608Metric
- R26, R27, R28, R29, R30, R31, R32, R33, R34, R35, R36, R37: footprint EEZ_DIB_MCU_r3B4:R0805 -> Resistor_SMD:R_0603_1608Metric
Changed lines of the file:
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@@
       (effects (font (size 1.778 1.5113)) (justify right top))
     )
-    (property "Footprint" "EEZ_DIB_MCU_r3B4:C0805" (at 83.82 35.56 0)
+    (property "Footprint" "Capacitor_SMD:C_0603_1608Metric" (at 83.82 35.56 0)
       (effects (font (size 1.27 1.27)) hide)
     )
@@
       (effects (font (size 1.778 1.5113)) (justify right top))
     )
-    (property "Footprint" "EEZ_DIB_MCU_r3B4:R0805" (at 259.08 91.44 0)
+    (property "Footprint" "Resistor_SMD:R_0603_1608Metric" (at 259.08 91.44 0)
       (effects (font (size 1.27 1.27)) hide)
     )
@@
       (effects (font (size 1.778 1.5113)) (justify left bottom))
     )
-    (property "Footprint" "EEZ_DIB_MCU_r3B4:R0805" (at 264.16 40.64 0)
+    (property "Footprint" "Resistor_SMD:R_0603_1608Metric" (at 264.16 40.64 0)
       (effects (font (size 1.27 1.27)) hide)
     )
@@
       (effects (font (size 1.778 1.5113)) (justify right top))
     )
-    (property "Footprint" "EEZ_DIB_MCU_r3B4:R0805" (at 86.36 93.98 0)
+    (property "Footprint" "Resistor_SMD:R_0603_1608Metric" (at 86.36 93.98 0)
       (effects (font (size 1.27 1.27)) hide)
     )
@@
       (effects (font (size 1.778 1.5113)) (justify left bottom))
     )
-    (property "Footprint" "EEZ_DIB_MCU_r3B4:R0805" (at 254 58.42 0)
+    (property "Footprint" "Resistor_SMD:R_0603_1608Metric" (at 254 58.42 0)
       (effects (font (size 1.27 1.27)) hide)
     )
@@
       (effects (font (size 1.778 1.5113)) (justify right bottom))
     )
-    (property "Footprint" "EEZ_DIB_MCU_r3B4:R0805" (at 213.36 71.12 0)
+    (property "Footprint" "Resistor_SMD:R_0603_1608Metric" (at 213.36 71.12 0)
       (effects (font (size 1.27 1.27)) hide)
     )
@@
       (effects (font (size 1.778 1.5113)) (justify right top))
     )
-    (property "Footprint" "EEZ_DIB_MCU_r3B4:R0805" (at 248.92 91.44 0)
+    (property "Footprint" "Resistor_SMD:R_0603_1608Metric" (at 248.92 91.44 0)
       (effects (font (size 1.27 1.27)) hide)
     )
@@
       (effects (font (size 1.778 1.5113)) (justify left top))
     )
-    (property "Footprint" "EEZ_DIB_MCU_r3B4:C0603" (at 139.7 147.32 0)
+    (property "Footprint" "Capacitor_SMD:C_0603_1608Metric" (at 139.7 147.32 0)
       (effects (font (size 1.27 1.27)) hide)
     )
@@
       (effects (font (size 1.778 1.5113)) (justify right bottom))
     )
-    (property "Footprint" "EEZ_DIB_MCU_r3B4:R0805" (at 195.58 66.04 0)
+    (property "Footprint" "Resistor_SMD:R_0603_1608Metric" (at 195.58 66.04 0)
       (effects (font (size 1.27 1.27)) hide)
     )
@@
       (effects (font (size 1.778 1.5113)) (justify right bottom))
     )
-    (property "Footprint" "EEZ_DIB_MCU_r3B4:C0805" (at 104.14 60.96 0)
+    (property "Footprint" "Capacitor_SMD:C_0603_1608Metric" (at 104.14 60.96 0)
       (effects (font (size 1.27 1.27)) hide)
     )
@@
       (effects (font (size 1.778 1.5113)) (justify right bottom))
     )
-    (property "Footprint" "EEZ_DIB_MCU_r3B4:R0805" (at 43.18 38.1 0)
+    (property "Footprint" "Resistor_SMD:R_0603_1608Metric" (at 43.18 38.1 0)
       (effects (font (size 1.27 1.27)) hide)
     )
@@
       (effects (font (size 1.778 1.5113)) (justify left bottom))
     )
-    (property "Footprint" "EEZ_DIB_MCU_r3B4:R0805" (at 190.5 48.26 0)
+    (property "Footprint" "Resistor_SMD:R_0603_1608Metric" (at 190.5 48.26 0)
       (effects (font (size 1.27 1.27)) hide)
     )
@@
       (effects (font (size 1.778 1.5113)) (justify left bottom))
     )
-    (property "Footprint" "EEZ_DIB_MCU_r3B4:R0805" (at 78.74 53.34 0)
+    (property "Footprint" "Resistor_SMD:R_0603_1608Metric" (at 78.74 53.34 0)
       (effects (font (size 1.27 1.27)) hide)
     )
@@
       (effects (font (size 1.778 1.5113)) (justify right top))
     )
-    (property "Footprint" "EEZ_DIB_MCU_r3B4:C0805" (at 147.32 147.32 0)
+    (property "Footprint" "Capacitor_SMD:C_0603_1608Metric" (at 147.32 147.32 0)
       (effects (font (size 1.27 1.27)) hide)
     )
@@
       (effects (font (size 1.778 1.5113)) (justify left top))
     )
-    (property "Footprint" "EEZ_DIB_MCU_r3B4:R0805" (at 190.5 81.28 0)
+    (property "Footprint" "Resistor_SMD:R_0603_1608Metric" (at 190.5 81.28 0)
       (effects (font (size 1.27 1.27)) hide)
     )
@@
       (effects (font (size 1.778 1.5113)) (justify left top))
     )
-    (property "Footprint" "EEZ_DIB_MCU_r3B4:C0603" (at 203.2 91.44 0)
+    (property "Footprint" "Capacitor_SMD:C_0603_1608Metric" (at 203.2 91.44 0)
       (effects (font (size 1.27 1.27)) hide)
     )
@@
       (effects (font (size 1.778 1.5113)) (justify right bottom))
     )
-    (property "Footprint" "EEZ_DIB_MCU_r3B4:R0805" (at 213.36 68.58 0)
-      (effects (font (size 1.27 1.27)) hide)
-    )
+    (property "Footprint" "Resistor_SMD:R_0603_1608Metric" (at 213.36 68.58 0)
+      (effects (font (size 1.27 1.27)) hide)
+    )

Commit message: Updating 3D models
Other:
- note added: "Missing?"
Changed lines of the file:
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@@
     (effects (font (size 1.778 1.5113)) (justify left bottom))
+  )
+  (text "Missing?" (at 173.99 63.5 0)
+    (effects (font (size 1.27 1.27)) (justify left bottom))
   )
   (text "Licensed under the TAPR Open Hardware License (www.tapr.org/OHL)"

Commit message: Updating License informations
Other:
- note removed: "Licensed under the TAPR Open Hardware License (www.tapr.org/OHL)"
- note removed: "More info at http://www.envox.hr/eez"
- note removed: "Repository: https://github.com/eez-open"
- company: (none) -> Intergalaktik d.o.o.
- title: (none) -> BB3 CM3
Changed lines of the file:
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@@
 (kicad_sch (version 20230121) (generator eeschema)
   (paper "User" 302.311 220.269)
+  (title_block
+    (title "BB3 CM3")
+    (date "2023-06-28")
+    (rev "v001")
+    (company "Intergalaktik d.o.o.")
+    (comment 1 "This hardware is licensed under CERN-OHL-S v2 or later.")
+  )
   (junction (at 83.82 30.48) (diameter 0) (color 0 0 0 0)
   )
@@
     (effects (font (size 1.27 1.27)) (justify left bottom))
   )
-  (text "Licensed under the TAPR Open Hardware License (www.tapr.org/OHL)"
-    (at 20.32 194.31 0)
-    (effects (font (size 1.27 1.0795)) (justify left bottom))
-  )
   (text "Pull-down to disconnect\nVBUS in bootloader mode" (at 192.405 50.165 0)
     (effects (font (size 1.27 1.0795)) (justify left bottom))
@@
     (effects (font (size 1.27 1.0795)) (justify left bottom))
   )
-  (text "Repository: https://github.com/eez-open" (at 20.32 198.12 0)
-    (effects (font (size 1.27 1.0795)) (justify left bottom))
-  )
   (text "Vfb = 0.204 V" (at 71.12 47.625 0)
-    (effects (font (size 1.27 1.0795)) (justify left bottom))
-  )
-  (text "More info at http://www.envox.hr/eez" (at 20.32 196.215 0)
     (effects (font (size 1.27 1.0795)) (justify left bottom))
   )
@@
         )
       )
-    )
-  )
-  (symbol (lib_id "EEZ_DIB_MCU_r3B4-eagle-import:DINA4_L") (at 180.34 200.66 0) (unit 2)
-    (in_bom yes) (on_board yes) (dnp no)
-    (property "Reference" "#FRAME4" (at 180.34 200.66 0)
-      (effects (font (size 1.27 1.27)) hide)
-    )
-    (property "Value" "DINA4_L" (at 180.34 200.66 0)
-      (effects (font (size 1.27 1.27)) hide)
-    )
-    (property "Footprint" "EEZ_DIB_MCU_r3B4:" (at 180.34 200.66 0)
-      (effects (font (size 1.27 1.27)) hide)
-    )
-    (property "Datasheet" "" (at 180.34 200.66 0)
-      (effects (font (size 1.27 1.27)) hide)
-    )
-    (instances
-      (project "EEZ_DIB_MCU_r3B4"
-        (path "/58be380a-4a3a-4b30-b3f5-a03bc3bf2660/905201e7-921c-4a04-8e23-b281298c7e45"
-          (reference "#FRAME4") (unit 2)
-        )
-      )

Commit message: Adding temperary PCIe connector - adding logos
Changed lines of the file:
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@@
-    )
-  )
-  (symbol (lib_id "EEZ_DIB_MCU_r3B4-eagle-import:DINA4_L") (at -436.88 104.14 0) (unit 1)
-    (in_bom yes) (on_board yes) (dnp no)
-    (property "Reference" "#FRAME4" (at -436.88 104.14 0)
-      (effects (font (size 1.27 1.27)) hide)
-    )
-    (property "Value" "DINA4_L" (at -436.88 104.14 0)
-      (effects (font (size 1.27 1.27)) hide)
-    )
-    (property "Footprint" "EEZ_DIB_MCU_r3B4:" (at -436.88 104.14 0)
-      (effects (font (size 1.27 1.27)) hide)
-    )
-    (property "Datasheet" "" (at -436.88 104.14 0)
-      (effects (font (size 1.27 1.27)) hide)
-    )
-    (instances
-      (project "EEZ_DIB_MCU_r3B4"
-        (path "/58be380a-4a3a-4b30-b3f5-a03bc3bf2660/905201e7-921c-4a04-8e23-b281298c7e45"
-          (reference "#FRAME4") (unit 1)
-        )
-      )
     )
   )
