File: EEZ_BB3_CM4_SoM/EEZ_BB3_CM4_SoM.kicad_pcb (KiCad board)
At the start: 4 copper layers, 106 parts, among them IC15 N.C., IC16 DP83848CVV/NOPB, IC4 STM32F769IIT6, IC6 N.C., IC7 IS42S16400J, J10 DF40C-100DP-0.4V(51), J11 DF40C-100DP-0.4V(51), X4 N.C., Y1 25MHz, Y2 XTAL016178-85SMX

Commit message: Routing - new ioc
Parts:
- removed C10, C12: 18p, EEZ_DIB_MCU_r3B4:C0603
- removed C11, C13: 4p7, EEZ_DIB_MCU_r3B4:C0603
- removed C16, C17, C18, C19, C20, C21, C22, C23, C25, C26, C27, C28, C29, C30, C33, C36, C42, C43, C44, C45, C46, C47, C48, C60, C61, C62, C63, C64, C65, C67, C68, C69, C70, C71: 100n, EEZ_DIB_MCU_r3B4:C0603
- removed C24, C34, C35: 1u, EEZ_DIB_MCU_r3B4:C0805
- removed C31, C32, C37, C38: 2u2, EEZ_DIB_MCU_r3B4:C0805
- removed C39, C59: N.C., EEZ_DIB_MCU_r3B4:C0603
- removed C66: 10u, EEZ_DIB_MCU_r3B4:EC1206
- removed IC15, IC6: N.C., EEZ_DIB_MCU_r3B4:DRL6
- removed IC16: DP83848CVV/NOPB, EEZ_DIB_MCU_r3B4:PT48
- removed IC4: STM32F769IIT6, EEZ_DIB_MCU_r3B4:LQFP-176_24X24MM
- removed IC7: IS42S16400J, EEZ_DIB_MCU_r3B4:TSOPII-54
- removed JP10, JP11, JP12, JP5: JP2-CUT, EEZ_DIB_MCU_r3B4:JP2-CUT
- removed JP13, JP14: JP2-NOCUT, EEZ_DIB_MCU_r3B4:JP2-NOCUT
- removed JP3, JP4: ~, EEZ_DIB_MCU_r3B4:R_0805
- removed L1, L3: BLM18AG102SH1D, EEZ_DIB_MCU_r3B4:BEAD0603
- removed LED2: N.C., EEZ_DIB_MCU_r3B4:LED_0805
- removed R12, R15: 4K7, EEZ_DIB_MCU_r3B4:R0805
- removed R13: 10K, EEZ_DIB_MCU_r3B4:R0805
- removed R14, R19, R20, R21, R22, R41, R44, R45, R46: N.C., EEZ_DIB_MCU_r3B4:R0805
- removed R16, R17, R38: 1K5, EEZ_DIB_MCU_r3B4:R0805
- removed R18: 47R, EEZ_DIB_MCU_r3B4:R0805
- removed R39, R40, R43, R48: 49R9, EEZ_DIB_MCU_r3B4:R0805
- removed R42, R47, R49, R52, R53, R55: 2K2, EEZ_DIB_MCU_r3B4:R0805
- removed R50, R51: 220R, EEZ_DIB_MCU_r3B4:R0805
- removed R54: 4K87, EEZ_DIB_MCU_r3B4:R0805
- removed RN1, RN2, RN3, RN4, RN5, RN6, RN7: DR1206-33R-4/8, EEZ_DIB_MCU_r3B4:CAY16
- removed TP1: ~, EEZ_DIB_MCU_r3B4:PCB_SHIELD_TAB
- removed X4: N.C., EEZ_DIB_MCU_r3B4:SSW-106-02-S-S
- removed Y1: 25MHz, EEZ_DIB_MCU_r3B4:HC-49_4H
- removed Y2: XTAL016178-85SMX, EEZ_DIB_MCU_r3B4:85SMX
- moved J10 57.6 mm to (150.9, 81.0)
- moved J11 57.6 mm to (116.9, 81.0)
Routing:
- net GND: track 104.0 -> 0.00 mm, vias 29 -> 0
- net +3V3: track 53.4 -> 0.00 mm, vias 12 -> 0
- net UART_RX/DIN1: track 27.1 -> 0.00 mm, vias 2 -> 0
- net FMC_A12: track 22.0 -> 0.00 mm, vias 3 -> 0
- net FMC_BA1: track 21.5 -> 0.00 mm, vias 1 -> 0
- net FMC_SDCKE0: track 21.4 -> 0.00 mm, vias 1 -> 0
- net FMC_D2: track 20.9 -> 0.00 mm, vias 1 -> 0
- net FMC_D0: track 20.9 -> 0.00 mm, vias 1 -> 0
- net FMC_D8: track 20.9 -> 0.00 mm, vias 1 -> 0
- net FMC_D4: track 20.8 -> 0.00 mm, vias 1 -> 0
- net FMC_D6: track 20.8 -> 0.00 mm, vias 1 -> 0
- net FMC_NBL0: track 20.8 -> 0.00 mm, vias 1 -> 0
- net FMC_D5: track 20.8 -> 0.00 mm, vias 1 -> 0
- net FMC_D11: track 20.8 -> 0.00 mm, vias 1 -> 0
- net FMC_D7: track 20.7 -> 0.00 mm, vias 1 -> 0
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