File: EEZ_BB3_CM4_H7/H745 CM4 module.kicad_pcb (KiCad board)
At the start: 6 copper layers, 55.1 x 40 mm, 121 parts, among them IC12 LAN8742A-CZ-TR, IC2 STM32H745IIT6, IC3 AP1117-33, IC4 IS42S16400J, IC6 M24256-BWMN6TP, IC7 SZNUP4114HMR6T1G, IC8 IP4252CZ8-4-TTL,13, J1 DF40C-100DP-0.4V(51), J2 DF40C-100DP-0.4V(51), X1 SSW-106-02-S-S, Y1 XTAL016178-85SMX

Commit message: Routing
Parts:
- added R5: 47K, Library:R_0402_1005Metric, F.Cu at (128.2, 107.8)
- added R6: 47K, Library:R_0402_1005Metric, F.Cu at (129.2, 107.8)
- IC2: value STM32H745IIT6 -> STM32H757IIT6
- IC8, R18, R19: moved to F.Cu
- moved L6 31.2 mm to (156.6, 89.8), turned to -90 degrees
- moved C63 23.7 mm to (156.9, 87.3)
- moved C68 23.7 mm to (155.9, 87.3)
- moved R35 12.8 mm to (121.1, 93.1), turned to -90 degrees
- moved R36 12.4 mm to (122.5, 95.1), turned to -90 degrees
- moved R34 11.7 mm to (125.5, 95.8)
- moved R33 11.7 mm to (125.5, 96.8)
- moved C62 11.3 mm to (123.2, 89.7), turned to 180 degrees
- moved C29 11.2 mm to (128.0, 70.7)
- moved R15 11.2 mm to (129.0, 70.7)
- moved R19 11.0 mm to (121.7, 108.7), turned to 0 degrees
- moved R18 11.0 mm to (121.8, 107.7), turned to 180 degrees
- moved C67 10.6 mm to (123.2, 88.7), turned to 0 degrees
- moved R29 10.4 mm to (123.2, 90.8), turned to 0 degrees
- moved R28 9.91 mm to (131.2, 93.5), turned to 0 degrees
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Connections:
- C33 pad 2: /STM32H7 MCU/VSSA -> /STM32H7 MCU/VDD_SDC
- C34 pad 2: /STM32H7 MCU/VSSA -> /STM32H7 MCU/VDD_SDC
- IC2 pad 101: SLAVE4_TX -> unconnected-(IC2C-VCAPDSI.101-Pad101)
- IC2 pad 102: SLAVE4_RX -> unconnected-(IC2C-VDD12DSI.102-Pad102)
- IC2 pad 103: LTDC_G3 -> DSI0_D0_P
- IC2 pad 104: LTDC_G4 -> DSI0_D0_N
- IC2 pad 105: +VDD_MCU -> GND
- IC2 pad 106: GND -> DSI0_C_P
- IC2 pad 107: LTDC_G5 -> DSI0_C_N
- IC2 pad 108: LTDC_G6 -> unconnected-(IC2C-VDD12DSI.108-Pad108)
- IC2 pad 109: LTDC_G7 -> GND
- IC2 pad 38: /STM32H7 MCU/VSSA -> /STM32H7 MCU/VDD_SDC
- IC8 pad 5: /SDRAM, JTAG, SD card, EEPROM/DAT0 -> SD_DAT0
- IC8 pad 6: /SDRAM, JTAG, SD card, EEPROM/CLK -> SD_CLK
- IC8 pad 7: /SDRAM, JTAG, SD card, EEPROM/CMD -> SD_CMD
- J1 pad 57: GPIO15 -> SD_CLK
- J1 pad 61: GPIO14 -> SD_DAT3
- J1 pad 62: GPIO27 -> SD_CMD
- J1 pad 63: GPIO4 -> SD_DAT0
- J1 pad 67: GPIO3 -> SD_DAT1
- J1 pad 69: GPIO2 -> SD_DAT2
- J2 pad 3: USB_N -> USB_OTG_HS_D_N
- J2 pad 5: USB_P -> USB_OTG_HS_D_P
- NT2 pad 2: /STM32H7 MCU/VSSA -> /STM32H7 MCU/VDD_SDC
Routing:
- net DSI0_D0_P: track 0.00 -> 41.5 mm, vias 0 -> 1
- net DSI0_D0_N: track 0.00 -> 39.8 mm, vias 0 -> 1
- net DSI0_C_N: track 0.00 -> 39.0 mm, vias 0 -> 1
- net DSI0_C_P: track 0.00 -> 37.9 mm, vias 0 -> 1
- net USB_OTG_HS_D_P: track 0.00 -> 35.2 mm, vias 0 -> 1
- net USB_OTG_HS_D_N: track 0.00 -> 34.1 mm, vias 0 -> 1
- net /Ethernet PHY, Audio, DACs/+3V3_LAN: track 0.00 -> 28.6 mm, vias 0 -> 8
- net ETH_REF_CLK: track 0.00 -> 27.7 mm, vias 0 -> 1
- net ETH_nLED2: track 0.00 -> 27.3 mm, vias 0 -> 2
- net ETH_nLED1: track 0.00 -> 27.2 mm, vias 0 -> 2
- net ~{RESET}: track 0.00 -> 25.7 mm, vias 0 -> 1
- net ETH_TXD1: track 0.00 -> 25.3 mm, vias 0 -> 1
- net ETH_0P: track 0.00 -> 24.3 mm, vias 0 -> 2
- net ETH_MDC: track 0.00 -> 23.8 mm, vias 0 -> 1
- net RCC_MCO_2: track 0.00 -> 23.7 mm, vias 0 -> 1
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
Commit message: Routing
Parts:
- C42, C44: moved to B.Cu
- moved R19 24.7 mm to (146.1, 104.9), turned to 180 degrees
- moved R18 24.7 mm to (146.1, 103.8)
- moved IC8 10.5 mm to (135.0, 107.7)
- moved C42 6.27 mm to (140.1, 103.2), turned to 90 degrees
- moved R5 4.38 mm to (132.5, 108.4), turned to 180 degrees
- moved C27 2.08 mm to (126.5, 103.3)
- moved C44 2.07 mm to (133.5, 105.6)
- moved R16 0.97 mm to (146.0, 100.7)
- moved R14 0.92 mm to (146.1, 102.8)
- moved C66 0.87 mm to (139.4, 107.6)
- moved C12 0.58 mm to (132.5, 105.7), turned to -90 degrees
Routing:
- net FMC_SDNCAS: track 0.00 -> 37.1 mm, vias 0 -> 2
- net /STM32H7 MCU/VDD_SDC: track 7.85 -> 42.3 mm, vias 1 -> 6
- net SDMMC1_CMD: track 0.00 -> 27.6 mm, vias 0 -> 2
- net /SDRAM, JTAG, SD card, EEPROM/TCK: track 0.00 -> 24.4 mm
- net /SDRAM, JTAG, SD card, EEPROM/TMS: track 0.00 -> 21.0 mm
- net SD_DAT0: track 0.00 -> 15.6 mm, vias 0 -> 1
- net SDMMC1_CK: track 0.00 -> 15.1 mm, vias 0 -> 2
- net SYS_SCL: track 0.00 -> 14.6 mm, vias 0 -> 1
- net GND: track 46.8 -> 60.9 mm, vias 57 -> 71
- net SD_CLK: track 0.00 -> 12.7 mm, vias 0 -> 1
- net SDMMC1_D0: track 0.00 -> 11.9 mm
- net SYS_SDA: track 0.00 -> 10.6 mm, vias 0 -> 1
- net /SDRAM, JTAG, SD card, EEPROM/SWD_NRST: track 0.00 -> 10.3 mm
- net CM4_3.3V: track 126.2 -> 135.7 mm, vias 16 -> 28
- net SD_CMD: track 0.00 -> 9.21 mm, vias 0 -> 1
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
Commit message: Adding GPIO connections
Connections:
- net IOEXP_SPI_MOSI renamed ~{FAULT}
- net RS485_TX_EN renamed PWR_SSTART
- net SLAVE2_RX renamed RTC_REF
- net SLAVE2_RX_OE renamed PWR_DIRECT
- C29 pad 2: ~{RESET} -> nEXTRST
- IC2 pad 1: IOEXP_GPIO0 -> GPIO21
- IC2 pad 110: IOEXP_GPIO3 -> ENC_SW
- IC2 pad 116: LTDC_R7 -> GPIO23
- IC2 pad 117: LTDC_CLK -> SD_DETECT
- IC2 pad 122: LTDC_HSYNC -> ENC_A
- IC2 pad 123: TFT_BRIGHTNESS -> ENC_B
- IC2 pad 127: LTDC_B3 -> GPIO6
- IC2 pad 128: RS485_TX -> unconnected-(IC2A-PA9-Pad128)
- IC2 pad 129: RS485_RX -> USB_OTG_ID
- IC2 pad 130: LTDC_R4 -> USB_OTG_HS_D_N
- IC2 pad 131: LTDC_R5 -> USB_OTG_HS_D_P
- IC2 pad 139: SLAVE3_TX -> GPIO22
- IC2 pad 140: IOEXP_SPI_CLK -> unconnected-(IC2A-PC10-Pad140)
- IC2 pad 141: SLAVE1_RX -> unconnected-(IC2A-PC11-Pad141)
- IC2 pad 146: ~{MTR_EN} -> unconnected-(IC2A-PD3-Pad146)
- IC2 pad 147: SLAVE4_RX_OE -> unconnected-(IC2A-PD4-Pad147)
- IC2 pad 148: SLAVE3_RX_OE -> DOUT2
- IC2 pad 150: SLAVE1_RX_OE -> GPIO4
- IC2 pad 153: IRQ_IOEXP8 -> unconnected-(IC2B-PG9-Pad153)
- IC2 pad 154: ~{MTR_BRK} -> unconnected-(IC2B-PG10-Pad154)
- IC2 pad 156: LTDC_B4 -> GPIO26
- IC2 pad 163: IOEXP_SPI_MISO -> GPIO8
- IC2 pad 164: BTM_FAN_PWM -> unconnected-(IC2A-PB5-Pad164)
- IC2 pad 165: IOEXP_I2C1_SCL -> I2C1_SCL
- IC2 pad 166: IOEXP_I2C1_SDA -> I2C1_SDA
- IC2 pad 167: /STM32H7 MCU/BOOT0 -> BOOT0
- IC2 pad 168: LTDC_B6 -> ID_SC
- IC2 pad 169: LTDC_B7 -> GPIO27
- IC2 pad 174: /STM32H7 MCU/PDR_ON -> BOOT0
- IC2 pad 2: ~{IOEXP_RESET} -> GPIO17
- IC2 pad 26: SLAVE3_RX -> GPIO12
- IC2 pad 27: TEST_24V_AIN -> GPIO15
- IC2 pad 28: TOP_FAN_PWM -> GPIO13
- IC2 pad 29: RAY_TMP -> GPIO14
- IC2 pad 3: PANIC_SW -> GPIO18
- IC2 pad 30: LTDC_DE -> unconnected-(IC2B-PF10-Pad30)
- IC2 pad 33: ~{RESET} -> nEXTRST
- IC2 pad 4: IOEXP_GPIO1 -> GPIO19
- IC2 pad 41: SLAVE1_TX -> ID_SD
- IC2 pad 46: LTDC_B5 -> DIN2
- IC2 pad 49: LTDC_VSYNC -> DAC_OUT1
- IC2 pad 5: IOEXP_GPIO2 -> GPIO20
- IC2 pad 51: LTDC_G2 -> unconnected-(IC2A-PA6-Pad51)
- IC2 pad 55: LTDC_R3 -> unconnected-(IC2A-PB0-Pad55)
- IC2 pad 56: LTDC_R6 -> unconnected-(IC2A-PB1-Pad56)
- IC2 pad 78: IOEXP_I2C2_SCL -> unconnected-(IC2A-PB10-Pad78)
- IC2 pad 79: IOEXP_I2C2_SDA -> unconnected-(IC2A-PB11-Pad79)
- IC2 pad 86: SLAVE2_TX -> GPIO11
- IC2 pad 87: USB_OTG_HS_D_N -> GPIO9
- IC2 pad 88: USB_OTG_HS_D_P -> GPIO10
- IC2 pad 94: IRQ_TOUCH -> GPIO7
- IC2 pad 95: SYS_SCL -> TFT_BRIGHTNESS
- IC2 pad 96: SYS_SDA -> OE_SYNC
- IC6 pad 5: SYS_SDA -> I2C1_SDA
- IC6 pad 6: SYS_SCL -> I2C1_SCL
- J1 pad 29: GPIO16 -> DOUT2
- J1 pad 34: GPIO5 -> DAC_OUT1
- J1 pad 41: GPIO25 -> DIN2
- J1 pad 45: GPIO24 -> ENC_SW
- J1 pad 56: GPIO3 -> ENC_B
- J1 pad 58: GPIO2 -> ENC_A
- J1 pad 80: SCL0 -> I2C1_SCL
- J1 pad 82: SDA0 -> I2C1_SDA
- JP1 pad COM: /STM32H7 MCU/PDR_ON -> BOOT0
- R1 pad 2: IOEXP_I2C1_SCL -> I2C1_SCL
- R11 pad 2: /STM32H7 MCU/BOOT0 -> BOOT0
- R3 pad 2: IOEXP_I2C1_SDA -> I2C1_SDA
Routing:
- net unconnected-(IC2A-PB11-Pad79): vias 0 -> 1
- net unconnected-(IC2A-PB10-Pad78): vias 0 -> 1
- net SYS_SDA: vias 1 -> 0
- net SYS_SCL: vias 1 -> 0
- net IOEXP_I2C2_SDA: vias 1 -> 0
- net IOEXP_I2C2_SCL: vias 1 -> 0
- net I2C1_SDA: vias 0 -> 1
- net I2C1_SCL: vias 0 -> 1

Commit message: Routing adding ioc
Parts:
- moved R13 1.93 mm to (123.2, 76.7)
- moved C8 1.72 mm to (112.3, 78.8)
- moved L2 1.63 mm to (121.5, 76.8)
- moved C36 0.98 mm to (116.7, 77.2)
- moved C19 0.97 mm to (116.7, 78.2)
- moved C35 0.90 mm to (118.6, 77.0)
- moved C28 0.16 mm to (122.2, 103.2)
Connections:
- IC2 pad 111: PWR_SSTART -> GPIO27
- IC2 pad 140: unconnected-(IC2A-PC10-Pad140) -> GPIO8
- IC2 pad 146: unconnected-(IC2A-PD3-Pad146) -> GPIO4
- IC2 pad 149: PWR_DIRECT -> unconnected-(IC2A-PD6-Pad149)
- IC2 pad 150: GPIO4 -> unconnected-(IC2A-PD7-Pad150)
- IC2 pad 155: ETH_TX_EN -> GPIO15
- IC2 pad 156: GPIO26 -> unconnected-(IC2B-PG12-Pad156)
- IC2 pad 163: GPIO8 -> GPIO13
- IC2 pad 164: unconnected-(IC2A-PB5-Pad164) -> GPIO14
- IC2 pad 169: GPIO27 -> unconnected-(IC2A-PB9-Pad169)
- IC2 pad 27: GPIO15 -> unconnected-(IC2B-PF7-Pad27)
- IC2 pad 28: GPIO13 -> unconnected-(IC2B-PF8-Pad28)
- IC2 pad 29: GPIO14 -> unconnected-(IC2B-PF9-Pad29)
- IC2 pad 51: unconnected-(IC2A-PA6-Pad51) -> GPIO26
- IC2 pad 55: unconnected-(IC2A-PB0-Pad55) -> CAM0_D1_N
- IC2 pad 56: unconnected-(IC2A-PB1-Pad56) -> CAM0_D1_P
- IC2 pad 57: ~{FAULT} -> CAM0_C_P
- IC2 pad 79: unconnected-(IC2A-PB11-Pad79) -> ETH_TX_EN
- IC2 pad 85: RTC_REF -> CAM0_C_N
- IC2 pad 9: WDG -> AnalogIP1
- IC2 pad 95: TFT_BRIGHTNESS -> CAM0_D0_N
- IC2 pad 96: OE_SYNC -> CAM0_D0_P
- J1 pad 75: SD_PWR_ON -> SD_DETECT
- J1 pad 93: nRPIBOOT -> BOOT0
- J1 pad 96: AnalogIP0 -> AUDIO_OUT
- R6 pad 2: SD_PWR_ON -> SD_DETECT
Routing:
- net GPIO20: track 0.00 -> 58.6 mm, vias 0 -> 1
- net GPIO21: track 0.00 -> 57.8 mm, vias 0 -> 1
- net ID_SD: track 0.00 -> 52.9 mm, vias 0 -> 5
- net GPIO19: track 0.00 -> 52.2 mm, vias 0 -> 1
- net GPIO13: track 0.00 -> 43.8 mm, vias 0 -> 1
- net DOUT2: track 0.00 -> 43.3 mm, vias 0 -> 2
- net GPIO12: track 0.00 -> 40.9 mm, vias 0 -> 3
- net CAM0_D0_P: track 0.00 -> 37.8 mm, vias 0 -> 1
- net DAC_OUT1: track 0.00 -> 37.7 mm, vias 0 -> 3
- net CAM0_D0_N: track 0.00 -> 37.5 mm, vias 0 -> 1
- net CAM0_C_N: track 0.00 -> 35.4 mm, vias 0 -> 1
- net GPIO6: track 0.00 -> 30.2 mm, vias 0 -> 3
- net GPIO26: track 0.00 -> 29.4 mm, vias 0 -> 2
- net USB_OTG_HS_D_N: track 34.1 -> 58.7 mm, vias 1 -> 2
- net USB_OTG_HS_D_P: track 35.2 -> 58.6 mm, vias 1 -> 2
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
Commit message: Routing - new ioc
Parts:
- removed R2, R4: 1K5, Library:R_0402_1005Metric
- moved R15 25.2 mm to (139.4, 93.7), turned to 0 degrees
- moved C29 9.28 mm to (126.1, 79.8)
- moved C40 4.34 mm to (136.9, 77.7), turned to 0 degrees
- moved L4 3.49 mm to (135.4, 79.3), turned to 0 degrees
- moved C33 0.33 mm to (120.9, 81.2)
- moved C42 0.26 mm to (139.8, 103.1)
- moved C18 0.23 mm to (138.9, 103.1)
- turned IC6 to 0 degrees
Routing:
- net USB_OTG_ID: track 0.00 -> 59.6 mm, vias 0 -> 2
- net GPIO18: track 0.00 -> 58.8 mm, vias 0 -> 2
- net AUDIO_OUT: track 0.00 -> 58.6 mm, vias 0 -> 1
- net ID_SC: track 0.00 -> 57.2 mm, vias 0 -> 1
- net GPIO17: track 0.00 -> 54.1 mm, vias 0 -> 2
- net DIN2: track 0.00 -> 47.0 mm, vias 0 -> 3
- net GPIO14: track 0.00 -> 43.1 mm, vias 0 -> 2
- net GPIO8: track 0.00 -> 32.9 mm, vias 0 -> 2
- net GPIO4: track 0.00 -> 30.4 mm, vias 0 -> 2
- net ENC_A: track 0.00 -> 26.9 mm, vias 0 -> 3
- net GPIO22: track 0.00 -> 26.4 mm, vias 0 -> 2
- net ENC_B: track 0.00 -> 25.7 mm, vias 0 -> 3
- net I2C1_SCL: track 0.00 -> 23.0 mm, vias 0 -> 1
- net GPIO23: track 0.00 -> 21.2 mm, vias 0 -> 3
- net I2C1_SDA: track 0.00 -> 20.0 mm, vias 0 -> 1
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
Commit message: Routing
Parts:
- moved C66 0.89 mm to (140.0, 108.3)
- moved C9 0.48 mm to (135.9, 103.2)
- moved R3 0.37 mm to (142.2, 86.9)
- moved R11 0.36 mm to (142.2, 85.9)
- moved C42 0.32 mm to (140.2, 103.0)
- moved C18 0.31 mm to (139.2, 103.0)
Routing:
- net GPIO15: track 0.88 -> 39.3 mm, vias 1 -> 2
- net BOOT0: track 0.00 -> 37.6 mm, vias 0 -> 3
- net AnalogIP1: track 0.00 -> 35.8 mm, vias 0 -> 2
- net nEXTRST: track 0.00 -> 35.0 mm, vias 0 -> 2
- net I2C1_SDA: track 20.0 -> 38.2 mm, vias 1 -> 4
- net SD_DETECT: track 5.10 -> 20.2 mm, vias 1 -> 4
- net I2C1_SCL: track 23.0 -> 37.7 mm, vias 1 -> 4
- net ~{RESET}: track 25.3 -> 39.4 mm, vias 1 -> 3
- net ENC_B: track 25.7 -> 29.1 mm
- net GPIO13: track 42.0 -> 45.4 mm, vias 1 -> 2
- net RCC_MCO_2: track 25.7 -> 28.6 mm
- net FMC_SDNCAS: track 36.6 -> 39.1 mm
- net GND: track 74.5 -> 76.7 mm, vias 82 -> 87
- net GPIO12: track 41.0 -> 39.0 mm
- net SDMMC1_CMD: track 29.2 -> 27.3 mm
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
Commit message: Routing
Parts:
- moved L6 31.2 mm to (125.5, 87.6), turned to 90 degrees
- moved R31 1.28 mm to (126.8, 88.1)
- moved R32 1.27 mm to (127.8, 88.1)
- moved C60 1.27 mm to (129.8, 88.1)
- moved R27 1.26 mm to (128.8, 88.1)
- moved C61 1.26 mm to (130.8, 88.1)
- moved C65 0.49 mm to (121.8, 87.0)
- moved C26 0.13 mm to (142.1, 101.8)
Routing:
- net CM4_3.3V: track 132.2 -> 192.4 mm, vias 25 -> 35
- net /STM32H7 MCU/VDD_SDC: track 33.8 -> 91.1 mm, vias 6 -> 10
- net +VDD_MCU: track 38.2 -> 61.2 mm, vias 16 -> 20
- net /SDRAM, JTAG, SD card, EEPROM/SWD_NRST: track 10.3 -> 17.1 mm
- net /STM32H7 MCU/VREF+: track 9.31 -> 14.1 mm, vias 2 -> 3
- net /STM32H7 MCU/VDDA: track 4.97 -> 9.54 mm, vias 0 -> 1
- net /STM32H7 MCU/VBAT: track 0.00 -> 3.56 mm, vias 0 -> 1
- net GPIO4: track 29.9 -> 27.1 mm
- net DOUT2: track 45.1 -> 42.9 mm
- net /SDRAM, JTAG, SD card, EEPROM/TMS: track 21.0 -> 19.1 mm, vias 0 -> 1
- net ETH_nLED1: track 26.6 -> 27.9 mm
- net SYS_JTDO-SWO: track 8.09 -> 9.29 mm, vias 0 -> 1
- net ID_SC: track 57.2 -> 56.0 mm
- net /Ethernet PHY, Audio, DACs/RXD1_IN: track 13.0 -> 14.0 mm
- net /Ethernet PHY, Audio, DACs/ETH_CLK_IN: track 1.45 -> 2.26 mm
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
Commit message: Routing
Parts:
- removed C30: CE5R5105HF-ZJ (1F), Library:CE5R5105HF-ZJ
- moved C63 36.6 mm to (120.4, 89.1)
- moved C68 34.6 mm to (121.4, 89.1)
- moved C15 1.68 mm to (133.6, 81.3)
- moved C37 0.80 mm to (133.4, 75.4)
- moved C39 0.76 mm to (131.3, 75.4)
- moved C20 0.23 mm to (125.7, 103.2)
- moved C27 0.22 mm to (126.7, 103.2)
- moved RN6 0.11 mm to (123.4, 84.1)
Connections:
- R12 pad 1: Net-(C30-Pad+) -> HDMI0_SCL
Routing:
- net GND: track 77.4 -> 136.9 mm, vias 89 -> 146
- net CM4_3.3V: track 192.4 -> 236.1 mm
- net +VDD_MCU: track 61.2 -> 82.2 mm, vias 20 -> 22
- net HDMI0_SCL: track 0.00 -> 17.7 mm, vias 0 -> 1
- net ~{RESET}: track 39.4 -> 25.4 mm, vias 3 -> 2
- net SYS_JTDO-SWO: track 9.29 -> 20.4 mm
- net /STM32H7 MCU/VBAT: track 3.56 -> 11.6 mm, vias 1 -> 2
- net /SDRAM, JTAG, SD card, EEPROM/TCK: track 24.7 -> 19.0 mm, vias 0 -> 1
- net /Ethernet PHY, Audio, DACs/+3V3_LAN: track 32.4 -> 37.9 mm, vias 8 -> 9
- net BOOT0: track 37.6 -> 41.7 mm, vias 3 -> 4
- net /STM32H7 MCU/VDD_SDC: track 91.1 -> 94.5 mm
- net ID_SC: track 56.0 -> 53.0 mm
- net CAM0_C_N: track 36.7 -> 34.0 mm
- net nEXTRST: track 35.0 -> 37.2 mm, vias 2 -> 3
- net /STM32H7 MCU/VLXSMPS: track 3.23 -> 4.80 mm
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