File: EEZ_BB3_CM4_H7/H745 CM4 module.kicad_pcb (KiCad board)
At the start: 6 copper layers, 55.1 x 40 mm, 120 parts, among them IC12 LAN8742A-CZ-TR, IC2 STM32H757IIT6, IC3 AP1117-33, IC4 IS42S16400J, IC6 M24256-BWMN6TP, IC7 SZNUP4114HMR6T1G, IC8 IP4252CZ8-4-TTL,13, J1 DF40C-100DP-0.4V(51), J2 DF40C-100DP-0.4V(51), X1 SSW-106-02-S-S, Y1 XTAL016178-85SMX

Commit message: Fixing errors - adding README
Parts:
- moved C66 0.78 mm to (140.6, 107.8)
Routing:
- net GPIO4: track 27.1 -> 26.0 mm, vias 2 -> 1
- net FMC_SDNCAS: track 39.1 -> 40.2 mm
- net unconnected-(IC2A-PB10-Pad78): track 1.05 -> 0.00 mm, vias 1 -> 0
- net CM4_3.3V: track 236.1 -> 236.9 mm, vias 35 -> 34
- net USB_OTG_HS_D_N: track 59.4 -> 59.9 mm
- net GND: track 136.9 -> 136.5 mm, vias 146 -> 148
