File: EEZ_BB3_CM4_H7/H745 CM4 module.kicad_pcb (KiCad board)
At the start: 6 copper layers, 55.1 x 40 mm, 120 parts, among them IC12 LAN8742A-CZ-TR, IC2 STM32H757IIT6, IC3 AP1117-33, IC4 IS42S16400J, IC6 M24256-BWMN6TP, IC7 SZNUP4114HMR6T1G, IC8 IP4252CZ8-4-TTL,13, J1 DF40C-100DP-0.4V(51), J2 DF40C-100DP-0.4V(51), X1 SSW-106-02-S-S, Y1 XTAL016178-85SMX

Commit message: Fix #6
Parts:
- added C1: 100n, Library:C_0402_1005Metric, F.Cu at (125.9, 106.9)
- added C2: 2u2, Library:C_0402_1005Metric, F.Cu at (124.8, 107.8)
- moved R6 0.45 mm to (129.0, 108.2)
Connections:
- IC2 pad 101: unconnected-(IC2C-VCAPDSI.101-Pad101) -> /STM32H7 MCU/VDD_DSI
- IC2 pad 102: unconnected-(IC2C-VDD12DSI.102-Pad102) -> /STM32H7 MCU/VDD_DSI
- IC2 pad 108: unconnected-(IC2C-VDD12DSI.108-Pad108) -> /STM32H7 MCU/VDD_DSI
Routing:
- net /STM32H7 MCU/VDD_DSI: track 0.00 -> 9.93 mm
- net GND: track 136.5 -> 142.1 mm, vias 148 -> 147
- net GPIO27: track 15.1 -> 17.6 mm
- net /Ethernet PHY, Audio, DACs/RXD0_IN: track 13.6 -> 15.4 mm
- net AUDIO_OUT: track 59.6 -> 61.2 mm
- net GPIO4: track 26.0 -> 27.1 mm
- net CAM0_D0_P: track 37.0 -> 38.0 mm
- net SD_DAT0: track 15.8 -> 14.9 mm
- net DIN2: track 47.6 -> 46.7 mm
- net SD_CLK: track 12.9 -> 12.1 mm
- net GPIO22: track 26.3 -> 27.1 mm
- net CM4_3.3V: track 236.9 -> 237.6 mm
- net SD_DETECT: track 20.2 -> 19.6 mm
- net GPIO7: track 9.04 -> 8.48 mm
- net GPIO19: track 55.7 -> 56.2 mm

Commit message: Updating pinout
Parts:
- moved FI3 0.23 mm to (147.5, 110.9)
- moved FI5 0.23 mm to (147.5, 110.9)
- moved FI1 0.22 mm to (95.6, 73.6)
- moved FI4 0.17 mm to (147.7, 73.6)
- moved FI2 0.13 mm to (95.7, 110.8)
- moved FI6 0.13 mm to (95.7, 110.8)
Routing:
- net GPIO12: track 39.0 -> 31.9 mm
- net ETH_TXD0: track 21.0 -> 18.4 mm
- net ETH_TXD1: track 23.0 -> 20.4 mm
- net HDMI0_SCL: track 17.7 -> 16.8 mm
- net ID_SD: track 55.6 -> 54.8 mm
- net I2C1_SCL: track 37.0 -> 36.3 mm

Commit message: Adding USB
Parts:
- removed R10: 1K5, Library:R_0402_1005Metric
- added C3: 4u7, Library:EC1206, F.Cu at (140.1, 74.5)
- added IC1: TPS2051BDBVR, Envox H745 Master MCU r2B6:DBV5, B.Cu at (138.7, 74.8)
- added R2: 10K, Library:R_0402_1005Metric, B.Cu at (139.8, 76.9)
- added R4: 10K, Library:R_0402_1005Metric, B.Cu at (135.9, 74.4)
- R7: value 1K5 -> 4K7
- moved R7 33.8 mm to (141.5, 74.2)
- moved C21 0.55 mm to (129.4, 76.4)
Connections:
- IC2 pad 128: unconnected-(IC2A-PA9-Pad128) -> HDMI0_CLK_P
- IC2 pad 141: unconnected-(IC2A-PC11-Pad141) -> HDMI0_TX0_N
- IC2 pad 147: unconnected-(IC2A-PD4-Pad147) -> HDMI0_TX0_P
- IC2 pad 149: unconnected-(IC2A-PD6-Pad149) -> DOUT3
- IC2 pad 150: unconnected-(IC2A-PD7-Pad150) -> DIN3
- IC2 pad 156: unconnected-(IC2B-PG12-Pad156) -> ETH_TXD1
- IC2 pad 158: ETH_TXD1 -> unconnected-(IC2B-PG14-Pad158)
- IC2 pad 26: GPIO12 -> CAM1_D0_N
- IC2 pad 27: unconnected-(IC2B-PF7-Pad27) -> CAM1_D0_P
- IC2 pad 28: unconnected-(IC2B-PF8-Pad28) -> CAM1_D1_N
- IC2 pad 29: unconnected-(IC2B-PF9-Pad29) -> GPIO12
- J2 pad 76: HDMI0_TX1_P -> DOUT3
- J2 pad 78: HDMI0_TX1_N -> DIN3
- R7 pad 1: CM4_3.3V -> Net-(IC1-OUT)
- R7 pad 2: SYS_SDA -> HDMI0_CLK_P
Routing:
- net HDMI0_CLK_P: track 0.00 -> 41.8 mm, vias 0 -> 2
- net HDMI0_TX0_P: track 0.00 -> 37.6 mm, vias 0 -> 2
- net HDMI0_TX0_N: track 0.00 -> 37.2 mm, vias 0 -> 2
- net DOUT3: track 0.00 -> 37.2 mm, vias 0 -> 2
- net DIN3: track 0.00 -> 35.1 mm, vias 0 -> 2
- net CAM1_D0_P: track 0.00 -> 25.0 mm, vias 0 -> 2
- net CAM1_D0_N: track 0.00 -> 22.0 mm, vias 0 -> 2
- net CAM1_D1_N: track 0.00 -> 20.9 mm, vias 0 -> 2
- net GPIO12: track 31.9 -> 39.6 mm
- net CM4_3.3V: track 237.6 -> 230.6 mm, vias 34 -> 32
- net ETH_TXD0: track 18.4 -> 21.0 mm
- net ETH_TXD1: track 20.4 -> 21.5 mm
- net +VDD_MCU: track 82.2 -> 83.0 mm
- net nEXTRST: track 37.2 -> 36.6 mm
- net /STM32H7 MCU/VDD_SDC: track 94.5 -> 95.0 mm
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
Commit message: Routing
Routing:
- net +5V: track 40.1 -> 125.4 mm, vias 2 -> 3
- net +VDD_MCU: track 83.0 -> 105.1 mm, vias 22 -> 23
- net HDMI0_CLK_P: track 41.8 -> 54.5 mm, vias 2 -> 3
- net HDMI0_SCL: track 16.8 -> 27.6 mm
- net HDMI0_TX0_P: track 37.6 -> 46.2 mm, vias 2 -> 3
- net HDMI0_TX0_N: track 37.2 -> 45.7 mm, vias 2 -> 3
- net GND: track 142.2 -> 148.0 mm, vias 147 -> 151
- net CM4_3.3V: track 230.6 -> 234.9 mm
- net Net-(IC1-OUT): track 0.00 -> 3.24 mm, vias 0 -> 1
- net /STM32H7 MCU/VDD_SDC: track 95.0 -> 97.3 mm
- net AnalogIP1: track 36.0 -> 37.8 mm
- net /Ethernet PHY, Audio, DACs/+3V3_LAN: track 38.4 -> 37.7 mm

Commit message: Moving components - moving EEZ logo to top
Parts:
- added G***: LOGO, EEZ:eez, F.Cu at (120.3, 108.9)
- moved R4 6.60 mm to (142.5, 74.2), turned to -90 degrees
- moved REF** 3.52 mm to (114.4, 109.3)
- moved C11 0.85 mm to (114.2, 105.4)
- moved C14 0.84 mm to (113.5, 103.9)
Routing:
- net GND: track 148.0 -> 147.4 mm
- net HDMI0_CLK_P: track 54.5 -> 54.8 mm, vias 3 -> 2

Commit message: Removing logo from back
Parts:
- removed the G*** at (106.1, 76.4)
