File: EEZ_BB3_CM4_H7/SDRAM,_JTAG,_SD_card,_EEPROM.kicad_sch (KiCad schematic)
At the start: 25 parts, among them IC4 IS42S16400J, IC6 M24256-BWMN6TP, IC7 SZNUP4114HMR6T1G, IC8 IP4252CZ8-4-TTL,13, X1 SSW-106-02-S-S, X2 TC2030-IDC

Commit message: Routing
Parts:
- added R5, R6: 47K, Library:R_0402_1005Metric, symbol Library:Envox_R-EU_R0402
Connections:
- net +3V3: now also R5.2, R6.1
- net SD_DETECT: now also R5.1
- net CLK renamed SD_CLK
- net CMD renamed SD_CMD
- net DAT0 renamed SD_DAT0
- net SYS_SCL renamed I2C1_SCL
- net SYS_SDA renamed I2C1_SDA
- new net SD_PWR_ON: R6.2

Commit message: Adding USB
Parts:
- added C52: 4u7, Library:EC1206, symbol EEZ_DIB_MCU_r3B4-eagle-import:ECAP1206
- added IC11: TPS2051BDBVR, Envox H745 Master MCU r2B6:DBV5, symbol EEZ_DIB_MCU_r3B4-eagle-import:TPS2051B
- added R28, R34: 10K, Library:R_0402_1005Metric, symbol EEZ_DIB_MCU_r3B4-eagle-import:R-EU_R0805
- added R31: 4K7, Library:R_0402_1005Metric, symbol EEZ_DIB_MCU_r3B4-eagle-import:R-EU_R0805
Connections:
- net GND: now also C52.-, IC11.2 (GND), R28.1, R34.2
- new net: C52.+, IC11.1 (OUT), R31.1
- new net +5V: IC11.5 (IN)
- new net USB_OTG_FS_OC: IC11.3 (~{OC})
- new net USB_OTG_FS_PSO: IC11.4 (EN), R28.2
- new net USB_OTG_FS_VBUS: R31.2, R34.1
Other:
- note added: "Pull-down to disconnect VBUS in bootloader mode"
- note added: "Tant."
- note added: "USB OTG port"
- note removed: "Watchdog/supervisor"

Commit message: Removing picture
Parts:
- renumbered C52 to C3, IC11 to IC1, R28 to R2, R34 to R4, R31 to R7

Commit message: Moving components - moving EEZ logo to top
Changed lines of the file:
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@@
-    )
-  )
-  (global_label "SD_DAT1" (shape input) (at 258.064 97.536 0)
-    (effects (font (size 1.524 1.524)) (justify left))
-    (property "Intersheetrefs" "${INTERSHEET_REFS}" (at 258.064 97.536 0)
-      (effects (font (size 1.27 1.27)) hide)
-    )
-  )
-  (global_label "SD_DAT2" (shape input) (at 258.064 100.584 0)
-    (effects (font (size 1.524 1.524)) (justify left))
-    (property "Intersheetrefs" "${INTERSHEET_REFS}" (at 258.064 100.584 0)
-      (effects (font (size 1.27 1.27)) hide)
-    )
-  )
-  (global_label "USB_OTG_FS_D_P" (shape bidirectional) (at 162.56 132.08 180) (fields_autoplaced)
-    (effects (font (size 0.889 0.889)) (justify right))
-    (property "Intersheetrefs" "${INTERSHEET_REFS}" (at 335.28 203.2 0)
-      (effects (font (size 1.27 1.27)) hide)
     )
   )
@@
     (effects (font (size 0.889 0.889)) (justify right))
     (property "Intersheetrefs" "${INTERSHEET_REFS}" (at 331.47 229.87 0)
-      (effects (font (size 1.27 1.27)) hide)
-    )
-  )
-  (global_label "USB_OTG_FS_ID" (shape bidirectional) (at 162.56 129.54 180) (fields_autoplaced)
-    (effects (font (size 0.889 0.889)) (justify right))
-    (property "Intersheetrefs" "${INTERSHEET_REFS}" (at 335.28 203.2 0)
-      (effects (font (size 1.27 1.27)) hide)
-    )
-  )
-  (global_label "SD_DAT3" (shape input) (at 258.064 103.632 0)
-    (effects (font (size 1.524 1.524)) (justify left))
-    (property "Intersheetrefs" "${INTERSHEET_REFS}" (at 258.064 103.632 0)
       (effects (font (size 1.27 1.27)) hide)
     )
@@
     )
   )
-  (global_label "USB_OTG_FS_D_N" (shape bidirectional) (at 162.56 134.62 180) (fields_autoplaced)
-    (effects (font (size 0.889 0.889)) (justify right))
-    (property "Intersheetrefs" "${INTERSHEET_REFS}" (at 335.28 203.2 0)
-      (effects (font (size 1.27 1.27)) hide)
-    )
-  )
