File: EEZ_BB3_CM4_H7/STM32H7_MCU.kicad_sch (KiCad schematic)
At the start: 68 parts, among them IC2 STM32H745IIT6, IC3 AP1117-33, Y1 XTAL016178-85SMX

Commit message: Routing
Parts:
- removed R10, R2, R4, R7: 1K5, Library:R_0402_1005Metric, symbol Library:Envox_R-EU_R0402
- IC2: value STM32H745IIT6 -> STM32H757IIT6; symbol Library:STM32H745IIT6 -> Library:STM32H757IIT6
Connections:
- net PDR_ON is gone; now on net BOOT0: IC2.174 (PDR_ON), JP1.COM
- net SLAVE1_RX_OE is gone; now on net IRQ_TOUCH: IC2.150 (PD7)
- net VSSA is gone; now on net VDD_SDC: C33.2, C34.2, IC2.38 (VSSA), NT2.2
- net +VDD_MCU: no longer IC2.105 (VDD.105)
- net GND: now also IC2.105 (VSSDSI.105), IC2.109 (VSSDSI.109); no longer IC2.106 (VSS.106)
- net IRQ_TOUCH: no longer IC2.94 (PD11)
- net LTDC_B3: no longer IC2.127 (PA8)
- net LTDC_B4: no longer IC2.156 (PG12)
- net LTDC_B5: no longer IC2.46 (PA3)
- net LTDC_B6: no longer IC2.168 (PB8)
- net LTDC_B7: no longer IC2.169 (PB9)
- net LTDC_CLK: no longer IC2.117 (PG7)
- net LTDC_DE: no longer IC2.30 (PF10)
- net LTDC_G2: no longer IC2.51 (PA6)
- net LTDC_G3: no longer IC2.103 (PJ10)
- net LTDC_G4: no longer IC2.104 (PJ11)
- net LTDC_G5: no longer IC2.107 (PK0)
- net LTDC_G6: no longer IC2.108 (PK1)
- net LTDC_G7: no longer IC2.109 (PK2)
- net LTDC_HSYNC: no longer IC2.122 (PC6)
- net LTDC_R3: no longer IC2.55 (PB0)
- net LTDC_R4: no longer IC2.130 (PA11)
- net LTDC_R5: no longer IC2.131 (PA12)
- net LTDC_R6: no longer IC2.56 (PB1)
- net LTDC_R7: no longer IC2.116 (PG6)
- net LTDC_VSYNC: no longer IC2.49 (PA4)
- net SLAVE4_RX: no longer IC2.102 (PJ9)
- net SLAVE4_TX: no longer IC2.101 (PJ8)
- net SYS_SCL: no longer IC2.95 (PD12)
- net SYS_SDA: no longer IC2.96 (PD13)
- net TFT_BRIGHTNESS: now also IC2.95 (PD12); no longer IC2.123 (PC7)
- net USB_OTG_HS_D_N: now also IC2.130 (PA11); no longer IC2.87 (PB14)
- net USB_OTG_HS_D_P: now also IC2.131 (PA12); no longer IC2.88 (PB15)
- net BTM_FAN_PWM: no longer names the net of IC2.164 (PB5)
- net IOEXP_GPIO0 renamed SPI4_CLK
- net IOEXP_GPIO1 renamed SPI4_MISO
- net IOEXP_GPIO2 renamed SPI4_MOSI
- net IOEXP_GPIO3 renamed ENC_SW
- net IOEXP_I2C1_SCL renamed I2C1_SCL
- net IOEXP_I2C1_SDA renamed I2C1_SDA
- net IOEXP_I2C2_SCL: no longer names the net of IC2.78 (PB10)
- net IOEXP_I2C2_SDA: no longer names the net of IC2.79 (PB11)
- net IOEXP_SPI_CLK: no longer names the net of IC2.140 (PC10)
- net IOEXP_SPI_MISO renamed SPI2_CSA
- net IOEXP_SPI_MOSI renamed ~{FAULT}
- net IRQ_IOEXP8: no longer names the net of IC2.153 (PG9)
- net PANIC_SW renamed SPI4_CSA
- net RAY_TMP renamed SPI5_MOSI
- net RS485_RX renamed USB_OTG_ID
- net RS485_TX: no longer names the net of IC2.128 (PA9)
- net RS485_TX_EN renamed PWR_SSTART
- net SLAVE1_RX: no longer names the net of IC2.141 (PC11)
- net SLAVE1_TX renamed UART_TX/DOUT1
- net SLAVE2_RX renamed RTC_REF
- net SLAVE2_RX_OE renamed PWR_DIRECT
- net SLAVE2_TX renamed SPI2_CLK
- net SLAVE3_RX renamed SPI5_CSA
- net SLAVE3_RX_OE renamed DOUT2
- net SLAVE3_TX renamed SPI5_IRQ
- net SLAVE4_RX_OE: no longer names the net of IC2.147 (PD4)
- net TEST_24V_AIN renamed SPI5_CLK
- net TOP_FAN_PWM renamed SPI5_MISO
- net ~{IOEXP_RESET} renamed SPI4_CSB
- net ~{MTR_BRK}: no longer names the net of IC2.154 (PG10)
- net ~{MTR_EN}: no longer names the net of IC2.146 (PD3)
- net ~{RESET} renamed nEXTRST
- new net DAC_OUT1: IC2.49 (PA4)
- new net DIN2: IC2.46 (PA3)
- new net DSI0_C_N: IC2.107 (DSI_CKN)
- new net DSI0_C_P: IC2.106 (DSI_CKP)
- new net DSI0_D0_N: IC2.104 (DSI_D0N)
- new net DSI0_D0_P: IC2.103 (DSI_D0P)
- new net ENC_A: IC2.122 (PC6)
- new net ENC_B: IC2.123 (PC7)
- new net OE_SYNC: IC2.96 (PD13)
- new net SD_DETECT: IC2.117 (PG7)
- new net SPI2_CSB: IC2.94 (PD11)
- new net SPI2_IRQ: IC2.127 (PA8)
- new net SPI2_MISO: IC2.87 (PB14)
- new net SPI2_MOSI: IC2.88 (PB15)
- new net SPI4_IRQ: IC2.169 (PB9)
- new net SPI5_CSB: IC2.156 (PG12)
- new net UART_RX/DIN1: IC2.168 (PB8)
- new net USER_SW: IC2.116 (PG6)
- no-connect marks 0 -> 4
Other:
- note added: "SD_DETECT"
- moved on the sheet: C33, C34, C35, C36, L2, NT2, R13

Commit message: Routing adding ioc
Connections:
- net ETH_TX_EN: now also IC2.79 (PB11); no longer IC2.155 (PG11)
- net IRQ_TOUCH: now also IC2.146 (PD3); no longer IC2.150 (PD7)
- net PWR_DIRECT: now also IC2.56 (PB1); no longer IC2.149 (PD6)
- net PWR_SSTART: now also IC2.55 (PB0); no longer IC2.111 (PG3)
- net SPI2_CSA: now also IC2.140 (PC10); no longer IC2.163 (PB4)
- net SPI4_IRQ: now also IC2.111 (PG3); no longer IC2.169 (PB9)
- net SPI5_CLK: now also IC2.155 (PG11); no longer IC2.27 (PF7)
- net SPI5_CSB: now also IC2.51 (PA6); no longer IC2.156 (PG12)
- net SPI5_MISO: now also IC2.163 (PB4); no longer IC2.28 (PF8)
- net SPI5_MOSI: now also IC2.164 (PB5); no longer IC2.29 (PF9)
- no-connect marks 4 -> 13
Changed lines of the file:
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@@
   (junction (at 206.502 86.106) (diameter 0) (color 0 0 0 0)
   )
-  (no_connect (at 59.69 68.58))
-  (no_connect (at 59.69 40.64))
+  (no_connect (at 90.17 83.82))
+  (no_connect (at 59.69 91.44))
+  (no_connect (at 147.32 86.36))
+  (no_connect (at 59.69 93.98))
   (no_connect (at 147.32 93.98))
-  (no_connect (at 59.69 71.12))
+  (no_connect (at 59.69 48.26))
+  (no_connect (at 90.17 78.74))
+  (no_connect (at 90.17 86.36))
+  (no_connect (at 147.32 91.44))
+  (no_connect (at 147.32 88.9))
+  (no_connect (at 177.8 50.8))
+  (no_connect (at 177.8 55.88))
+  (no_connect (at 177.8 48.26))
   (wire (pts (xy 130.81 147.32) (xy 140.97 147.32))
     (stroke (width 0.1524) (type solid))
@@
   )
   (wire (pts (xy 209.55 99.06) (xy 198.12 99.06))
-    (stroke (width 0.1524) (type solid))
-  )
-  (wire (pts (xy 147.32 91.44) (xy 140.97 91.44))
     (stroke (width 0.1524) (type solid))
   )
@@
     (stroke (width 0.1524) (type solid))
   )
+  (wire (pts (xy 59.69 81.28) (xy 53.34 81.28))
+    (stroke (width 0) (type default))
+  )
   (wire (pts (xy 147.32 78.74) (xy 140.97 78.74))
     (stroke (width 0.1524) (type solid))
@@
     (stroke (width 0) (type default))
   )
+  (wire (pts (xy 90.17 50.8) (xy 96.266 50.8))
+    (stroke (width 0) (type default))
+  )
   (wire (pts (xy 216.662 75.946) (xy 211.582 75.946))
     (stroke (width 0.1524) (type solid))
@@
     (stroke (width 0.1524) (type solid))
   )
-  (wire (pts (xy 90.17 86.36) (xy 96.52 86.36))
-    (stroke (width 0.1524) (type solid))
-  )
   (wire (pts (xy 266.7 106.68) (xy 269.24 106.68))
     (stroke (width 0.1524) (type solid))
@@
     (stroke (width 0.1524) (type solid))
   )
+  (wire (pts (xy 53.848 71.12) (xy 59.69 71.12))
+    (stroke (width 0) (type default))
+  )
   (wire (pts (xy 236.22 35.56) (xy 233.68 35.56))
     (stroke (width 0.1524) (type solid))
@@
     (stroke (width 0.1524) (type solid))
   )
+  (wire (pts (xy 96.52 76.2) (xy 90.17 76.2))
+    (stroke (width 0) (type default))
+  )
   (wire (pts (xy 236.22 90.17) (xy 233.68 90.17))
     (stroke (width 0.1524) (type solid))
   )
-  (wire (pts (xy 177.8 55.88) (xy 184.15 55.88))
-    (stroke (width 0.1524) (type solid))
-  )
   (wire (pts (xy 177.8 38.1) (xy 184.15 38.1))
     (stroke (width 0.1524) (type solid))
@@
   )
   (wire (pts (xy 233.68 69.85) (xy 233.68 72.39))
-    (stroke (width 0.1524) (type solid))
-  )
-  (wire (pts (xy 59.69 91.44) (xy 53.34 91.44))
     (stroke (width 0.1524) (type solid))
   )
@@
     (stroke (width 0.1524) (type solid) (color 132 0 132 1))
   )
+  (wire (pts (xy 53.848 68.58) (xy 59.69 68.58))
+    (stroke (width 0) (type default))
+  )
   (wire (pts (xy 99.06 119.38) (xy 99.06 124.46))
     (stroke (width 0.1524) (type solid))
@@
     (stroke (width 0.1524) (type solid))
   )
-  (wire (pts (xy 147.32 88.9) (xy 140.97 88.9))
-    (stroke (width 0.1524) (type solid))
+  (wire (pts (xy 53.34 40.64) (xy 59.69 40.64))
+    (stroke (width 0) (type default))
   )
   (wire (pts (xy 269.24 50.8) (xy 269.24 53.34))
@@
     (stroke (width 0.1524) (type solid))
   )
+  (wire (pts (xy 59.69 96.52) (xy 53.34 96.52))
+    (stroke (width 0) (type default))
+  )
   (wire (pts (xy 229.616 81.28) (xy 233.68 81.28))
     (stroke (width 0.1524) (type solid))
@@
   (wire (pts (xy 233.68 81.28) (xy 236.22 81.28))
     (stroke (width 0) (type default))
-  )
-  (wire (pts (xy 90.17 83.82) (xy 96.52 83.82))
-    (stroke (width 0.1524) (type solid))
   )
   (wire (pts (xy 120.65 134.62) (xy 115.57 134.62))
@@
   )
   (wire (pts (xy 236.22 69.85) (xy 233.68 69.85))
-    (stroke (width 0.1524) (type solid))
-  )
-  (wire (pts (xy 147.32 86.36) (xy 140.97 86.36))
     (stroke (width 0.1524) (type solid))
   )
@@
     )
   )
-  (global_label "SPI5_CLK" (shape output) (at 140.97 86.36 180) (fields_autoplaced)
-    (effects (font (size 0.889 0.889)) (justify right))
-    (property "Intersheetrefs" "${INTERSHEET_REFS}" (at 132.7554 86.36 0)
-      (effects (font (size 1.27 1.27)) (justify right) hide)
+  (global_label "SPI5_CLK" (shape output) (at 184.15 53.34 0) (fields_autoplaced)
+    (effects (font (size 0.889 0.889)) (justify left))
+    (property "Intersheetrefs" "${INTERSHEET_REFS}" (at 192.3646 53.34 0)
+      (effects (font (size 1.27 1.27)) (justify left) hide)
     )
   )
@@
     )
   )
-  (global_label "PWR_DIRECT" (shape output) (at 96.52 83.82 0) (fields_autoplaced)
-    (effects (font (size 0.889 0.889)) (justify left))
-    (property "Intersheetrefs" "${INTERSHEET_REFS}" (at 106.5971 83.82 0)
-      (effects (font (size 1.27 1.27)) (justify left) hide)
+  (global_label "PWR_DIRECT" (shape output) (at 53.848 71.12 180) (fields_autoplaced)
+    (effects (font (size 0.889 0.889)) (justify right))
+    (property "Intersheetrefs" "${INTERSHEET_REFS}" (at 43.7709 71.12 0)
+      (effects (font (size 1.27 1.27)) (justify right) hide)
     )
   )
@@
     )
   )
-  (global_label "SPI4_IRQ" (shape output) (at 53.34 91.44 180) (fields_autoplaced)
-    (effects (font (size 0.889 0.889)) (justify right))
-    (property "Intersheetrefs" "${INTERSHEET_REFS}" (at 45.3795 91.44 0)
-      (effects (font (size 1.27 1.27)) (justify right) hide)
+  (global_label "SPI4_IRQ" (shape output) (at 184.15 33.02 0) (fields_autoplaced)
+    (effects (font (size 0.889 0.889)) (justify left))
+    (property "Intersheetrefs" "${INTERSHEET_REFS}" (at 192.1105 33.02 0)
+      (effects (font (size 1.27 1.27)) (justify left) hide)
     )
   )
@@
     )
   )
-  (global_label "SPI5_MISO" (shape input) (at 140.97 88.9 180) (fields_autoplaced)
-    (effects (font (size 0.889 0.889)) (justify right))
-    (property "Intersheetrefs" "${INTERSHEET_REFS}" (at 132.0358 88.9 0)
+  (global_label "SPI5_MISO" (shape input) (at 53.34 78.74 180) (fields_autoplaced)
+    (effects (font (size 0.889 0.889)) (justify right))
+    (property "Intersheetrefs" "${INTERSHEET_REFS}" (at 44.4058 78.74 0)
       (effects (font (size 1.27 1.27)) (justify right) hide)
     )
@@
     )
   )
-  (global_label "SPI5_CSB" (shape bidirectional) (at 184.15 55.88 0) (fields_autoplaced)
-    (effects (font (size 0.889 0.889)) (justify left))
-    (property "Intersheetrefs" "${INTERSHEET_REFS}" (at 193.2695 55.88 0)
-      (effects (font (size 1.27 1.27)) (justify left) hide)
+  (global_label "SPI5_CSB" (shape bidirectional) (at 53.34 40.64 180) (fields_autoplaced)
+    (effects (font (size 0.889 0.889)) (justify right))
+    (property "Intersheetrefs" "${INTERSHEET_REFS}" (at 44.2205 40.64 0)
+      (effects (font (size 1.27 1.27)) (justify right) hide)
     )
   )
@@
     )
   )
-  (global_label "SPI2_CSA" (shape output) (at 53.34 78.74 180) (fields_autoplaced)
-    (effects (font (size 0.889 0.889)) (justify right))
-    (property "Intersheetrefs" "${INTERSHEET_REFS}" (at 45.1254 78.74 0)
-      (effects (font (size 1.27 1.27)) (justify right) hide)
+  (global_label "SPI2_CSA" (shape output) (at 96.266 50.8 0) (fields_autoplaced)
+    (effects (font (size 0.889 0.889)) (justify left))
+    (property "Intersheetrefs" "${INTERSHEET_REFS}" (at 104.4806 50.8 0)
+      (effects (font (size 1.27 1.27)) (justify left) hide)
     )
   )
@@
     )
   )
-  (global_label "SPI5_MOSI" (shape output) (at 140.97 91.44 180) (fields_autoplaced)
-    (effects (font (size 0.889 0.889)) (justify right))
-    (property "Intersheetrefs" "${INTERSHEET_REFS}" (at 132.0358 91.44 0)
+  (global_label "SPI5_MOSI" (shape output) (at 53.34 81.28 180) (fields_autoplaced)
+    (effects (font (size 0.889 0.889)) (justify right))
+    (property "Intersheetrefs" "${INTERSHEET_REFS}" (at 44.4058 81.28 0)
       (effects (font (size 1.27 1.27)) (justify right) hide)
     )
@@
     )
   )
-  (global_label "PWR_SSTART" (shape output) (at 184.15 33.02 0) (fields_autoplaced)
-    (effects (font (size 0.889 0.889)) (justify left))
-    (property "Intersheetrefs" "${INTERSHEET_REFS}" (at 194.3542 33.02 0)
-      (effects (font (size 1.27 1.27)) (justify left) hide)
+  (global_label "PWR_SSTART" (shape output) (at 53.848 68.58 180) (fields_autoplaced)
+    (effects (font (size 0.889 0.889)) (justify right))
+    (property "Intersheetrefs" "${INTERSHEET_REFS}" (at 43.6438 68.58 0)
+      (effects (font (size 1.27 1.27)) (justify right) hide)
     )
   )
@@
     )
   )
-  (global_label "IRQ_TOUCH" (shape output) (at 96.52 86.36 0) (fields_autoplaced)
-    (effects (font (size 0.889 0.889)) (justify left))
-    (property "Intersheetrefs" "${INTERSHEET_REFS}" (at 105.835 86.36 0)
+  (global_label "IRQ_TOUCH" (shape output) (at 96.52 76.2 0) (fields_autoplaced)
+    (effects (font (size 0.889 0.889)) (justify left))
+    (property "Intersheetrefs" "${INTERSHEET_REFS}" (at 105.835 76.2 0)
       (effects (font (size 1.27 1.27)) (justify left) hide)
     )
@@
     )
   )
-  (global_label "ETH_TX_EN" (shape bidirectional) (at 184.15 53.34 0) (fields_autoplaced)
-    (effects (font (size 0.889 0.889)) (justify left))
-    (property "Intersheetrefs" "${INTERSHEET_REFS}" (at 194.0445 53.34 0)
-      (effects (font (size 1.27 1.27)) (justify left) hide)
-    )
-  )
+  (global_label "ETH_TX_EN" (shape bidirectional) (at 53.34 96.52 180) (fields_autoplaced)
+    (effects (font (size 0.889 0.889)) (justify right))
+    (property "Intersheetrefs" "${INTERSHEET_REFS}" (at 43.5011 96.52 0)
+      (effects (font (size 1.27 1.27)) (justify right) hide)
+    )
+  )

Commit message: Routing - fixing errors
Parts:
- C30: footprint Library:CE5R5105HF-ZJ -> (none)
Connections:
- net SUPER_CAP: now reaches C30.+, R12.1
Other:
- moved on the sheet: D1
Changed lines of the file:
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@@
   (junction (at 181.61 134.62) (diameter 0) (color 0 0 0 0)
   )
+  (junction (at 198.755 20.32) (diameter 0) (color 0 0 0 0)
+  )
   (junction (at 269.24 114.3) (diameter 0) (color 0 0 0 0)
   )
@@
     (stroke (width 0.1524) (type solid))
   )
+  (wire (pts (xy 213.995 15.24) (xy 213.995 17.78))
+    (stroke (width 0) (type default))
+  )
   (wire (pts (xy 90.17 25.4) (xy 96.52 25.4))
     (stroke (width 0.1524) (type solid))
@@
     (stroke (width 0.1524) (type solid))
   )
-  (wire (pts (xy 198.12 17.78) (xy 213.995 17.78))
+  (wire (pts (xy 196.596 20.32) (xy 198.755 20.32))
+    (stroke (width 0) (type default))
+  )
+  (wire (pts (xy 198.12 15.24) (xy 213.995 15.24))
     (stroke (width 0) (type default))
   )
@@
     (stroke (width 0.1524) (type solid))
   )
-  (wire (pts (xy 198.755 20.32) (xy 201.295 20.32))
-    (stroke (width 0) (type default))
-  )
   (wire (pts (xy 233.68 43.18) (xy 233.68 45.72))
     (stroke (width 0.1524) (type solid))
@@
     (stroke (width 0.1524) (type solid))
   )
+  (wire (pts (xy 198.755 20.32) (xy 201.295 20.32))
+    (stroke (width 0) (type default))
+  )
   (polyline (pts (xy 54.356 52.07) (xy 55.118 52.07))
     (stroke (width 0.1524) (type solid) (color 132 0 132 1))
@@
     (stroke (width 0.1524) (type solid))
   )
-  (wire (pts (xy 190.5 17.78) (xy 193.04 17.78))
+  (wire (pts (xy 183.388 15.24) (xy 193.04 15.24))
     (stroke (width 0) (type default))
   )
@@
     )
   )
+  (global_label "SUPER_CAP" (shape input) (at 196.596 20.32 180) (fields_autoplaced)
+    (effects (font (size 1.27 1.27)) (justify right))
+    (property "Intersheetrefs" "${INTERSHEET_REFS}" (at 182.865 20.32 0)
+      (effects (font (size 1.27 1.27)) (justify right) hide)
+    )
+  )
   (global_label "DIN2" (shape input) (at 53.34 33.02 180)
     (effects (font (size 0.889 0.889)) (justify right))
@@
     )
   )
-  (symbol (lib_id "Library:SCHOTTKY") (at 195.58 17.78 0) (unit 1)
+  (symbol (lib_id "Library:SCHOTTKY") (at 195.58 15.24 0) (unit 1)
     (in_bom yes) (on_board yes) (dnp no)
-    (property "Reference" "D1" (at 193.675 15.24 0)
+    (property "Reference" "D1" (at 199.644 14.478 0)
       (effects (font (size 1.778 1.5113)) (justify left bottom))
     )
-    (property "Value" "RB751V40T1G" (at 187.96 20.955 0)
+    (property "Value" "RB751V40T1G" (at 190.5 13.716 0)
       (effects (font (size 0.889 0.889)) (justify left bottom))
     )
-    (property "Footprint" "Library:SOD323-R" (at 195.58 20.32 0)
+    (property "Footprint" "Library:SOD323-R" (at 195.58 17.78 0)
       (effects (font (size 1.27 1.27)) hide)
     )
-    (property "Datasheet" "" (at 195.58 17.78 0)
+    (property "Datasheet" "" (at 195.58 15.24 0)
       (effects (font (size 1.27 1.27)) hide)
     )
@@
     )
   )
-  (symbol (lib_id "Envox H745 Master MCU r2B6-eagle-import:+3V3") (at 187.96 17.78 90) (mirror x) (unit 1)
+  (symbol (lib_id "Envox H745 Master MCU r2B6-eagle-import:+3V3") (at 180.848 15.24 90) (mirror x) (unit 1)
     (in_bom yes) (on_board yes) (dnp no)
-    (property "Reference" "#+3V06" (at 187.96 17.78 0)
+    (property "Reference" "#+3V06" (at 180.848 15.24 0)
       (effects (font (size 1.27 1.27)) hide)
     )
-    (property "Value" "+3V3" (at 182.245 14.605 90)
+    (property "Value" "+3V3" (at 175.133 12.065 90)
       (effects (font (size 1.778 1.5113)) (justify right top))
     )
-    (property "Footprint" "" (at 187.96 17.78 0)
+    (property "Footprint" "" (at 180.848 15.24 0)
       (effects (font (size 1.27 1.27)) hide)
     )
-    (property "Datasheet" "" (at 187.96 17.78 0)
+    (property "Datasheet" "" (at 180.848 15.24 0)
       (effects (font (size 1.27 1.27)) hide)
     )
@@
       (effects (font (size 0.889 0.889)) (justify left bottom))
     )
-    (property "Footprint" "Library:CE5R5105HF-ZJ" (at 198.755 25.4 0)
+    (property "Footprint" "" (at 198.755 25.4 0)
       (effects (font (size 1.27 1.27)) hide)
     )

Commit message: Fixing errors - adding README
Other:
- moved on the sheet: JP1
Changed lines of the file:
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@@
   (junction (at 130.81 134.62) (diameter 0) (color 0 0 0 0)
   )
-  (junction (at 193.04 114.3) (diameter 0) (color 0 0 0 0)
+  (junction (at 193.04 115.57) (diameter 0) (color 0 0 0 0)
   )
   (junction (at 233.68 67.31) (diameter 0) (color 0 0 0 0)
@@
     (stroke (width 0.1524) (type solid))
   )
+  (wire (pts (xy 193.04 117.348) (xy 193.04 115.57))
+    (stroke (width 0) (type default))
+  )
   (wire (pts (xy 233.68 104.14) (xy 233.68 95.25))
     (stroke (width 0.1524) (type solid))
@@
     (stroke (width 0.1524) (type solid))
   )
+  (wire (pts (xy 187.96 115.57) (xy 193.04 115.57))
+    (stroke (width 0.1524) (type solid))
+  )
   (wire (pts (xy 266.7 55.88) (xy 269.24 55.88))
     (stroke (width 0.1524) (type solid))
@@
     (stroke (width 0.1524) (type solid))
   )
+  (wire (pts (xy 179.324 115.57) (xy 182.88 115.57))
+    (stroke (width 0.1524) (type solid))
+  )
   (wire (pts (xy 140.97 154.94) (xy 130.81 154.94))
     (stroke (width 0.1524) (type solid))
@@
     (stroke (width 0.1524) (type solid))
   )
-  (wire (pts (xy 182.88 114.3) (xy 180.34 114.3))
-    (stroke (width 0.1524) (type solid))
-  )
   (wire (pts (xy 140.97 134.62) (xy 130.81 134.62))
     (stroke (width 0.1524) (type solid))
@@
     (stroke (width 0.1524) (type solid))
   )
+  (wire (pts (xy 193.04 115.57) (xy 193.04 114.3))
+    (stroke (width 0) (type default))
+  )
   (wire (pts (xy 233.68 43.18) (xy 233.68 45.72))
     (stroke (width 0.1524) (type solid))
@@
     (stroke (width 0.1524) (type solid))
   )
-  (wire (pts (xy 187.96 114.3) (xy 193.04 114.3))
-    (stroke (width 0.1524) (type solid))
-  )
   (wire (pts (xy 229.362 73.406) (xy 229.362 81.026))
     (stroke (width 0.1524) (type solid))
@@
     (stroke (width 0) (type default))
   )
-  (wire (pts (xy 185.42 111.76) (xy 185.42 104.14))
+  (wire (pts (xy 185.42 113.03) (xy 185.42 104.14))
     (stroke (width 0.1524) (type solid))
   )
@@
     )
   )
-  (symbol (lib_id "Envox H745 Master MCU r2B6-eagle-import:GND") (at 193.04 116.84 0) (mirror y) (unit 1)
+  (symbol (lib_id "Envox H745 Master MCU r2B6-eagle-import:GND") (at 193.04 119.888 0) (mirror y) (unit 1)
     (in_bom yes) (on_board yes) (dnp no)
-    (property "Reference" "#SUPPLY012" (at 193.04 116.84 0)
+    (property "Reference" "#SUPPLY012" (at 193.04 119.888 0)
       (effects (font (size 1.27 1.27)) hide)
     )
-    (property "Value" "GND" (at 191.135 118.745 0)
+    (property "Value" "GND" (at 191.135 121.793 0)
       (effects (font (size 1.778 1.5113)) (justify right top))
     )
-    (property "Footprint" "" (at 193.04 116.84 0)
+    (property "Footprint" "" (at 193.04 119.888 0)
       (effects (font (size 1.27 1.27)) hide)
     )
-    (property "Datasheet" "" (at 193.04 116.84 0)
+    (property "Datasheet" "" (at 193.04 119.888 0)
       (effects (font (size 1.27 1.27)) hide)
     )
@@
     )
   )
-  (symbol (lib_id "Envox H745 Master MCU r2B6-eagle-import:+VDD_MCU") (at 180.34 114.3 90) (mirror x) (unit 1)
+  (symbol (lib_id "Envox H745 Master MCU r2B6-eagle-import:+VDD_MCU") (at 179.324 115.57 90) (mirror x) (unit 1)
     (in_bom yes) (on_board yes) (dnp no)
-    (property "Reference" "#+VDD_MCU01" (at 180.34 114.3 0)
+    (property "Reference" "#+VDD_MCU01" (at 179.324 115.57 0)
       (effects (font (size 1.27 1.27)) hide)
     )
-    (property "Value" "+VDD_MCU" (at 183.515 112.395 90)
+    (property "Value" "+VDD_MCU" (at 182.499 113.665 90)
       (effects (font (size 1.778 1.5113)) (justify left bottom))
     )
-    (property "Footprint" "" (at 180.34 114.3 0)
+    (property "Footprint" "" (at 179.324 115.57 0)
       (effects (font (size 1.27 1.27)) hide)
     )
-    (property "Datasheet" "" (at 180.34 114.3 0)
+    (property "Datasheet" "" (at 179.324 115.57 0)
       (effects (font (size 1.27 1.27)) hide)
     )
@@
     )
   )
-  (symbol (lib_id "Library:JP3-CUT-0805-ROTATED") (at 185.42 114.3 90) (unit 1)
+  (symbol (lib_id "Library:JP3-CUT-0805-ROTATED") (at 185.42 115.57 90) (unit 1)
     (in_bom no) (on_board yes) (dnp no)
-    (property "Reference" "JP1" (at 183.515 117.475 90)
+    (property "Reference" "JP1" (at 183.515 118.745 90)
       (effects (font (size 1.778 1.5113)) (justify right top))
     )
-    (property "Value" "JP3-CUT-0805-ROTATED" (at 185.42 114.3 0)
+    (property "Value" "JP3-CUT-0805-ROTATED" (at 185.42 115.57 0)
       (effects (font (size 1.27 1.27)) hide)
     )
-    (property "Footprint" "Library:JP3-0805-CUT2" (at 185.42 114.3 0)
+    (property "Footprint" "Library:JP3-0805-CUT2" (at 185.42 115.57 0)
       (effects (font (size 1.27 1.27)) hide)
     )
-    (property "Datasheet" "" (at 185.42 114.3 0)
+    (property "Datasheet" "" (at 185.42 115.57 0)
       (effects (font (size 1.27 1.27)) hide)
     )
