File: EEZ_BB3_CM4_H7/cm4_connector.kicad_sch (KiCad schematic)
At the start: 2 parts, among them J1 DF40C-100DP-0.4V(51), J2 DF40C-100DP-0.4V(51)

Commit message: Routing
Connections:
- net GPIO14: no longer J1.61
- net GPIO15: no longer J1.57
- net GPIO2: no longer J1.69
- net GPIO27: no longer J1.62
- net GPIO3: no longer J1.67
- net GPIO4: no longer J1.63
- net USB_N renamed USB_OTG_HS_D_N
- net USB_P renamed USB_OTG_HS_D_P
- new net SD_CLK: J1.57
- new net SD_CMD: J1.62
- new net SD_DAT0: J1.63
- new net SD_DAT1: J1.67
- new net SD_DAT2: J1.69
- new net SD_DAT3: J1.61

Commit message: Routing
Other:
- note added: "SD_DETECT"
Changed lines of the file:
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@@
     (effects (font (size 1.524 1.524)) (justify left bottom))
+  )
+  (text "SD_DETECT" (at 116.078 76.962 0)
+    (effects (font (size 1.27 1.27)) (justify left bottom))
   )
   (global_label "GND" (shape input) (at 167.64 33.02 180)

Commit message: Adding GPIO connections
Connections:
- net GPIO25 is gone; now on net DIN2: J1.41
- net GPIO5 is gone; now on net DAC_OUT1: J1.34
- net SCL0 is gone; now on net I2C1_SCL: J1.80
- net SDA0 is gone; now on net I2C1_SDA: J1.82
- net GPIO16 renamed DOUT2
- net GPIO2 renamed ENC_A
- net GPIO24 renamed ENC_SW
- net GPIO3 renamed ENC_B

Commit message: Routing adding ioc
Connections:
- net AnalogIP0 is gone; now on net AUDIO_OUT: J1.96
- net SD_PWR_ON renamed SD_DETECT
- net nRPIBOOT renamed BOOT0

Commit message: Routing - fixing errors
Changed lines of the file:
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@@
+    (stroke (width 0) (type default))
+  )
+  (wire (pts (xy 248.412 155.448) (xy 249.174 155.448))
     (stroke (width 0) (type default))
   )
@@
     )
   )
+  (global_label "HDMI0_SCL" (shape input) (at 249.174 155.448 0)
+    (effects (font (size 1.524 1.524)) (justify left))
+    (property "Intersheetrefs" "${INTERSHEET_REFS}" (at 249.174 155.448 0)
+      (effects (font (size 1.27 1.27)) hide)
+    )
+  )
   (global_label "GPIO16" (shape input) (at 25.908 69.342 180)
     (effects (font (size 1.524 1.524)) (justify right))
@@
     )
   )
+  (global_label "SUPER_CAP" (shape input) (at 248.412 155.448 180) (fields_autoplaced)
+    (effects (font (size 1.27 1.27)) (justify right))
+    (property "Intersheetrefs" "${INTERSHEET_REFS}" (at 234.681 155.448 0)
+      (effects (font (size 1.27 1.27)) (justify right) hide)
+    )
+  )

Commit message: Updating pinout
Other:
- note added: "USB_OTG_FS_PSO USB_OTG_FS_OC USB_OTG_FS_VBUS USB_OTG_FS_ID"
Changed lines of the file:
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@@
     (stroke (width 0) (type default))
+  )
+  (text "USB_OTG_FS_PSO\nUSB_OTG_FS_OC\nUSB_OTG_FS_VBUS\nUSB_OTG_FS_ID"
+    (at 123.19 30.48 0)
+    (effects (font (size 1.27 1.27)) (justify left bottom))
   )
   (text "CM4 needs to provide 3.3V to CM4 IO board" (at 122.555 140.97 90)

Commit message: Adding USB
Connections:
- net HDMI0_TX1_N renamed DIN3
- net HDMI0_TX1_P renamed DOUT3
Other:
- note removed: "SD_DETECT"
- note removed: "USB_OTG_FS_PSO USB_OTG_FS_OC USB_OTG_FS_VBUS USB_OTG_FS_ID"

Commit message: Moving components - moving EEZ logo to top
Connections:
- no-connect marks 0 -> 3
Changed lines of the file:
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@@
   (junction (at 161.29 128.27) (diameter 0) (color 0 0 0 0)
   )
+  (no_connect (at 261.62 27.94))
+  (no_connect (at 194.31 119.38))
+  (no_connect (at 261.62 30.48))
   (wire (pts (xy 167.64 88.9) (xy 168.91 88.9))
     (stroke (width 0) (type default))
